File: gateway/Project Architecture.kicad_sch (KiCad schematic)
At the start: 0 parts

Commit message: Working on PCB
Other:
- sheet Section A renamed Power
- sheet Section B renamed System on Module
- added sheet Battery (Battery.kicad_sch)
- added sheet Interfaces (Interfaces.kicad_sch)
- added sheet Radio (Radio.kicad_sch)
- sheet Power: file Section A - Title A.kicad_sch -> Power A.kicad_sch
- sheet System on Module: file Section B - TItle B.kicad_sch -> SoM.kicad_sch
Changed lines of the file:
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@@
 (kicad_sch
-	(version 20250114)
+	(version 20260306)
 	(generator "eeschema")
-	(generator_version "9.0")
+	(generator_version "10.0")
 	(paper "A3")
 	(title_block
@@
 	(text "Page 8"
 		(exclude_from_sim no)
+		(at 287.02 95.25 0)
+		(effects
+			(font
+				(size 2.54 2.54)
+				(bold yes)
+				(color 100 70 50 1)
+			)
+			(justify right bottom)
+			(href "#8")
+		)
+	)
+	(text "Page 8"
+		(exclude_from_sim no)
 		(at 226.06 133.35 0)
 		(effects
@@
 	)
 	(sheet
-		(at 190.5 114.3)
+		(at 251.46 76.2)
 		(size 36.83 20.32)
 		(exclude_from_sim no)
@@
 		)
 		(fill
-			(color 255 200 0 0.5020)
-		)
-		(property "Sheetname" "Section B"
-			(at 190.5 113.2709 0)
+			(color 255 200 0 0.502)
+		)
+		(property "Sheetname" "Interfaces"
+			(at 251.46 75.1709 0)
+			(show_name no)
+			(do_not_autoplace no)
 			(effects
 				(font
@@
 			)
 		)
-		(property "Sheetfile" "Section B - TItle B.kicad_sch"
+		(property "Sheetfile" "Interfaces.kicad_sch"
+			(at 251.46 97.1046 0)
+			(show_name no)
+			(do_not_autoplace no)
+			(effects
+				(font
+					(face "Arial")
+					(size 1.27 1.27)
+				)
+				(justify left top)
+			)
+		)
+		(instances
+			(project "Gateway"
+				(path "/d5742f03-3b1a-42e5-a384-018bd4b919aa/c5103ceb-5325-4a84-a025-9638a412984e"
+					(page "9")
+				)
+			)
+		)
+	)
+	(sheet
+		(at 298.45 76.2)
+		(size 36.83 20.32)
+		(exclude_from_sim no)
+		(in_bom yes)
+		(on_board yes)
+		(dnp no)
+		(fields_autoplaced yes)
+		(stroke
+			(width 0.1524)
+			(type solid)
+		)
+		(fill
+			(color 255 200 0 0.502)
+		)
+		(property "Sheetname" "Radio"
+			(at 298.45 75.1709 0)
+			(show_name no)
+			(do_not_autoplace no)
+			(effects
+				(font
+					(size 1.905 1.905)
+					(bold yes)
+				)
+				(justify left bottom)
+			)
+		)
+		(property "Sheetfile" "Radio.kicad_sch"
+			(at 298.45 97.1046 0)
+			(show_name no)
+			(do_not_autoplace no)
+			(effects
+				(font
+					(face "Arial")
+					(size 1.27 1.27)
+				)
+				(justify left top)
+			)
+		)
+		(instances
+			(project "Gateway"
+				(path "/d5742f03-3b1a-42e5-a384-018bd4b919aa/c5103ceb-5325-4a84-a025-9638a412984e"
+					(page "10")
+				)
+			)
+		)
+	)
+	(sheet
+		(at 271.78 114.3)
+		(size 36.83 20.32)
+		(exclude_from_sim no)
+		(in_bom yes)
+		(on_board yes)
+		(dnp no)
+		(fields_autoplaced yes)
+		(stroke
+			(width 0.1524)
+			(type solid)
+		)
+		(fill
+			(color 255 200 0 0.502)
+		)
+		(property "Sheetname" "Battery"
+			(at 271.78 113.2709 0)
+			(show_name no)
+			(do_not_autoplace no)
+			(effects
+				(font
+					(size 1.905 1.905)
+					(bold yes)
+				)
+				(justify left bottom)
+			)
+		)
+		(property "Sheetfile" "Battery.kicad_sch"
+			(at 271.78 135.2046 0)
+			(show_name no)
+			(do_not_autoplace no)
+			(effects
+				(font
+					(face "Arial")
+					(size 1.27 1.27)
+				)
+				(justify left top)
+			)
+		)
+		(instances
+			(project "Gateway"
+				(path "/d5742f03-3b1a-42e5-a384-018bd4b919aa/c5103ceb-5325-4a84-a025-9638a412984e"
+					(page "8")
+				)
+			)
+		)
+	)
+	(sheet
+		(at 190.5 114.3)
+		(size 36.83 20.32)
+		(exclude_from_sim no)
+		(in_bom yes)
+		(on_board yes)
+		(dnp no)
+		(fields_autoplaced yes)
+		(stroke
+			(width 0.1524)
+			(type solid)
+		)
+		(fill
+			(color 255 200 0 0.502)
+		)
+		(property "Sheetname" "System on Module"
+			(at 190.5 113.2709 0)
+			(show_name no)
+			(do_not_autoplace no)
+			(effects
+				(font
+					(size 1.905 1.905)
+					(bold yes)
+				)
+				(justify left bottom)
+			)
+		)
+		(property "Sheetfile" "SoM.kicad_sch"
 			(at 190.5 135.2046 0)
+			(show_name no)
+			(do_not_autoplace no)
 			(effects
 				(font
@@
 				)
 			)
-			(project "Template"
+			(project "Gateway"
 				(path "/d5742f03-3b1a-42e5-a384-018bd4b919aa/c5103ceb-5325-4a84-a025-9638a412984e"
-					(page "8")
+					(page "9")
 				)
 			)
@@
 		)
 		(fill
-			(color 128 255 128 0.5000)
-		)
-		(property "Sheetname" "Section A"
+			(color 128 255 128 0.5)
+		)
+		(property "Sheetname" "Power"
 			(at 190.5 75.1709 0)
+			(show_name no)
+			(do_not_autoplace no)
 			(effects
 				(font
@@
 			)
 		)
-		(property "Sheetfile" "Section A - Title A.kicad_sch"
+		(property "Sheetfile" "Power A.kicad_sch"
 			(at 190.5 97.1046 0)
+			(show_name no)
+			(do_not_autoplace no)
 			(effects
 				(font
@@
 				)
 			)
-			(project "Template"
+			(project "Gateway"
 				(path "/d5742f03-3b1a-42e5-a384-018bd4b919aa/c5103ceb-5325-4a84-a025-9638a412984e"
 					(page "7")
