File: gateway/Project Architecture.kicad_sch (KiCad schematic)
At the start: 0 parts

Commit message: Prepare Release 1.0.0
Co-Authored-By: Claude Opus 5.5 <noreply@anthropic.com>
Other:
- note added: "Page 16"
- note added: "Page 6"
- note removed: "Page 17"
Changed lines of the file:
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@@
 		(company "${COMPANY}")
 	)
-	(text "Page 14"
+	(text "Page 13"
 		(exclude_from_sim no)
 		(at 298.45 130.81 0)
@@
 			)
 			(justify right bottom)
-			(href "#14")
-		)
-	)
-	(text "Page 12"
+			(href "#13")
+		)
+	)
+	(text "Page 11"
 		(exclude_from_sim no)
 		(at 298.45 102.87 0)
@@
 			)
 			(justify right bottom)
-			(href "#12")
-		)
-	)
-	(text "Page 13"
+			(href "#11")
+		)
+	)
+	(text "Page 12"
 		(exclude_from_sim no)
 		(at 298.45 73.66 0)
@@
 			)
 			(justify right bottom)
-			(href "#13")
-		)
-	)
-	(text "Page 11"
+			(href "#12")
+		)
+	)
+	(text "Page 10"
 		(exclude_from_sim no)
 		(at 147.32 165.1 0)
@@
 			)
 			(justify right bottom)
-			(href "#11")
-		)
-	)
-	(text "Page 15"
+			(href "#10")
+		)
+	)
+	(text "Page 14"
 		(exclude_from_sim no)
 		(at 298.45 161.29 0)
@@
 			)
 			(justify right bottom)
-			(href "#15")
-		)
-	)
-	(text "Page 17"
+			(href "#14")
+		)
+	)
+	(text "Page 15"
 		(exclude_from_sim no)
 		(at 146.685 194.31 0)
@@
 			)
 			(justify right bottom)
-			(href "#17")
-		)
-	)
-	(text "Page 17"
+			(href "#15")
+		)
+	)
+	(text "Page 16"
 		(exclude_from_sim no)
 		(at 298.45 189.23 0)
@@
 			)
 			(justify right bottom)
-			(href "#17")
-		)
-	)
-	(text "Page 10"
+			(href "#16")
+		)
+	)
+	(text "Page 9"
 		(exclude_from_sim no)
 		(at 224.79 177.8 0)
@@
 			)
 			(justify right bottom)
-			(href "#10")
-		)
-	)
-	(text "Page 7"
+			(href "#9")
+		)
+	)
+	(text "Page 6"
 		(exclude_from_sim no)
 		(at 147.32 73.66 0)
@@
 			)
 			(justify right bottom)
-			(href "#7")
-		)
-	)
-	(text "Page 8"
+			(href "#6")
+		)
+	)
+	(text "Page 7"
 		(exclude_from_sim no)
 		(at 147.32 102.87 0)
@@
 			)
 			(justify right bottom)
-			(href "#8")
-		)
-	)
-	(text "Page 9"
+			(href "#7")
+		)
+	)
+	(text "Page 8"
 		(exclude_from_sim no)
 		(at 147.32 134.62 0)
@@
 			)
 			(justify right bottom)
-			(href "#98")
+			(href "#8")
 		)
 	)
@@
 			(project "Gateway"
 				(path "/d5742f03-3b1a-42e5-a384-018bd4b919aa/c5103ceb-5325-4a84-a025-9638a412984e"
-					(page "7")
+					(page "6")
 				)
 			)
@@
 			(project "Gateway"
 				(path "/d5742f03-3b1a-42e5-a384-018bd4b919aa/c5103ceb-5325-4a84-a025-9638a412984e"
-					(page "13")
+					(page "12")
 				)
 			)
@@
 			(project "Gateway"
 				(path "/d5742f03-3b1a-42e5-a384-018bd4b919aa/c5103ceb-5325-4a84-a025-9638a412984e"
-					(page "11")
+					(page "10")
 				)
 			)
@@
 			(project "Gateway"
 				(path "/d5742f03-3b1a-42e5-a384-018bd4b919aa/c5103ceb-5325-4a84-a025-9638a412984e"
-					(page "12")
+					(page "11")
 				)
 			)
@@
 			(project "Gateway"
 				(path "/d5742f03-3b1a-42e5-a384-018bd4b919aa/c5103ceb-5325-4a84-a025-9638a412984e"
-					(page "16")
+					(page "15")
 				)
 			)
@@
 			(project "Gateway"
 				(path "/d5742f03-3b1a-42e5-a384-018bd4b919aa/c5103ceb-5325-4a84-a025-9638a412984e"
-					(page "14")
+					(page "13")
 				)
 			)
@@
 			(project "Gateway"
 				(path "/d5742f03-3b1a-42e5-a384-018bd4b919aa/c5103ceb-5325-4a84-a025-9638a412984e"
-					(page "15")
+					(page "14")
 				)
 			)
@@
 			(project "Gateway"
 				(path "/d5742f03-3b1a-42e5-a384-018bd4b919aa/c5103ceb-5325-4a84-a025-9638a412984e"
-					(page "17")
+					(page "16")
 				)
 			)
@@
 			(project "Gateway"
 				(path "/d5742f03-3b1a-42e5-a384-018bd4b919aa/c5103ceb-5325-4a84-a025-9638a412984e"
-					(page "9")
+					(page "8")
 				)
 			)
@@
 			(project "Gateway"
 				(path "/d5742f03-3b1a-42e5-a384-018bd4b919aa/c5103ceb-5325-4a84-a025-9638a412984e"
-					(page "10")
+					(page "9")
 				)
 			)
@@
 			(project "Gateway"
 				(path "/d5742f03-3b1a-42e5-a384-018bd4b919aa/c5103ceb-5325-4a84-a025-9638a412984e"
-					(page "8")
-				)
-			)
+					(page "7")
+				)
+			)
