File: gateway/Radio.kicad_sch (KiCad schematic)
At the start: 0 parts

Commit message: Working on PCB
Other:
- title: Block Diagram -> System on Module
Changed lines of the file:
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@@
 	(paper "A3")
 	(title_block
-		(title "Block Diagram")
+		(title "System on Module")
 		(date "2025-06-05")
 		(rev "${REVISION}")
