File: gateway/Section A - Title A.kicad_sch (KiCad schematic)
At the start: 1 part

Commit message: Working on PCB
Parts:
- removed R1: 100R, Resistor_SMD:R_0805_2012Metric_Pad1.20x1.40mm_HandSolder, symbol Device:R
- added C801, C802, C807, C808, C815, C823, C832, C836, C838: 10u, symbol Device:C
- added C803, C806: 2u2, symbol Device:C
- added C804, C805, C811, C813, C817, C819, C821, C828, C830, C840: 100n, symbol Device:C
- added C809, C810, C812, C816, C818, C820, C824, C825, C826, C827, C829, C833, C834, C835: 1u, symbol Device:C
- added C814, C822, C831: 10n, symbol Device:C
- added C837, C839: 470n, symbol Device:C
- added C841, C842, C843, C844, C845: 22u, symbol Device:C
- added C846: 10p, symbol Device:C
- added D801: Power, symbol Device:LED
- added F801: 3 A, symbol Device:Fuse
- added IC801, IC802: XC6220B331MR, Package_TO_SOT_SMD:SOT-23-5, symbol Regulator_Linear:XC6220B331MR
- added IC803, IC806: MIC5317-1.8xM5, Package_TO_SOT_SMD:SOT-23-5, symbol Regulator_Linear:MIC5317-1.8xM5
- added IC804: TLV75801PDBV, Package_TO_SOT_SMD:SOT-23-5, symbol Regulator_Linear:TLV75801PDBV
- added IC805: MIC5317-2.5xM5, Package_TO_SOT_SMD:SOT-23-5, symbol Regulator_Linear:MIC5317-2.5xM5
- added IC807: LM62460, Package_QFN:RPH0016A, symbol Texas Instruments:LM62460
- added L801: 2u7, symbol Device:L
- added R801, R802, R805, R806: 10k, symbol Device:R
- added R803, R804: 3k3, symbol Device:R
- added R807: 4k99, symbol Device:R
- added R808: 100k, symbol Device:R
- added R809: 24k9, symbol Device:R
- added R810: 3k, symbol Device:R
- added TP801, TP802, TP803, TP804, TP805, TP806, TP807, TP808, TP809, TP810: ~, symbol Connector:TestPoint
- added X1: 7-24 V, symbol Connector_Generic:Conn_01x02
Connections:
- new net: C846.1, IC807.5 (BIAS), IC807.7 (FB), R808.2, R809.1
- new net: C846.2, R807.2
- new net: C840.2, IC807.16 (SW), L801.1
- new net: IC804.4 (FB), R803.2, R804.1
- new net: F801.1, X1.2 (Pin_2)
- new net: IC807.10 (RESET), R806.2, TP807.1
- new net: C835.2, IC807.11 (SpSp), IC807.6 (VCC), IC807.9 (RT)
- new net: D801.2 (A), R810.2
- new net: C840.1, IC807.3 (RBOOT), IC807.4 (CBOOT)
- new net +1V8: C834.2, IC806.5 (VOUT), TP808.1
- new net +5V: C801.1, C808.1, C809.2, C825.2, C826.2, C833.2, C841.2, C842.2, C843.2, C844.2, C845.2, IC801.1 (VIN), IC802.1 (VIN), IC803.1 (VIN), IC803.3 (EN), IC804.1 (IN), IC804.3 (EN), IC805.1 (VIN), IC805.3 (EN), IC806.1 (VIN), L801.2, R807.1, R808.1, R810.1, TP806.1
- new net GND: C801.2, C802.2, C803.2, C804.2, C805.2, C806.2, C807.2, C808.2, C809.1, C810.1, C811.1, C812.1, C813.1, C814.1, C815.1, C816.1, C817.1, C818.1, C819.1, C820.1, C821.1, C822.1, C823.1, C824.1, C825.1, C826.1, C827.1, C828.1, C829.1, C830.1, C831.1, C832.1, C833.1, C834.1, C835.1, C836.1, C837.1, C838.1, C839.1, C841.1, C842.1, C843.1, C844.1, C845.1, D801.1 (K), IC801.2 (GND), IC802.2 (GND), IC803.2 (GND), IC804.2 (GND), IC805.2 (GND), IC806.2 (GND), IC807.1 (PGND), IC807.12 (SYNC_MODE), IC807.15 (PGND), IC807.8 (AGND), R801.2, R802.2, R804.2, R805.2, R809.2, X1.1 (Pin_1)
- new net SFP-Enable: IC801.3 (CE), IC802.3 (CE), R801.1, R802.1
- new net SFP-PHY-VCCA_{2P5}: C827.2, C828.2, C829.2, C830.2, C831.2, C832.2, IC805.5 (VOUT), TP801.1
- new net SFP-PHY-VCC_{1P1}: C816.2, C817.2, C818.2, C819.2, C820.2, C821.2, C822.2, C823.2, C824.2, IC804.5 (OUT), R803.1, TP802.1
- new net SFP-PHY-VCC_{IO}: C810.2, C811.2, C812.2, C813.2, C814.2, C815.2, IC803.5 (VOUT), TP805.1
- new net SFP-VCC_{R}: C805.1, C806.1, C807.1, IC802.5 (VOUT), TP804.1
- new net SFP-VCC_{T}: C802.1, C803.1, C804.1, IC801.5 (VOUT), TP803.1
- new net SoM-Power-Enable: IC806.3 (EN), R805.1
- new net VDD: C836.2, C837.2, C838.2, C839.2, F801.2, IC807.13 (EN), IC807.14 (VIN), IC807.2 (VIN), R806.1, TP809.1, TP810.1
Other:
- note removed: "AN5346"
- note removed: "J. Pieper ADC investigation"
- note removed: "STM32G474 Datasheet p.81"
- title: Section A -> Power
