File: gateway/Power - Topology.kicad_sch (KiCad schematic)
At the start: 0 parts

Commit message: Working on first version
Changed lines of the file:
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@@
 		)
 	)
-	(text_box "?? - ?? V"
+	(text_box "7 - 24 V"
 		(exclude_from_sim no)
 		(at 381 208.28 0)
-		(size 24.13 7.62)
+		(size 24.13 9.3123)
 		(margins 2.2859 2.2859 2.2859 2.2859)
 		(stroke
 			(width -0.0001)
-			(type default)
+			(type solid)
 		)
 		(fill

Commit message: Working on version 1.0
Changed lines of the file:
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@@
 		)
 	)
-	(text_box "7 - 24 V"
+	(text_box "7 - 16 V"
 		(exclude_from_sim no)
 		(at 381 208.28 0)
