File: gateway/Gateway.kicad_pcb (KiCad board)
At the start: 4 copper layers, 15 x 11 mm, 1 part

Commit message: Working on version 1.0
Parts:
- removed R1: 100R, Resistor_SMD:R_0805_2012Metric_Pad1.20x1.40mm_HandSolder
Routing:
- net Net-(R1-Pad1): track 21.4 -> 0.00 mm
- net (no net): vias 9 -> 0
Other:
- board outline removed

Commit message: Working on PCB
Parts:
- added BAT801: Backup Power, Keystone:1043, F.Cu at (152.3, -125.3)
- added C1001: 1u, Capacitor_SMD:C_0805_2012Metric, F.Cu at (198.1, -26.6)
- added C1002: 1u, Capacitor_SMD:C_0805_2012Metric, F.Cu at (198.1, -23.6)
- added C1003: 100n, Capacitor_SMD:C_0805_2012Metric, F.Cu at (198.1, -20.6)
- added C1004: 100n, Capacitor_SMD:C_0805_2012Metric, F.Cu at (198.1, -17.6)
- added C1005: 27p, Capacitor_SMD:C_0805_2012Metric, F.Cu at (198.1, -14.6)
- added C1006: 27p, Capacitor_SMD:C_0805_2012Metric, F.Cu at (198.1, -11.6)
- added C1007: 100n, Capacitor_SMD:C_0805_2012Metric, F.Cu at (202.5, -26.6)
- added C1008: 100n, Capacitor_SMD:C_0805_2012Metric, F.Cu at (202.5, -23.6)
- added C1009: 100n, Capacitor_SMD:C_0805_2012Metric, F.Cu at (202.5, -20.6)
- added C1010: 100n, Capacitor_SMD:C_0805_2012Metric, F.Cu at (202.5, -17.6)
- added C1011: 1u, Capacitor_SMD:C_0805_2012Metric, F.Cu at (202.5, -14.6)
- added C1012: 100n, Capacitor_SMD:C_0805_2012Metric, F.Cu at (202.5, -11.6)
- added C1013: 100n, Capacitor_SMD:C_0805_2012Metric, F.Cu at (207.0, -26.6)
- added C1014: ~, Capacitor_SMD:C_0805_2012Metric, F.Cu at (207.0, -23.6)
- added C1015: ~, Capacitor_SMD:C_0805_2012Metric, F.Cu at (207.0, -20.6)
- added C1016: ~, Capacitor_SMD:C_0805_2012Metric, F.Cu at (207.0, -17.6)
- added C1017: 100n, Capacitor_SMD:C_0805_2012Metric, F.Cu at (207.0, -14.6)
- added C1018: ~, Capacitor_SMD:C_0805_2012Metric, F.Cu at (207.0, -11.6)
- added C1019: 15p, Capacitor_SMD:C_0805_2012Metric, F.Cu at (211.4, -26.6)
- added C1020: 15p, Capacitor_SMD:C_0805_2012Metric, F.Cu at (211.4, -23.6)
- added C1021: ~, Capacitor_SMD:C_0805_2012Metric, F.Cu at (211.4, -20.6)
- added C1022: 100n, Capacitor_SMD:C_0805_2012Metric, F.Cu at (211.4, -17.6)
- added C1023: 100n, Capacitor_SMD:C_0805_2012Metric, F.Cu at (211.4, -14.6)
- added C1101: 100n, Capacitor_SMD:C_0805_2012Metric, F.Cu at (240.1, -26.6)
- added C1102: 100n, Capacitor_SMD:C_0805_2012Metric, F.Cu at (240.1, -23.6)
- added C1201: 1u, Capacitor_SMD:C_0805_2012Metric, F.Cu at (247.6, -134.9)
- added C1202: 1u, Capacitor_SMD:C_0805_2012Metric, F.Cu at (247.6, -131.9)
- added C1203: 100n, Capacitor_SMD:C_0805_2012Metric, F.Cu at (247.6, -128.9)
- added C1204: 100n, Capacitor_SMD:C_0805_2012Metric, F.Cu at (247.6, -125.9)
- added C1301: 100n, Capacitor_SMD:C_0805_2012Metric, F.Cu at (157.4, -12.7)
- added C1302: 100n, Capacitor_SMD:C_0805_2012Metric, F.Cu at (157.4, -9.65)
- added C1303: 1n / 2 kV, Capacitor_SMD:C_1206_3216Metric, F.Cu at (162.5, -12.5)
- added C1401: 10u, Capacitor_SMD:C_0805_2012Metric, F.Cu at (194.3, -113.6)
- added C1402: 10u, Capacitor_SMD:C_0805_2012Metric, F.Cu at (194.3, -110.6)
- added C1403: 100n, Capacitor_SMD:C_0402_1005Metric, F.Cu at (218.5, -116.0)
- added C1404: 68n, Capacitor_SMD:C_0402_1005Metric, F.Cu at (218.5, -114.0)
- added C1405: 100n, Capacitor_SMD:C_0402_1005Metric, F.Cu at (218.5, -112.1)
- added C1406: 150p, Capacitor_SMD:C_0402_1005Metric, F.Cu at (218.5, -110.1)
- added C1407: 470u, Capacitor_SMD:CP_Elec_6.3x7.7, F.Cu at (207.3, -121.1)
- added C1408: 100n, Capacitor_SMD:C_0402_1005Metric, F.Cu at (218.5, -108.1)
- added C1409: 100n, Capacitor_SMD:C_0402_1005Metric, F.Cu at (218.5, -106.1)
- added C1410: 33p, Capacitor_SMD:C_0402_1005Metric, F.Cu at (218.5, -104.2)
- added C1411: 10u, Capacitor_SMD:C_0805_2012Metric, F.Cu at (194.3, -107.6)
- added C701: 10u, Capacitor_SMD:C_0805_2012Metric, F.Cu at (117.2, -33.5)
- added C702: 10u, Capacitor_SMD:C_0805_2012Metric, F.Cu at (117.2, -30.5)
- added C703: 1u, Capacitor_SMD:C_0805_2012Metric, F.Cu at (117.2, -27.4)
- added C704: 47n, Capacitor_SMD:C_0805_2012Metric, F.Cu at (117.2, -24.4)
- added C705: 470n, Capacitor_SMD:C_0805_2012Metric, F.Cu at (117.2, -21.4)
- added C706: 470n, Capacitor_SMD:C_0805_2012Metric, F.Cu at (117.2, -18.4)
- added C707: 10u, Capacitor_SMD:C_0805_2012Metric, F.Cu at (117.2, -15.4)
- added C708: 100n, Capacitor_SMD:C_0805_2012Metric, F.Cu at (121.7, -33.5)
- added C709: 22u, Capacitor_SMD:C_0805_2012Metric, F.Cu at (121.7, -30.5)
- added C710: 22n, Capacitor_SMD:C_0805_2012Metric, F.Cu at (121.7, -27.4)
- added C711: 22u, Capacitor_SMD:C_0805_2012Metric, F.Cu at (121.7, -24.4)
- added C712: 33p, Capacitor_SMD:C_0805_2012Metric, F.Cu at (121.7, -21.4)
- added C713: 22u, Capacitor_SMD:C_0805_2012Metric, F.Cu at (121.7, -18.4)
- added C714: 22u, Capacitor_SMD:C_0805_2012Metric, F.Cu at (121.7, -15.4)
- added C715: 22u, Capacitor_SMD:C_0805_2012Metric, F.Cu at (126.1, -33.5)
- added C716: 10p, Capacitor_SMD:C_0805_2012Metric, F.Cu at (126.1, -30.5)
- added C717: 1u, Capacitor_SMD:C_0805_2012Metric, F.Cu at (126.1, -27.4)
- added C718: 10n, Capacitor_SMD:C_0805_2012Metric, F.Cu at (126.1, -24.4)
- added C719: 1u, Capacitor_SMD:C_0805_2012Metric, F.Cu at (126.1, -21.4)
- added C720: 1u, Capacitor_SMD:C_0805_2012Metric, F.Cu at (126.1, -18.4)
- added C721: 1u, Capacitor_SMD:C_0805_2012Metric, F.Cu at (126.1, -15.4)
- added C801: 10u, Capacitor_SMD:C_0805_2012Metric, F.Cu at (117.2, -112.8)
- added C802: 2u2, Capacitor_SMD:C_0805_2012Metric, F.Cu at (117.2, -109.8)
- added C803: 2u2, Capacitor_SMD:C_0805_2012Metric, F.Cu at (117.2, -106.8)
- added C804: 47n, Capacitor_SMD:C_0805_2012Metric, F.Cu at (117.2, -103.8)
- added C805: 10u, Capacitor_SMD:C_0805_2012Metric, F.Cu at (117.2, -100.8)
- added C806: 100n, Capacitor_SMD:C_0805_2012Metric, F.Cu at (117.2, -97.7)
- added C807: 100n, Capacitor_SMD:C_0805_2012Metric, F.Cu at (117.2, -94.7)
- added C808: 4u7, Capacitor_SMD:C_0805_2012Metric, F.Cu at (117.2, -91.7)
- added C901: 1u, Capacitor_SMD:C_0805_2012Metric, F.Cu at (231.7, -56.6)
- added C902: 1u, Capacitor_SMD:C_0805_2012Metric, F.Cu at (231.7, -53.6)
- added C903: 100n, Capacitor_SMD:C_0805_2012Metric, F.Cu at (146.5, -54.5)
- added D1403: STPS3L60U, Diode_SMD:D_SMB, F.Cu at (206.3, -105.8)
- added H1401: MountingHole, Wuerth:9774025151R, F.Cu at (197.1, -120.1)
- added H901: MountingHole, Wuerth:9774025151R, F.Cu at (230.1, -83.2)
- added H902: MountingHole, Wuerth:9774025151R, F.Cu at (230.1, -73.1)
- added H903: MountingHole, Wuerth:9774025151R, F.Cu at (124.4, -55.5)
- added H904: MountingHole, Wuerth:9774025151R, F.Cu at (124.4, -45.5)
- added IC1001: MIC5317-3.3xM5, Package_TO_SOT_SMD:SOT-23-5, F.Cu at (198.4, -1.56)
- added IC1002: TXU0102, Package_SO:VSSOP-8_2.3x2mm_P0.5mm, F.Cu at (207.8, 0.19)
- added IC1003: CC2530F128RHAR, Package_DFN_QFN:VQFN-40-1EP_6x6mm_P0.5mm_EP3.5x3.5mm_ThermalVias, F.Cu at (209.5, -5.91)
- added IC1101: TUSB320, Package_DFN_QFN:Texas_X2QFN-12_1.6x1.6mm_P0.4mm, F.Cu at (239.8, -20.2)
- added IC1102: ATECC608B-SSHDA, Package_SO:SOIC-8_3.9x4.9mm_P1.27mm, F.Cu at (236.8, -14.8)
- added IC1201: MIC5317-3.3xM5, Package_TO_SOT_SMD:SOT-23-5, F.Cu at (244.8, -114.3)
- added IC1202: TXU0102, Package_SO:VSSOP-8_2.3x2mm_P0.5mm, F.Cu at (235.8, -108.7)
- added IC1402: ST1S14PHR, Package_SO:HSOP-8-1EP_3.9x4.9mm_P1.27mm_EP2.41x3.1mm, F.Cu at (216.8, -121.8)
- added IC701: LM62460, Package_QFN:RPH0016A, F.Cu at (117.5, -1.75)
- added IC702: ADP1614ACPZ-R7, Texas Instruments:LFCSP-10, F.Cu at (122.7, -2.42)
- added IC703: TPS2121RUXT, Texas Instruments:RUX0012A, F.Cu at (147.2, -3.44)
- added IC704: MIC5317-3.3xM5, Package_TO_SOT_SMD:SOT-23-5, F.Cu at (144.2, -32.6)
- added IC705: MIC5317-1.8xM5, Package_TO_SOT_SMD:SOT-23-5, F.Cu at (144.2, -27.9)
- added IC801: BQ25308, Package_DFN_QFN:WQFN-16-1EP_3x3mm_P0.5mm_EP1.68x1.68mm, F.Cu at (129.9, -93.9)
- added IC802: MAX17048, Package_DFN_QFN:TDFN-8-1EP_2x2mm_P0.5mm_EP0.8x1.2mm, F.Cu at (138.6, -112.4)
- added IC803: BQ297xy, Package_SON:WSON-6_1.5x1.5mm_P0.5mm, F.Cu at (138.2, -108.9)
- added IC901: MIC5317-3.3xM5, Package_TO_SOT_SMD:SOT-23-5, F.Cu at (227.7, -46.9)
- added JP901: Recovery, Connector_PinHeader_2.54mm:PinHeader_2x01_P2.54mm_Vertical, F.Cu at (146.6, -58.3)
- added L1401: 10u, Inductor_SMD:L_Wuerth_HCI-7050, F.Cu at (206.8, -112.8)
- added L701: 4u7, Inductor_SMD:L_Coilcraft_XAL5030-XXX, F.Cu at (145.1, -22.1)
- added L702: 2u2, Inductor_SMD:L_Wuerth_WE-PD-Typ-7345, F.Cu at (145.4, -9.89)
- added L801: 2u2, Inductor_SMD:L_Wuerth_WE-PD-Typ-7345, F.Cu at (131.7, -109.9)
- added LED1001: Zigbee, LED_SMD:LED_0805_2012Metric, F.Cu at (215.9, -12.2)
- added LED1201: wm-Bus, LED_SMD:LED_0805_2012Metric, F.Cu at (247.6, -122.8)
- added LED1401: Power Good, LED_SMD:LED_0805_2012Metric, F.Cu at (194.3, -104.5)
- added LED901: LoRa, LED_SMD:LED_0805_2012Metric, F.Cu at (232.3, -43.1)
- added M1201: iM891A-XL, IMST:iM891A-XL, F.Cu at (236.4, -126.5)
- added MP1001: ~, Bivar:SLP3-300-100-F, F.Cu at (216.5, -23.7)
- added MP1201: ~, Bivar:SLP3-300-100-F, F.Cu at (230.2, -112.2)
- added MP1401: ~, Bivar:SLP3-300-100-F, F.Cu at (214.3, -112.5)
- added MP901: ~, Bivar:SLP3-300-100-F, F.Cu at (227.9, -63.7)
- added Q1001: BSS123, Package_TO_SOT_SMD:SOT-23, F.Cu at (216.1, -15.9)
- added Q1201: BSS123, Package_TO_SOT_SMD:SOT-23, F.Cu at (244.6, -109.9)
- added Q701: BSS123, Package_TO_SOT_SMD:SOT-23, F.Cu at (143.1, -3.25)
- added Q801: Si2342DS, Package_TO_SOT_SMD:SOT-23, F.Cu at (129.4, -103.2)
- added Q802: Si2342DS, Package_TO_SOT_SMD:SOT-23, F.Cu at (129.4, -98.8)
- added Q901: BSS123, Package_TO_SOT_SMD:SOT-23, F.Cu at (227.6, -42.4)
- added R1001: 10k, Resistor_SMD:R_0805_2012Metric, F.Cu at (193.7, -26.6)
- added R1002: 0R, Resistor_SMD:R_0805_2012Metric, F.Cu at (193.7, -23.7)
- added R1003: 0R, Resistor_SMD:R_0805_2012Metric, F.Cu at (193.7, -20.7)
- added R1004: 10k, Resistor_SMD:R_0805_2012Metric, F.Cu at (193.7, -17.8)
- added R1005: 68R, Resistor_SMD:R_0402_1005Metric, F.Cu at (219.6, -12.7)
- added R1006: 0R, Resistor_SMD:R_0805_2012Metric, F.Cu at (193.7, -14.8)
- added R1007: 0R, Resistor_SMD:R_0805_2012Metric, F.Cu at (193.7, -11.9)
- added R1008: 10k, Resistor_SMD:R_0805_2012Metric, F.Cu at (193.7, -8.95)
- added R1009: 56k, Resistor_SMD:R_0805_2012Metric, F.Cu at (193.7, -6.00)
- added R1101: 1k, Resistor_SMD:R_0805_2012Metric, F.Cu at (243.3, -16.7)
- added R1102: 10k, Resistor_SMD:R_0805_2012Metric, F.Cu at (243.3, -13.7)
- added R1201: 10k, Resistor_SMD:R_0805_2012Metric, F.Cu at (225.2, -134.9)
- added R1202: 68R, Resistor_SMD:R_0402_1005Metric, F.Cu at (246.8, -120.3)
- added R1203: 0R, Resistor_SMD:R_0805_2012Metric, F.Cu at (225.2, -132.0)
- added R1204: 0R, Resistor_SMD:R_0805_2012Metric, F.Cu at (225.2, -129.0)
- added R1205: 10k, Resistor_SMD:R_0805_2012Metric, F.Cu at (225.2, -126.1)
- added R1206: 0R, Resistor_SMD:R_0805_2012Metric, F.Cu at (225.2, -123.1)
- added R1207: 0R, Resistor_SMD:R_0805_2012Metric, F.Cu at (225.2, -120.2)
- added R1208: 10k, Resistor_SMD:R_0805_2012Metric, F.Cu at (225.2, -117.2)
- added R1301: 470R, Resistor_SMD:R_0402_1005Metric, F.Cu at (172.4, -13.2)
- added R1302: 470R, Resistor_SMD:R_0402_1005Metric, F.Cu at (172.4, -11.2)
- added R1303: 1M, Resistor_SMD:R_1206_3216Metric, F.Cu at (168.1, -12.5)
- added R1401: 100k, Resistor_SMD:R_0402_1005Metric, F.Cu at (198.0, -114.1)
- added R1402: 100k, Resistor_SMD:R_0402_1005Metric, F.Cu at (198.0, -112.1)
- added R1403: 150R, Resistor_SMD:R_0402_1005Metric, F.Cu at (198.0, -110.1)
- added R1404: 82k5, Resistor_SMD:R_0402_1005Metric, F.Cu at (198.0, -108.1)
- added R1405: 48k7, Resistor_SMD:R_0402_1005Metric, F.Cu at (198.0, -106.1)
- added R1406: 4k7, Resistor_SMD:R_0805_2012Metric, F.Cu at (198.0, -104.1)
- added R701: 10k, Resistor_SMD:R_0805_2012Metric, F.Cu at (130.6, -33.5)
- added R702: 0R, Resistor_SMD:R_0805_2012Metric, F.Cu at (130.6, -30.5)
- added R703: 2k, Resistor_SMD:R_0805_2012Metric, F.Cu at (130.6, -27.6)
- added R704: 30k9, Resistor_SMD:R_0805_2012Metric, F.Cu at (130.6, -24.6)
- added R705: 10k, Resistor_SMD:R_0805_2012Metric, F.Cu at (130.6, -21.7)
- added R706: 100k, Resistor_SMD:R_0805_2012Metric, F.Cu at (130.6, -18.7)
- added R707: 24k9, Resistor_SMD:R_0805_2012Metric, F.Cu at (130.6, -15.8)
- added R708: 4k99, Resistor_SMD:R_0805_2012Metric, F.Cu at (135.0, -33.5)
- added R709: 21k, Resistor_SMD:R_0805_2012Metric, F.Cu at (135.0, -30.5)
- added R710: 5k1, Resistor_SMD:R_0805_2012Metric, F.Cu at (135.0, -27.6)
- added R711: 21k, Resistor_SMD:R_0805_2012Metric, F.Cu at (135.0, -24.6)
- added R712: 5k1, Resistor_SMD:R_0805_2012Metric, F.Cu at (135.0, -21.7)
- added R713: 10k, Resistor_SMD:R_0805_2012Metric, F.Cu at (135.0, -18.7)
- added R714: 51k1, Resistor_SMD:R_0805_2012Metric, F.Cu at (135.0, -15.8)
- added R715: 10k, Resistor_SMD:R_0805_2012Metric, F.Cu at (139.4, -33.5)
- added R716: 10k, Resistor_SMD:R_0805_2012Metric, F.Cu at (139.4, -30.5)
- added R717: 10k, Resistor_SMD:R_0805_2012Metric, F.Cu at (139.4, -27.6)
- added R718: 0R, Resistor_SMD:R_0805_2012Metric, F.Cu at (139.4, -24.6)
- added R801: 100k, Resistor_SMD:R_0402_1005Metric, F.Cu at (133.3, -104.5)
- added R802: 0R, Resistor_SMD:R_0805_2012Metric, F.Cu at (121.7, -112.8)
- added R803: 18k, Resistor_SMD:R_0805_2012Metric, F.Cu at (121.7, -109.9)
- added R804: 100k, Resistor_SMD:R_0402_1005Metric, F.Cu at (133.3, -102.5)
- added R805: 4k53, Resistor_SMD:R_0805_2012Metric, F.Cu at (121.7, -106.9)
- added R806: 22k6, Resistor_SMD:R_0805_2012Metric, F.Cu at (121.7, -104.0)
- added R807: 2k2, Resistor_SMD:R_0805_2012Metric, F.Cu at (121.7, -101.0)
- added R808: 100k, Resistor_SMD:R_0402_1005Metric, F.Cu at (133.3, -100.5)
- added R809: 330R, Resistor_SMD:R_0805_2012Metric, F.Cu at (121.7, -98.1)
- added R901: 10k, Resistor_SMD:R_0805_2012Metric, F.Cu at (227.3, -56.6)
- added R902: 68R, Resistor_SMD:R_0402_1005Metric, F.Cu at (226.6, -39.2)
- added R903: 10k, Resistor_SMD:R_0805_2012Metric, F.Cu at (227.3, -53.7)
- added R904: 10k, Resistor_SMD:R_0805_2012Metric, F.Cu at (227.3, -50.7)
- added R905: 10k, Resistor_SMD:R_0805_2012Metric, F.Cu at (117.2, -59.1)
- added R906: 10k, Resistor_SMD:R_0805_2012Metric, F.Cu at (117.2, -56.1)
- added R907: 10k, Resistor_SMD:R_0805_2012Metric, F.Cu at (117.2, -53.2)
- added R908: 10k, Resistor_SMD:R_0805_2012Metric, F.Cu at (117.2, -50.2)
- added R909: 1k, Resistor_SMD:R_0805_2012Metric, F.Cu at (117.2, -47.3)
- added R910: ~, Resistor_SMD:R_0805_2012Metric, F.Cu at (117.2, -44.3)
- added R911: ~, Resistor_SMD:R_0805_2012Metric, F.Cu at (117.2, -41.4)
- added R912: ~, Resistor_SMD:R_0805_2012Metric, F.Cu at (117.2, -38.4)
- added SW901: Reset, Same Sky:TS11, F.Cu at (134.6, -57.0)
- added SW902: On / Off, Same Sky:TS11, F.Cu at (134.6, -47.5)
- added TH801: 10k, Resistor_SMD:R_0805_2012Metric, F.Cu at (121.7, -95.1)
- added TP1001: ~, Testpoints_Kampi:TestPoint_Pad_1.0x1.0mm, F.Cu at (197.4, -8.54)
- added TP1002: ~, Testpoints_Kampi:TestPoint_Pad_1.0x1.0mm, F.Cu at (197.4, -5.49)
- added TP1003: ~, Testpoints_Kampi:TestPoint_Pad_1.0x1.0mm, F.Cu at (200.4, -8.54)
- added TP1004: ~, Testpoints_Kampi:TestPoint_Pad_1.0x1.0mm, F.Cu at (200.4, -5.49)
- added TP1005: ~, Testpoints_Kampi:TestPoint_Pad_1.0x1.0mm, F.Cu at (203.5, -8.54)
- added TP1006: ~, Testpoints_Kampi:TestPoint_Pad_1.0x1.0mm, F.Cu at (203.5, -5.49)
- added TP1101: ~, Testpoints_Kampi:TestPoint_Pad_1.0x1.0mm, F.Cu at (243.3, -20.6)
- added TP1201: ~, Testpoints_Kampi:TestPoint_Pad_1.0x1.0mm, F.Cu at (234.6, -115.2)
- added TP1202: ~, Testpoints_Kampi:TestPoint_Pad_1.0x1.0mm, F.Cu at (234.6, -112.1)
- added TP1203: ~, Testpoints_Kampi:TestPoint_Pad_1.0x1.0mm, F.Cu at (237.6, -115.2)
- added TP1204: ~, Testpoints_Kampi:TestPoint_Pad_1.0x1.0mm, F.Cu at (237.6, -112.1)
- added TP1205: ~, Testpoints_Kampi:TestPoint_Pad_1.0x1.0mm, F.Cu at (240.7, -115.2)
- added TP1206: ~, Testpoints_Kampi:TestPoint_Pad_1.0x1.0mm, F.Cu at (240.7, -112.1)
- added TP1301: ~, Testpoints_Kampi:TestPoint_Pad_1.0x1.0mm, F.Cu at (153.7, -12.6)
- added TP1302: ~, Testpoints_Kampi:TestPoint_Pad_1.0x1.0mm, F.Cu at (153.7, -9.60)
- added TP1401: ~, Testpoints_Kampi:TestPoint_Pad_1.0x1.0mm, F.Cu at (217.1, -134.9)
- added TP1402: ~, Testpoints_Kampi:TestPoint_Pad_1.0x1.0mm, F.Cu at (217.1, -131.8)
- added TP1403: ~, Testpoints_Kampi:TestPoint_Pad_1.0x1.0mm, F.Cu at (217.1, -128.8)
- added TP701: ~, Testpoints_Kampi:TestPoint_Pad_1.0x1.0mm, F.Cu at (116.5, -12.4)
- added TP702: ~, Testpoints_Kampi:TestPoint_Pad_1.0x1.0mm, F.Cu at (116.5, -9.32)
- added TP703: ~, Testpoints_Kampi:TestPoint_Pad_1.0x1.0mm, F.Cu at (116.5, -6.28)
- added TP704: ~, Testpoints_Kampi:TestPoint_Pad_1.0x1.0mm, F.Cu at (119.6, -12.4)
- added TP705: ~, Testpoints_Kampi:TestPoint_Pad_1.0x1.0mm, F.Cu at (119.6, -9.32)
- added TP706: ~, Testpoints_Kampi:TestPoint_Pad_1.0x1.0mm, F.Cu at (119.6, -6.28)
- added TP707: ~, Testpoints_Kampi:TestPoint_Pad_1.0x1.0mm, F.Cu at (122.6, -12.4)
- added TP708: ~, Testpoints_Kampi:TestPoint_Pad_1.0x1.0mm, F.Cu at (122.6, -9.32)
- added TP709: ~, Testpoints_Kampi:TestPoint_Pad_1.0x1.0mm, F.Cu at (122.6, -6.28)
- added TP710: ~, Testpoints_Kampi:TestPoint_Pad_1.0x1.0mm, F.Cu at (125.7, -12.4)
- added TP711: ~, Testpoints_Kampi:TestPoint_Pad_1.0x1.0mm, F.Cu at (125.7, -9.32)
- added TP712: ~, Testpoints_Kampi:TestPoint_Pad_1.0x1.0mm, F.Cu at (125.7, -6.28)
- added TP801: ~, Testpoints_Kampi:TestPoint_Pad_1.0x1.0mm, F.Cu at (125.4, -112.8)
- added TP802: ~, Testpoints_Kampi:TestPoint_Pad_1.0x1.0mm, F.Cu at (125.4, -109.7)
- added TP803: ~, Testpoints_Kampi:TestPoint_Pad_1.0x1.0mm, F.Cu at (125.4, -106.7)
- added TP804: ~, Testpoints_Kampi:TestPoint_Pad_1.0x1.0mm, F.Cu at (125.4, -103.6)
- added TP805: ~, Testpoints_Kampi:TestPoint_Pad_1.0x1.0mm, F.Cu at (125.4, -100.6)
- added TP901: ~, Testpoints_Kampi:TestPoint_Pad_1.0x1.0mm, F.Cu at (232.2, -66.6)
- added TP902: ~, Testpoints_Kampi:TestPoint_Pad_1.0x1.0mm, F.Cu at (232.2, -63.5)
- added TP903: ~, Testpoints_Kampi:TestPoint_Pad_1.0x1.0mm, F.Cu at (232.2, -60.5)
- added TP904: ~, Testpoints_Kampi:TestPoint_Pad_1.0x1.0mm, F.Cu at (145.8, -51.4)
- added X1001: Zigbee, Amphenol:A-1JB, F.Cu at (216.6, -2.11)
- added X1101: OTG, Connector_USB:USB_C_Receptacle_GCT_USB4110, F.Cu at (230.7, -22.8)
- added X1103: I2C, Connector_PinHeader_2.54mm:PinHeader_1x02_P2.54mm_Vertical, F.Cu at (225.7, -15.8)
- added X1104: I2C, Connector_PinHeader_2.54mm:PinHeader_1x02_P2.54mm_Vertical, F.Cu at (230.3, -15.8)
- added X1301: Ethernet, Connector_RJ:RJ45_Pulse_JK00177NL_Horizontal, F.Cu at (160.0, -29.6)
- added X1401: SSD, Amphenol:MDT420M03001, F.Cu at (203.8, -128.9)
- added X701: 7-16 V, Connector_BarrelJack:BarrelJack_Wuerth_6941xx301002, F.Cu at (133.9, -12.4)
- added X901: SoM, TE:2309409-2, F.Cu at (152.2, -74.4)
- added X902: UART, Connector_PinHeader_2.54mm:PinHeader_1x03_P2.54mm_Vertical, F.Cu at (142.0, -58.3)
- added X903: LoRa, Connector_PCBEdge:BUS_PCI_Express_Mini_Full, F.Cu at (208.3, -36.2)
- added Y1001: 32MHz, Crystal:Crystal_SMD_Abracon_ABM7-2Pin_6.0x3.5mm, F.Cu at (217.6, -7.54)

Commit message: Adding level shifter, update documentation
Parts:
- removed BAT801: Backup Power, Keystone:1043
- removed C1001, C1002, C1011, C1201, C1202, C703, C717, C719, C720, C721, C901, C902: 1u, Capacitor_SMD:C_0805_2012Metric
- removed C1003, C1004, C1007, C1008, C1009, C1010, C1012, C1013, C1017, C1022, C1023, C1101, C1102, C1203, C1204, C1301, C1302, C708, C806, C807, C903: 100n, Capacitor_SMD:C_0805_2012Metric
- removed C1005, C1006: 27p, Capacitor_SMD:C_0805_2012Metric
- removed C1014, C1015, C1016, C1018, C1021: ~, Capacitor_SMD:C_0805_2012Metric
- removed C1019, C1020: 15p, Capacitor_SMD:C_0805_2012Metric
- removed C1303: 1n / 2 kV, Capacitor_SMD:C_1206_3216Metric
- removed C1401, C1402, C1411, C701, C702, C707, C801, C805: 10u, Capacitor_SMD:C_0805_2012Metric
- removed C1403, C1405, C1408, C1409: 100n, Capacitor_SMD:C_0402_1005Metric
- removed C1404: 68n, Capacitor_SMD:C_0402_1005Metric
- removed C1406: 150p, Capacitor_SMD:C_0402_1005Metric
- removed C1407: 470u, Capacitor_SMD:CP_Elec_6.3x7.7
- removed C1410: 33p, Capacitor_SMD:C_0402_1005Metric
- removed C704, C804: 47n, Capacitor_SMD:C_0805_2012Metric
- removed C705, C706: 470n, Capacitor_SMD:C_0805_2012Metric
- removed C709, C711, C713, C714, C715: 22u, Capacitor_SMD:C_0805_2012Metric
- removed C710: 22n, Capacitor_SMD:C_0805_2012Metric
- removed C712: 33p, Capacitor_SMD:C_0805_2012Metric
- removed C716: 10p, Capacitor_SMD:C_0805_2012Metric
- removed C718: 10n, Capacitor_SMD:C_0805_2012Metric
- removed C802, C803: 2u2, Capacitor_SMD:C_0805_2012Metric
- removed C808: 4u7, Capacitor_SMD:C_0805_2012Metric
- removed D1403: STPS3L60U, Diode_SMD:D_SMB
- removed H1401, H901, H902, H903, H904: MountingHole, Wuerth:9774025151R
- removed IC1001, IC1201, IC704, IC901: MIC5317-3.3xM5, Package_TO_SOT_SMD:SOT-23-5
- removed IC1002, IC1202: TXU0102, Package_SO:VSSOP-8_2.3x2mm_P0.5mm
- removed IC1003: CC2530F128RHAR, Package_DFN_QFN:VQFN-40-1EP_6x6mm_P0.5mm_EP3.5x3.5mm_ThermalVias
- removed IC1101: TUSB320, Package_DFN_QFN:Texas_X2QFN-12_1.6x1.6mm_P0.4mm
- removed IC1102: ATECC608B-SSHDA, Package_SO:SOIC-8_3.9x4.9mm_P1.27mm
- removed IC1402: ST1S14PHR, Package_SO:HSOP-8-1EP_3.9x4.9mm_P1.27mm_EP2.41x3.1mm
- removed IC701: LM62460, Package_QFN:RPH0016A
- removed IC702: ADP1614ACPZ-R7, Texas Instruments:LFCSP-10
- removed IC703: TPS2121RUXT, Texas Instruments:RUX0012A
- removed IC705: MIC5317-1.8xM5, Package_TO_SOT_SMD:SOT-23-5
- removed IC801: BQ25308, Package_DFN_QFN:WQFN-16-1EP_3x3mm_P0.5mm_EP1.68x1.68mm
- removed IC802: MAX17048, Package_DFN_QFN:TDFN-8-1EP_2x2mm_P0.5mm_EP0.8x1.2mm
- removed IC803: BQ297xy, Package_SON:WSON-6_1.5x1.5mm_P0.5mm
- removed JP901: Recovery, Connector_PinHeader_2.54mm:PinHeader_2x01_P2.54mm_Vertical
- removed L1401: 10u, Inductor_SMD:L_Wuerth_HCI-7050
- removed L701: 4u7, Inductor_SMD:L_Coilcraft_XAL5030-XXX
- removed L702, L801: 2u2, Inductor_SMD:L_Wuerth_WE-PD-Typ-7345
- removed LED1001: Zigbee, LED_SMD:LED_0805_2012Metric
- removed LED1201: wm-Bus, LED_SMD:LED_0805_2012Metric
- removed LED1401: Power Good, LED_SMD:LED_0805_2012Metric
- removed LED901: LoRa, LED_SMD:LED_0805_2012Metric
- removed M1201: iM891A-XL, IMST:iM891A-XL
- removed MP1001, MP1201, MP1401, MP901: ~, Bivar:SLP3-300-100-F
- removed Q1001, Q1201, Q701, Q901: BSS123, Package_TO_SOT_SMD:SOT-23
- removed Q801, Q802: Si2342DS, Package_TO_SOT_SMD:SOT-23
- removed R1001, R1004, R1008, R1102, R1201, R1205, R1208, R701, R705, R713, R715, R716, R717, R901, R903, R904, R905, R906, R907, R908, TH801: 10k, Resistor_SMD:R_0805_2012Metric
- removed R1002, R1003, R1006, R1007, R1203, R1204, R1206, R1207, R702, R718, R802: 0R, Resistor_SMD:R_0805_2012Metric
- removed R1005, R1202, R902: 68R, Resistor_SMD:R_0402_1005Metric
- removed R1009: 56k, Resistor_SMD:R_0805_2012Metric
- removed R1101, R909: 1k, Resistor_SMD:R_0805_2012Metric
- removed R1301, R1302: 470R, Resistor_SMD:R_0402_1005Metric
- removed R1303: 1M, Resistor_SMD:R_1206_3216Metric
- removed R1401, R1402, R801, R804, R808: 100k, Resistor_SMD:R_0402_1005Metric
- removed R1403: 150R, Resistor_SMD:R_0402_1005Metric
- removed R1404: 82k5, Resistor_SMD:R_0402_1005Metric
- removed R1405: 48k7, Resistor_SMD:R_0402_1005Metric
- removed R1406: 4k7, Resistor_SMD:R_0805_2012Metric
- removed R703: 2k, Resistor_SMD:R_0805_2012Metric
- removed R704: 30k9, Resistor_SMD:R_0805_2012Metric
- removed R706: 100k, Resistor_SMD:R_0805_2012Metric
- removed R707: 24k9, Resistor_SMD:R_0805_2012Metric
- removed R708: 4k99, Resistor_SMD:R_0805_2012Metric
- removed R709, R711: 21k, Resistor_SMD:R_0805_2012Metric
- removed R710, R712: 5k1, Resistor_SMD:R_0805_2012Metric
- removed R714: 51k1, Resistor_SMD:R_0805_2012Metric
- removed R803: 18k, Resistor_SMD:R_0805_2012Metric
- removed R805: 4k53, Resistor_SMD:R_0805_2012Metric
- removed R806: 22k6, Resistor_SMD:R_0805_2012Metric
- removed R807: 2k2, Resistor_SMD:R_0805_2012Metric
- removed R809: 330R, Resistor_SMD:R_0805_2012Metric
- removed R910, R911, R912: ~, Resistor_SMD:R_0805_2012Metric
- removed SW901: Reset, Same Sky:TS11
- removed SW902: On / Off, Same Sky:TS11
- removed TP1001, TP1002, TP1003, TP1004, TP1005, TP1006, TP1101, TP1201, TP1202, TP1203, TP1204, TP1205, TP1206, TP1301, TP1302, TP1401, TP1402, TP1403, TP701, TP702, TP703, TP704, TP705, TP706, TP707, TP708, TP709, TP710, TP711, TP712, TP801, TP802, TP803, TP804, TP805, TP901, TP902, TP903, TP904: ~, Testpoints_Kampi:TestPoint_Pad_1.0x1.0mm
- removed X1001: Zigbee, Amphenol:A-1JB
- removed X1101: OTG, Connector_USB:USB_C_Receptacle_GCT_USB4110
- removed X1103, X1104: I2C, Connector_PinHeader_2.54mm:PinHeader_1x02_P2.54mm_Vertical
- removed X1301: Ethernet, Connector_RJ:RJ45_Pulse_JK00177NL_Horizontal
- removed X1401: SSD, Amphenol:MDT420M03001
- removed X701: 7-16 V, Connector_BarrelJack:BarrelJack_Wuerth_6941xx301002
- removed X901: SoM, TE:2309409-2
- removed X902: UART, Connector_PinHeader_2.54mm:PinHeader_1x03_P2.54mm_Vertical
- removed X903: LoRa, Connector_PCBEdge:BUS_PCI_Express_Mini_Full
- removed Y1001: 32MHz, Crystal:Crystal_SMD_Abracon_ABM7-2Pin_6.0x3.5mm
