File: gateway/Gateway.kicad_pcb (KiCad board)
At the start: 4 copper layers, 0 parts

Commit message: Improving Thread
- Add boot signal for Thread MCU
- Add debug LED for nRF5340
Parts:
- added BAT901: Backup Power, Keystone:1043, F.Cu at (216.0, 184.9)
- added C1001: 100n, Capacitor_SMD:C_0805_2012Metric, F.Cu at (218.7, 168.4)
- added C1101: 1u, Capacitor_SMD:C_0805_2012Metric, F.Cu at (173.0, 95.7)
- added C1102: 1u, Capacitor_SMD:C_0805_2012Metric, F.Cu at (173.0, 98.7)
- added C1201: 1u, Capacitor_SMD:C_0805_2012Metric, F.Cu at (158.5, 159.6)
- added C1202: 1u, Capacitor_SMD:C_0805_2012Metric, F.Cu at (158.5, 162.6)
- added C1203: 100n, Capacitor_SMD:C_0805_2012Metric, F.Cu at (158.5, 165.6)
- added C1204: 100n, Capacitor_SMD:C_0805_2012Metric, F.Cu at (158.5, 168.6)
- added C1205: 100n, Capacitor_SMD:C_0805_2012Metric, F.Cu at (158.5, 171.6)
- added C1206: 10u, Capacitor_SMD:C_0805_2012Metric, F.Cu at (158.5, 174.6)
- added C1301: 1u, Capacitor_SMD:C_0805_2012Metric, F.Cu at (257.1, 143.2)
- added C1302: 1u, Capacitor_SMD:C_0805_2012Metric, F.Cu at (257.1, 146.2)
- added C1303: 100n, Capacitor_SMD:C_0805_2012Metric, F.Cu at (257.1, 149.2)
- added C1304: 100n, Capacitor_SMD:C_0805_2012Metric, F.Cu at (257.1, 152.3)
- added C1401: 1u, Capacitor_SMD:C_0805_2012Metric, F.Cu at (280.3, 175.3)
- added C1402: 1u, Capacitor_SMD:C_0805_2012Metric, F.Cu at (280.3, 178.3)
- added C1403: 100n, Capacitor_SMD:C_0805_2012Metric, F.Cu at (280.3, 181.3)
- added C1404: 100n, Capacitor_SMD:C_0805_2012Metric, F.Cu at (280.3, 184.4)
- added C1501: 100n, Capacitor_SMD:C_0805_2012Metric, F.Cu at (209.4, 80.1)
- added C1502: 100n, Capacitor_SMD:C_0805_2012Metric, F.Cu at (209.4, 83.1)
- added C1503: 100n, Capacitor_SMD:C_0805_2012Metric, F.Cu at (209.4, 86.1)
- added C1504: 100n, Capacitor_SMD:C_0805_2012Metric, F.Cu at (209.4, 89.1)
- added C1505: 100n, Capacitor_SMD:C_0805_2012Metric, F.Cu at (209.4, 92.1)
- added C1506: 100n, Capacitor_SMD:C_0805_2012Metric, F.Cu at (213.9, 80.1)
- added C1507: 100n, Capacitor_SMD:C_0805_2012Metric, F.Cu at (213.9, 83.1)
- added C1508: 100n, Capacitor_SMD:C_0805_2012Metric, F.Cu at (213.9, 86.1)
- added C1509: 100n, Capacitor_SMD:C_0805_2012Metric, F.Cu at (213.9, 89.1)
- added C1510: 100n, Capacitor_SMD:C_0805_2012Metric, F.Cu at (213.9, 92.1)
- added C1601: 10u, Capacitor_SMD:C_0805_2012Metric, F.Cu at (134.9, 137.0)
- added C1602: 10u, Capacitor_SMD:C_0805_2012Metric, F.Cu at (134.9, 140.0)
- added C1603: 100n, Capacitor_SMD:C_0805_2012Metric, F.Cu at (134.9, 143.0)
- added C1604: 68n, Capacitor_SMD:C_0805_2012Metric, F.Cu at (134.9, 146.0)
- added C1605: 100n, Capacitor_SMD:C_0805_2012Metric, F.Cu at (134.9, 149.0)
- added C1606: 150p, Capacitor_SMD:C_0805_2012Metric, F.Cu at (139.4, 137.0)
- added C1607: 470u, Capacitor_SMD:CP_Elec_6.3x7.7, F.Cu at (151.2, 149.6)
- added C1608: 100n, Capacitor_SMD:C_0805_2012Metric, F.Cu at (139.4, 140.0)
- added C1609: 100n, Capacitor_SMD:C_0805_2012Metric, F.Cu at (139.4, 143.0)
- added C1610: 33p, Capacitor_SMD:C_0805_2012Metric, F.Cu at (139.4, 146.0)
- added C1611: 10u, Capacitor_SMD:C_0805_2012Metric, F.Cu at (139.4, 149.0)
- added C1701: 100n, Capacitor_SMD:C_0805_2012Metric, F.Cu at (138.0, 213.6)
- added C1702: 100n, Capacitor_SMD:C_0805_2012Metric, F.Cu at (138.0, 216.6)
- added C1703: 1n / 2 kV, Capacitor_SMD:C_1206_3216Metric, F.Cu at (147.4, 213.7)
- added C701: 100n, Capacitor_SMD:C_0805_2012Metric, F.Cu at (285.0, 82.2)
- added C801: 10u, Capacitor_SMD:C_0805_2012Metric, F.Cu at (250.7, 65.6)
- added C802: 10u, Capacitor_SMD:C_0805_2012Metric, F.Cu at (250.7, 68.6)
- added C803: 1u, Capacitor_SMD:C_0805_2012Metric, F.Cu at (250.7, 71.6)
- added C804: 47n, Capacitor_SMD:C_0805_2012Metric, F.Cu at (250.7, 74.6)
- added C805: 470n, Capacitor_SMD:C_0805_2012Metric, F.Cu at (250.7, 77.6)
- added C806: 470n, Capacitor_SMD:C_0805_2012Metric, F.Cu at (250.7, 80.7)
- added C807: 10u, Capacitor_SMD:C_0805_2012Metric, F.Cu at (255.2, 65.6)
- added C808: 100n, Capacitor_SMD:C_0805_2012Metric, F.Cu at (255.2, 68.6)
- added C809: 22u, Capacitor_SMD:C_0805_2012Metric, F.Cu at (255.2, 71.6)
- added C810: 22n, Capacitor_SMD:C_0805_2012Metric, F.Cu at (255.2, 74.6)
- added C811: 22u, Capacitor_SMD:C_0805_2012Metric, F.Cu at (255.2, 77.6)
- added C812: 33p, Capacitor_SMD:C_0805_2012Metric, F.Cu at (255.2, 80.7)
- added C813: 22u, Capacitor_SMD:C_0805_2012Metric, F.Cu at (259.6, 65.6)
- added C814: 22u, Capacitor_SMD:C_0805_2012Metric, F.Cu at (259.6, 68.6)
- added C815: 22u, Capacitor_SMD:C_0805_2012Metric, F.Cu at (259.6, 71.6)
- added C816: 10p, Capacitor_SMD:C_0805_2012Metric, F.Cu at (259.6, 74.6)
- added C817: 1u, Capacitor_SMD:C_0805_2012Metric, F.Cu at (259.6, 77.6)
- added C818: 10n, Capacitor_SMD:C_0805_2012Metric, F.Cu at (259.6, 80.7)
- added C819: 1u, Capacitor_SMD:C_0805_2012Metric, F.Cu at (264.1, 65.6)
- added C820: 1u, Capacitor_SMD:C_0805_2012Metric, F.Cu at (264.1, 68.6)
- added C821: 1u, Capacitor_SMD:C_0805_2012Metric, F.Cu at (264.1, 71.6)
- added C822: 10u, Capacitor_SMD:C_0805_2012Metric, F.Cu at (264.1, 74.6)
- added C823: 10u, Capacitor_SMD:C_0805_2012Metric, F.Cu at (264.1, 77.6)
- added C901: 10u, Capacitor_SMD:C_0805_2012Metric, F.Cu at (180.6, 197.4)
- added C902: 2u2, Capacitor_SMD:C_0805_2012Metric, F.Cu at (180.6, 200.4)
- added C903: 2u2, Capacitor_SMD:C_0805_2012Metric, F.Cu at (180.6, 203.4)
- added C904: 47n, Capacitor_SMD:C_0805_2012Metric, F.Cu at (180.6, 206.5)
- added C905: 10u, Capacitor_SMD:C_0805_2012Metric, F.Cu at (180.6, 209.5)
- added C906: 100n, Capacitor_SMD:C_0805_2012Metric, F.Cu at (180.6, 212.5)
- added C907: 100n, Capacitor_SMD:C_0805_2012Metric, F.Cu at (180.6, 215.5)
- added C908: 4u7, Capacitor_SMD:C_0805_2012Metric, F.Cu at (180.6, 218.5)
- added D1601: STPS3L60U, Diode_SMD:D_SMB, F.Cu at (136.9, 153.3)
- added D801: CMS05, Toshiba:M-FLAT-2, F.Cu at (243.7, 94.0)
- added H1001: MountingHole, Wuerth:9774015151R, F.Cu at (183.4, 156.7)
- added H1002: MountingHole, Wuerth:9774015151R, F.Cu at (183.4, 166.8)
- added H1101: MountingHole, Wuerth:9774015151R, F.Cu at (171.4, 69.1)
- added H1102: MountingHole, Wuerth:9774015151R, F.Cu at (171.4, 79.2)
- added H1601: MountingHole, Wuerth:9774015151R, F.Cu at (151.0, 140.5)
- added IC1101: MIC5317-3.3xM5, Package_TO_SOT_SMD:SOT-23-5, F.Cu at (168.9, 105.5)
- added IC1102: 74LVC1G07, Package_TO_SOT_SMD:SOT-353_SC-70-5, F.Cu at (168.3, 109.5)
- added IC1201: MIC5317-3.3xM5, Package_TO_SOT_SMD:SOT-23-5, F.Cu at (163.3, 170.5)
- added IC1202: TXB0102DCT, Package_SO:VSSOP-8_2.3x2mm_P0.5mm, F.Cu at (163.0, 184.2)
- added IC1203: 74LVC1G07, Package_TO_SOT_SMD:SOT-353_SC-70-5, F.Cu at (158.2, 184.1)
- added IC1204: 74LVC1G07, Package_TO_SOT_SMD:SOT-353_SC-70-5, F.Cu at (158.2, 187.6)
- added IC1301: MIC5317-3.3xM5, Package_TO_SOT_SMD:SOT-23-5, F.Cu at (261.9, 154.1)
- added IC1302: 74LVC1G07, Package_TO_SOT_SMD:SOT-353_SC-70-5, F.Cu at (280.6, 151.0)
- added IC1303: TXB0104PWR, Package_SO:TSSOP-14_4.4x5mm_P0.65mm, F.Cu at (273.9, 154.3)
- added IC1304: 74LVC1G07, Package_TO_SOT_SMD:SOT-353_SC-70-5, F.Cu at (280.6, 154.5)
- added IC1401: MIC5317-3.3xM5, Package_TO_SOT_SMD:SOT-23-5, F.Cu at (277.5, 195.9)
- added IC1402: 74LVC1G07, Package_TO_SOT_SMD:SOT-353_SC-70-5, F.Cu at (280.1, 187.7)
- added IC1403: TXB0102DCT, Package_SO:VSSOP-8_2.3x2mm_P0.5mm, F.Cu at (268.6, 201.6)
- added IC1501: ATECC608B-SSHDA, Package_SO:SOIC-8_3.9x4.9mm_P1.27mm, F.Cu at (226.1, 97.0)
- added IC1502: TUSB320, Package_DFN_QFN:Texas_X2QFN-12_1.6x1.6mm_P0.4mm, F.Cu at (214.7, 103.6)
- added IC1503: TXS0108EPW, Package_SO:TSSOP-20_4.4x6.5mm_P0.65mm, F.Cu at (217.5, 97.7)
- added IC1504: TXS0102DCU, Package_SO:VSSOP-8_2.3x2mm_P0.5mm, F.Cu at (210.0, 95.6)
- added IC1505: TXB0102DCU, Package_SO:VSSOP-8_2.3x2mm_P0.5mm, F.Cu at (210.0, 99.3)
- added IC1506: TXS0102DCU, Package_SO:VSSOP-8_2.3x2mm_P0.5mm, F.Cu at (210.0, 103.0)
- added IC1601: ST1S14PHR, Package_SO:HSOP-8-1EP_3.9x4.9mm_P1.27mm_EP2.41x3.1mm, F.Cu at (160.5, 127.6)
- added IC701: INA219AxD, Package_SO:SOIC-8_3.9x4.9mm_P1.27mm, F.Cu at (278.6, 84.0)
- added IC801: LM62460, Package_QFN:RPH0016A, F.Cu at (260.1, 94.0)
- added IC802: ADP1614ACPZ-650-R7, Texas Instruments:LFCSP-10, F.Cu at (265.3, 93.3)
- added IC803: TPS2121RUXT, Texas Instruments:RUX0012A, F.Cu at (250.2, 96.4)
- added IC804: MIC5317-3.3xM5, Package_TO_SOT_SMD:SOT-23-5, F.Cu at (237.8, 87.2)
- added IC805: MIC5317-1.8xM5, Package_TO_SOT_SMD:SOT-23-5, F.Cu at (237.8, 91.8)
- added IC901: BQ25308, Package_DFN_QFN:WQFN-16-1EP_3x3mm_P0.5mm_EP1.68x1.68mm, F.Cu at (197.8, 216.3)
- added IC902: MAX17048, Package_DFN_QFN:TDFN-8-1EP_2x2mm_P0.5mm_EP0.8x1.2mm, F.Cu at (201.8, 206.7)
- added IC903: BQ297xy, Package_SON:WSON-6_1.5x1.5mm_P0.5mm, F.Cu at (201.4, 210.2)
- added JP1001: Recovery, Connector_PinHeader_2.54mm:PinHeader_2x01_P2.54mm_Vertical, F.Cu at (218.8, 154.0)
- added L1601: 10u, Inductor_SMD:L_Wuerth_HCI-7050, F.Cu at (160.7, 139.7)
- added L801: 4u7, Inductor_SMD:L_Coilcraft_XAL5030-XXX, F.Cu at (243.9, 88.4)
- added L802: 2u2, Inductor_SMD:L_Wuerth_WE-PD-Typ-7345, F.Cu at (262.4, 86.6)
- added L901: 2u2, Inductor_SMD:L_Wuerth_WE-PD-Typ-7345, F.Cu at (199.5, 200.3)
- added LED1001: Ready, LED_SMD:LED_0805_2012Metric, F.Cu at (225.9, 153.2)
- added LED1101: LoRa, LED_SMD:LED_0805_2012Metric, F.Cu at (173.7, 104.6)
- added LED1201: Zigbee, LED_SMD:LED_0805_2012Metric, F.Cu at (163.0, 174.2)
- added LED1301: Thread, LED_SMD:LED_0805_2012Metric, F.Cu at (267.1, 152.9)
- added LED1302: Debug, LED_SMD:LED_0805_2012Metric, F.Cu at (267.1, 155.9)
- added LED1401: wM-Bus, LED_SMD:LED_0805_2012Metric, F.Cu at (277.2, 199.7)
- added LED1601: Power Good, LED_SMD:LED_0805_2012Metric, F.Cu at (158.5, 132.3)
- added M1201: RF-BM-2652, Rf-star:RF-BM-2652, F.Cu at (142.3, 173.6)
- added M1301: BT40, Fanstel:BT40E, F.Cu at (263.5, 132.9)
- added M1401: iM891A-XL, IMST:iM891A-XL, F.Cu at (269.2, 183.7)
- added MP1101: ~, Bivar:SLP3-300-100-F, F.Cu at (169.2, 88.7)
- added MP1201: ~, Bivar:SLP3-300-100-F, F.Cu at (163.5, 162.5)
- added MP1301: ~, Bivar:SLP3-300-100-F, F.Cu at (262.1, 146.2)
- added MP1401: ~, Bivar:SLP3-300-100-F, F.Cu at (263.0, 198.0)
- added MP1601: ~, Bivar:SLP3-300-100-F, F.Cu at (159.3, 150.0)
- added Q1001: BSS123, Package_TO_SOT_SMD:SOT-23, F.Cu at (219.0, 164.6)
- added Q801: BSS123, Package_TO_SOT_SMD:SOT-23, F.Cu at (237.7, 96.2)
- added Q901: Si2342DS, Package_TO_SOT_SMD:SOT-23, F.Cu at (197.2, 207.0)
- added Q902: Si2342DS, Package_TO_SOT_SMD:SOT-23, F.Cu at (197.2, 211.4)
- added R1001: 1k8, Resistor_SMD:R_0805_2012Metric, F.Cu at (200.9, 153.2)
- added R1002: 1k8, Resistor_SMD:R_0805_2012Metric, F.Cu at (200.9, 156.1)
- added R1003: 10k, Resistor_SMD:R_0805_2012Metric, F.Cu at (200.9, 159.1)
- added R1004: 10k, Resistor_SMD:R_0805_2012Metric, F.Cu at (200.9, 162.0)
- added R1005: 10k, Resistor_SMD:R_0805_2012Metric, F.Cu at (205.3, 153.2)
- added R1006: 1k8, Resistor_SMD:R_0805_2012Metric, F.Cu at (205.3, 156.1)
- added R1007: ~, Resistor_SMD:R_0805_2012Metric, F.Cu at (205.3, 159.1)
- added R1008: 10k, Resistor_SMD:R_0805_2012Metric, F.Cu at (205.3, 162.0)
- added R1009: ~, Resistor_SMD:R_0805_2012Metric, F.Cu at (209.7, 153.2)
- added R1010: 0R, Resistor_SMD:R_0805_2012Metric, F.Cu at (209.7, 156.1)
- added R1011: 10k, Resistor_SMD:R_0805_2012Metric, F.Cu at (209.7, 159.1)
- added R1012: 1k5, Resistor_SMD:R_0805_2012Metric, F.Cu at (209.7, 162.0)
- added R1101: 10k, Resistor_SMD:R_0805_2012Metric, F.Cu at (168.6, 95.7)
- added R1102: 68R, Resistor_SMD:R_0805_2012Metric, F.Cu at (168.6, 98.6)
- added R1103: 10k, Resistor_SMD:R_0805_2012Metric, F.Cu at (168.6, 101.6)
- added R1201: 10k, Resistor_SMD:R_0805_2012Metric, F.Cu at (154.1, 159.5)
- added R1202: 0R, Resistor_SMD:R_0805_2012Metric, F.Cu at (154.1, 162.5)
- added R1203: 0R, Resistor_SMD:R_0805_2012Metric, F.Cu at (154.1, 165.4)
- added R1204: 68R, Resistor_SMD:R_0805_2012Metric, F.Cu at (154.1, 168.4)
- added R1205: 0R, Resistor_SMD:R_0805_2012Metric, F.Cu at (154.1, 171.3)
- added R1206: 0R, Resistor_SMD:R_0805_2012Metric, F.Cu at (154.1, 174.3)
- added R1207: 10k, Resistor_SMD:R_0805_2012Metric, F.Cu at (154.1, 177.2)
- added R1208: 10k, Resistor_SMD:R_0805_2012Metric, F.Cu at (154.1, 180.2)
- added R1301: 10k, Resistor_SMD:R_0805_2012Metric, F.Cu at (274.3, 125.5)
- added R1302: 68R, Resistor_SMD:R_0805_2012Metric, F.Cu at (274.3, 128.5)
- added R1303: 10k, Resistor_SMD:R_0805_2012Metric, F.Cu at (274.3, 131.4)
- added R1304: 0R, Resistor_SMD:R_0805_2012Metric, F.Cu at (274.3, 134.4)
- added R1305: 0R, Resistor_SMD:R_0805_2012Metric, F.Cu at (274.3, 137.3)
- added R1306: 0R, Resistor_SMD:R_0805_2012Metric, F.Cu at (278.7, 125.5)
- added R1307: 0R, Resistor_SMD:R_0805_2012Metric, F.Cu at (278.7, 128.5)
- added R1308: 0R, Resistor_SMD:R_0805_2012Metric, F.Cu at (278.7, 131.4)
- added R1309: 0R, Resistor_SMD:R_0805_2012Metric, F.Cu at (278.7, 134.4)
- added R1310: 0R, Resistor_SMD:R_0805_2012Metric, F.Cu at (278.7, 137.3)
- added R1311: 0R, Resistor_SMD:R_0805_2012Metric, F.Cu at (283.1, 125.5)
- added R1312: 10k, Resistor_SMD:R_0805_2012Metric, F.Cu at (283.1, 128.5)
- added R1313: 68R, Resistor_SMD:R_0805_2012Metric, F.Cu at (283.1, 131.4)
- added R1401: 10k, Resistor_SMD:R_0805_2012Metric, F.Cu at (258.0, 175.3)
- added R1402: 68R, Resistor_SMD:R_0805_2012Metric, F.Cu at (258.0, 178.2)
- added R1403: 0R, Resistor_SMD:R_0805_2012Metric, F.Cu at (258.0, 181.2)
- added R1404: 0R, Resistor_SMD:R_0805_2012Metric, F.Cu at (258.0, 184.1)
- added R1405: 0R, Resistor_SMD:R_0805_2012Metric, F.Cu at (258.0, 187.1)
- added R1406: 0R, Resistor_SMD:R_0805_2012Metric, F.Cu at (258.0, 190.0)
- added R1407: 10k, Resistor_SMD:R_0805_2012Metric, F.Cu at (258.0, 193.0)
- added R1501: 887k, Resistor_SMD:R_0805_2012Metric, F.Cu at (205.0, 80.1)
- added R1503: 4k7, Resistor_SMD:R_0805_2012Metric, F.Cu at (205.0, 83.0)
- added R1504: 3k3, Resistor_SMD:R_0805_2012Metric, F.Cu at (205.0, 86.0)
- added R1505: 3k3, Resistor_SMD:R_0805_2012Metric, F.Cu at (205.0, 88.9)
- added R1506: 3k3, Resistor_SMD:R_0805_2012Metric, F.Cu at (205.0, 91.9)
- added R1507: 3k3, Resistor_SMD:R_0805_2012Metric, F.Cu at (205.0, 94.8)
- added R1508: 1k8, Resistor_SMD:R_0805_2012Metric, F.Cu at (205.0, 97.8)
- added R1601: 100k, Resistor_SMD:R_0805_2012Metric, F.Cu at (143.8, 136.9)
- added R1602: 100k, Resistor_SMD:R_0805_2012Metric, F.Cu at (143.8, 139.9)
- added R1603: 150R, Resistor_SMD:R_0805_2012Metric, F.Cu at (143.8, 142.8)
- added R1604: 82k5, Resistor_SMD:R_0805_2012Metric, F.Cu at (143.8, 145.8)
- added R1605: 48k7, Resistor_SMD:R_0805_2012Metric, F.Cu at (143.8, 148.7)
- added R1606: 4k7, Resistor_SMD:R_0805_2012Metric, F.Cu at (143.8, 151.7)
- added R1701: 470R, Resistor_SMD:R_0805_2012Metric, F.Cu at (142.4, 213.5)
- added R1702: 470R, Resistor_SMD:R_0805_2012Metric, F.Cu at (142.4, 216.5)
- added R1703: 1M, Resistor_SMD:R_1206_3216Metric, F.Cu at (153.1, 213.7)
- added R701: 0R01, Resistor_SMD:R_0805_2012Metric, F.Cu at (272.1, 65.6)
- added R702: 100k, Resistor_SMD:R_0805_2012Metric, F.Cu at (272.1, 68.5)
- added R703: 12k, Resistor_SMD:R_0805_2012Metric, F.Cu at (272.1, 71.5)
- added R704: 0R, Resistor_SMD:R_0805_2012Metric, F.Cu at (272.1, 74.4)
- added R705: 0R, Resistor_SMD:R_0805_2012Metric, F.Cu at (272.1, 77.4)
- added R706: 0R, Resistor_SMD:R_0805_2012Metric, F.Cu at (272.1, 80.3)
- added R707: 0R, Resistor_SMD:R_0805_2012Metric, F.Cu at (272.1, 83.3)
- added R801: 10k, Resistor_SMD:R_0805_2012Metric, F.Cu at (237.5, 65.6)
- added R802: 66k5, Resistor_SMD:R_0805_2012Metric, F.Cu at (237.5, 68.5)
- added R803: 2k, Resistor_SMD:R_0805_2012Metric, F.Cu at (237.5, 71.5)
- added R804: 30k9, Resistor_SMD:R_0805_2012Metric, F.Cu at (237.5, 74.4)
- added R805: 10k, Resistor_SMD:R_0805_2012Metric, F.Cu at (237.5, 77.4)
- added R806: 100k, Resistor_SMD:R_0805_2012Metric, F.Cu at (237.5, 80.3)
- added R807: 24k9, Resistor_SMD:R_0805_2012Metric, F.Cu at (237.5, 83.3)
- added R808: 4k99, Resistor_SMD:R_0805_2012Metric, F.Cu at (241.9, 65.6)
- added R809: 21k, Resistor_SMD:R_0805_2012Metric, F.Cu at (241.9, 68.5)
- added R810: 5k1, Resistor_SMD:R_0805_2012Metric, F.Cu at (241.9, 71.5)
- added R811: 21k, Resistor_SMD:R_0805_2012Metric, F.Cu at (241.9, 74.4)
- added R812: 5k1, Resistor_SMD:R_0805_2012Metric, F.Cu at (241.9, 77.4)
- added R813: 10k, Resistor_SMD:R_0805_2012Metric, F.Cu at (241.9, 80.3)
- added R814: 51k1, Resistor_SMD:R_0805_2012Metric, F.Cu at (241.9, 83.3)
- added R815: 10k, Resistor_SMD:R_0805_2012Metric, F.Cu at (246.3, 65.6)
- added R816: 10k, Resistor_SMD:R_0805_2012Metric, F.Cu at (246.3, 68.5)
- added R817: 10k, Resistor_SMD:R_0805_2012Metric, F.Cu at (246.3, 71.5)
- added R818: 0R, Resistor_SMD:R_0805_2012Metric, F.Cu at (246.3, 74.4)
- added R901: 100k, Resistor_SMD:R_0805_2012Metric, F.Cu at (188.1, 197.4)
- added R902: 0R, Resistor_SMD:R_0805_2012Metric, F.Cu at (188.1, 200.3)
- added R903: 18k, Resistor_SMD:R_0805_2012Metric, F.Cu at (188.1, 203.3)
- added R904: 100k, Resistor_SMD:R_0805_2012Metric, F.Cu at (188.1, 206.2)
- added R905: 4k53, Resistor_SMD:R_0805_2012Metric, F.Cu at (188.1, 209.2)
- added R906: 22k6, Resistor_SMD:R_0805_2012Metric, F.Cu at (192.5, 197.4)
- added R907: 2k2, Resistor_SMD:R_0805_2012Metric, F.Cu at (192.5, 200.3)
- added R908: 100k, Resistor_SMD:R_0805_2012Metric, F.Cu at (192.5, 203.3)
- added R909: 330R, Resistor_SMD:R_0805_2012Metric, F.Cu at (192.5, 206.2)
- added SW1001: Reset, Same Sky:TS11, F.Cu at (193.6, 155.2)
- added SW1002: On / Off, Same Sky:TS11, F.Cu at (193.6, 164.8)
- added TH901: 10k, Resistor_SMD:R_0805_2012Metric, F.Cu at (192.5, 209.2)
- added TP1001: ~, Testpoints_Kampi:TestPoint_Pad_1.0x1.0mm, F.Cu at (218.0, 157.8)
- added TP1002: ~, Testpoints_Kampi:TestPoint_Pad_1.0x1.0mm, F.Cu at (218.0, 160.9)
- added TP1101: ~, Testpoints_Kampi:TestPoint_Pad_1.0x1.0mm, F.Cu at (173.5, 85.7)
- added TP1102: ~, Testpoints_Kampi:TestPoint_Pad_1.0x1.0mm, F.Cu at (173.5, 88.8)
- added TP1103: ~, Testpoints_Kampi:TestPoint_Pad_1.0x1.0mm, F.Cu at (173.5, 91.8)
- added TP1201: ~, Testpoints_Kampi:TestPoint_Pad_1.0x1.0mm, F.Cu at (157.8, 177.7)
- added TP1202: ~, Testpoints_Kampi:TestPoint_Pad_1.0x1.0mm, F.Cu at (157.8, 180.7)
- added TP1203: ~, Testpoints_Kampi:TestPoint_Pad_1.0x1.0mm, F.Cu at (160.8, 177.7)
- added TP1204: ~, Testpoints_Kampi:TestPoint_Pad_1.0x1.0mm, F.Cu at (160.8, 180.7)
- added TP1205: ~, Testpoints_Kampi:TestPoint_Pad_1.0x1.0mm, F.Cu at (163.9, 177.7)
- added TP1206: ~, Testpoints_Kampi:TestPoint_Pad_1.0x1.0mm, F.Cu at (163.9, 180.7)
- added TP1301: ~, Testpoints_Kampi:TestPoint_Pad_1.0x1.0mm, F.Cu at (271.0, 143.2)
- added TP1302: ~, Testpoints_Kampi:TestPoint_Pad_1.0x1.0mm, F.Cu at (271.0, 146.3)
- added TP1303: ~, Testpoints_Kampi:TestPoint_Pad_1.0x1.0mm, F.Cu at (271.0, 149.3)
- added TP1304: ~, Testpoints_Kampi:TestPoint_Pad_1.0x1.0mm, F.Cu at (274.1, 143.2)
- added TP1305: ~, Testpoints_Kampi:TestPoint_Pad_1.0x1.0mm, F.Cu at (274.1, 146.3)
- added TP1306: ~, Testpoints_Kampi:TestPoint_Pad_1.0x1.0mm, F.Cu at (274.1, 149.3)
- added TP1307: ~, Testpoints_Kampi:TestPoint_Pad_1.0x1.0mm, F.Cu at (277.1, 143.2)
- added TP1308: ~, Testpoints_Kampi:TestPoint_Pad_1.0x1.0mm, F.Cu at (277.1, 146.3)
- added TP1309: ~, Testpoints_Kampi:TestPoint_Pad_1.0x1.0mm, F.Cu at (277.1, 149.3)
- added TP1401: ~, Testpoints_Kampi:TestPoint_Pad_1.0x1.0mm, F.Cu at (267.3, 195.0)
- added TP1402: ~, Testpoints_Kampi:TestPoint_Pad_1.0x1.0mm, F.Cu at (267.3, 198.1)
- added TP1403: ~, Testpoints_Kampi:TestPoint_Pad_1.0x1.0mm, F.Cu at (270.4, 195.0)
- added TP1404: ~, Testpoints_Kampi:TestPoint_Pad_1.0x1.0mm, F.Cu at (270.4, 198.1)
- added TP1405: ~, Testpoints_Kampi:TestPoint_Pad_1.0x1.0mm, F.Cu at (273.4, 195.0)
- added TP1406: ~, Testpoints_Kampi:TestPoint_Pad_1.0x1.0mm, F.Cu at (273.4, 198.1)
- added TP1501: ~, Testpoints_Kampi:TestPoint_Pad_1.0x1.0mm, F.Cu at (214.3, 107.1)
- added TP1601: ~, Testpoints_Kampi:TestPoint_Pad_1.0x1.0mm, F.Cu at (163.6, 147.0)
- added TP1602: ~, Testpoints_Kampi:TestPoint_Pad_1.0x1.0mm, F.Cu at (163.6, 150.1)
- added TP1603: ~, Testpoints_Kampi:TestPoint_Pad_1.0x1.0mm, F.Cu at (163.6, 153.1)
- added TP1701: ~, Testpoints_Kampi:TestPoint_Pad_1.0x1.0mm, F.Cu at (134.2, 213.6)
- added TP1702: ~, Testpoints_Kampi:TestPoint_Pad_1.0x1.0mm, F.Cu at (134.2, 216.6)
- added TP701: ~, Testpoints_Kampi:TestPoint_Pad_1.0x1.0mm, F.Cu at (284.3, 85.2)
- added TP801: ~, Testpoints_Kampi:TestPoint_Pad_1.0x1.0mm, F.Cu at (250.0, 83.7)
- added TP802: ~, Testpoints_Kampi:TestPoint_Pad_1.0x1.0mm, F.Cu at (250.0, 86.7)
- added TP803: ~, Testpoints_Kampi:TestPoint_Pad_1.0x1.0mm, F.Cu at (250.0, 89.8)
- added TP804: ~, Testpoints_Kampi:TestPoint_Pad_1.0x1.0mm, F.Cu at (250.0, 92.8)
- added TP806: ~, Testpoints_Kampi:TestPoint_Pad_1.0x1.0mm, F.Cu at (253.1, 83.7)
- added TP807: ~, Testpoints_Kampi:TestPoint_Pad_1.0x1.0mm, F.Cu at (253.1, 86.7)
- added TP808: ~, Testpoints_Kampi:TestPoint_Pad_1.0x1.0mm, F.Cu at (253.1, 89.8)
- added TP809: ~, Testpoints_Kampi:TestPoint_Pad_1.0x1.0mm, F.Cu at (253.1, 92.8)
- added TP810: ~, Testpoints_Kampi:TestPoint_Pad_1.0x1.0mm, F.Cu at (256.1, 83.7)
- added TP811: ~, Testpoints_Kampi:TestPoint_Pad_1.0x1.0mm, F.Cu at (256.1, 86.7)
- added TP812: ~, Testpoints_Kampi:TestPoint_Pad_1.0x1.0mm, F.Cu at (256.1, 89.8)
- added TP901: ~, Testpoints_Kampi:TestPoint_Pad_1.0x1.0mm, F.Cu at (184.4, 197.4)
- added TP902: ~, Testpoints_Kampi:TestPoint_Pad_1.0x1.0mm, F.Cu at (184.4, 200.5)
- added TP903: ~, Testpoints_Kampi:TestPoint_Pad_1.0x1.0mm, F.Cu at (184.4, 203.5)
- added TP904: ~, Testpoints_Kampi:TestPoint_Pad_1.0x1.0mm, F.Cu at (184.4, 206.6)
- added TP905: ~, Testpoints_Kampi:TestPoint_Pad_1.0x1.0mm, F.Cu at (184.4, 209.6)
- added X1001: UART, Connector_PinHeader_2.54mm:PinHeader_1x03_P2.54mm_Vertical, F.Cu at (214.2, 154.0)
- added X1002: SoM, TE:2309409-2, F.Cu at (215.6, 137.9)
- added X1101: LoRa, Connector_PCBEdge:BUS_PCI_Express_Mini_Full, F.Cu at (149.5, 116.1)
- added X1301: DEBUG, Samtec:SHF-105-01-L-D-SM-TR, F.Cu at (282.4, 145.5)
- added X1302: UART, Connector_PinHeader_2.54mm:PinHeader_1x03_P2.54mm_Vertical, F.Cu at (267.2, 144.0)
- added X1501: OTG, Connector_USB:USB_C_Receptacle_GCT_USB4110, F.Cu at (223.3, 83.9)
- added X1502: GPIO, Connector_Phoenix_MSTB:PhoenixContact_MSTBA_2,5_10-G-5,08_1x10_P5.08mm_Horizontal, F.Cu at (183.0, 67.6)
- added X1503: I2C, Connector_Phoenix_MSTB:PhoenixContact_MSTBA_2,5_4-G-5,08_1x04_P5.08mm_Horizontal, F.Cu at (183.0, 82.1)
- added X1504: CAN, Connector_Phoenix_MSTB:PhoenixContact_MSTBA_2,5_4-G-5,08_1x04_P5.08mm_Horizontal, F.Cu at (183.0, 96.6)
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
Commit message: Working on PCB
Parts:
- removed LED1601: Power Good, LED_SMD:LED_0805_2012Metric
- removed R1508: 1k8, Resistor_SMD:R_0805_2012Metric
- removed R1602: 100k, Resistor_SMD:R_0805_2012Metric
- removed R1603: 150R, Resistor_SMD:R_0805_2012Metric
- removed TP1204, TP1205, TP1305, TP1306, TP1307, TP1308, TP1404, TP1405, TP1406, TP812: ~, Testpoints_Kampi:TestPoint_Pad_1.0x1.0mm
- added C1704: 10n, Capacitor_SMD:C_0805_2012Metric, F.Cu at (241.5, 350.6)
- added C1705: 100n, Capacitor_SMD:C_0805_2012Metric, F.Cu at (217.9, 657.6)
- added C1706: 100n, Capacitor_SMD:C_0805_2012Metric, F.Cu at (194.2, 657.5)
- added C1707: 1n, Capacitor_SMD:C_1206_3216Metric, F.Cu at (220.9, 638.9)
- added C702: 100n, Capacitor_SMD:C_0805_2012Metric, F.Cu at (170.2, 490.7)
- added D1701: SS36, Diode_SMD:D_SMA, F.Cu at (235.3, 339.1)
- added D1702: SS36, Diode_SMD:D_SMA, F.Cu at (235.3, 343.7)
- added D1703: SS36, Diode_SMD:D_SMA, F.Cu at (235.3, 348.2)
- added D1704: SS36, Diode_SMD:D_SMA, F.Cu at (235.3, 352.8)
- added IC1701: TLP293, Toshiba:TLP293(TPL,E, F.Cu at (232.5, 685.0)
- added IC702: INA219AxD, Package_SO:SOIC-8_3.9x4.9mm_P1.27mm, F.Cu at (165.3, 489.4)
- added M1701: Ag5400, Silvertel:Ag5400, F.Cu at (250.6, 692.3)
- added Q701: BSS123, Package_TO_SOT_SMD:SOT-23, F.Cu at (213.4, 486.7)
- added R1013: 0R, Resistor_SMD:R_0805_2012Metric, F.Cu at (220.9, 754.8)
- added R1502: 1k8, Resistor_SMD:R_0805_2012Metric, F.Cu at (228.6, 854.1)
- added R1607: 100k, Resistor_SMD:R_0805_2012Metric, F.Cu at (104.7, 400.6)
- added R1704: 470R, Resistor_SMD:R_0805_2012Metric, F.Cu at (209.5, 664.2)
- added R1705: 1M, Resistor_SMD:R_2010_5025Metric, F.Cu at (217.9, 639.0)
- added R708: 0R, Resistor_SMD:R_0805_2012Metric, F.Cu at (159.8, 486.8)
- added R709: 100k, Resistor_SMD:R_0805_2012Metric, F.Cu at (194.7, 475.7)
- added R710: 12k, Resistor_SMD:R_0805_2012Metric, F.Cu at (191.2, 475.7)
- added TP1703: ~, Testpoints_Kampi:TestPoint_Pad_1.0x1.0mm, F.Cu at (240.8, 344.5)
- added TP1704: ~, Testpoints_Kampi:TestPoint_Pad_1.0x1.0mm, F.Cu at (240.8, 347.5)
- added TP702: ~, Testpoints_Kampi:TestPoint_Pad_1.0x1.0mm, F.Cu at (212.5, 483.8)
- added TP703: ~, Testpoints_Kampi:TestPoint_Pad_1.0x1.0mm, F.Cu at (195.7, 473.5)
- added TP805: ~, Testpoints_Kampi:TestPoint_Pad_1.0x1.0mm, F.Cu at (234.5, 440.5)
- C1701: value 100n -> 470u; footprint Capacitor_SMD:C_0805_2012Metric -> Capacitor_SMD:CP_Elec_6.3x7.7
- C1702: value 100n -> 4n7; footprint Capacitor_SMD:C_0805_2012Metric -> Capacitor_SMD:C_1206_3216Metric
- C1703: value 1n / 2 kV -> 4n7
- C701: value 100n -> 10n
- C815: value 22u -> 10u
- C816: value 10p -> 22u
- C817: value 1u -> 10u
- C818: value 10n -> 10p
- C820: value 1u -> 10n
- C822, C823: value 10u -> 1u
- IC1101, IC1201, IC1301, IC1401, IC804: value MIC5317-3.3xM5 -> TLV75733PDBV
- IC1303: value TXB0104PWR -> 74LVC1G07; footprint Package_SO:TSSOP-14_4.4x5mm_P0.65mm -> Package_TO_SOT_SMD:SOT-353_SC-70-5
- IC1304: value 74LVC1G07 -> TXB0104PWR; footprint Package_TO_SOT_SMD:SOT-353_SC-70-5 -> Package_SO:TSSOP-14_4.4x5mm_P0.65mm
- IC701: value INA219AxD -> TPS2121RUXT; footprint Package_SO:SOIC-8_3.9x4.9mm_P1.27mm -> Texas Instruments:RUX0012A
- IC805: value MIC5317-1.8xM5 -> TLV75733PDBV
- R1003: value 10k -> 1k8
- R1005: value 10k -> 1k5
- R1006: value 1k8 -> 10k
- R1007: value ~ -> 10k
- R1009: value ~ -> 1k8
- R1010: value 0R -> ~
- R1012: value 1k5 -> ~
- R1303: value 10k -> 68R
- R1304, R1307: value 0R -> 10k
- R1312: value 10k -> 0R
- R1313: value 68R -> 0R
- R1701, R1702: value 470R -> ~
- R1703: value 1M -> 470R; footprint Resistor_SMD:R_1206_3216Metric -> Resistor_SMD:R_0805_2012Metric
- R701: value 0R01 -> 51k1
- R702: value 100k -> 10k
- R703: value 12k -> 10k
- R704: value 0R -> 0R01
- X1502: footprint Connector_Phoenix_MSTB:PhoenixContact_MSTBA_2,5_10-G-5,08_1x10_P5.08mm_Horizontal -> Phoenix:MSTBA_2,5_10-G-5,08_1x10_P5.08mm_Horizontal
- X1503, X1504, X1505: footprint Connector_Phoenix_MSTB:PhoenixContact_MSTBA_2,5_4-G-5,08_1x04_P5.08mm_Horizontal -> Phoenix:MSTBA_2,5_4-G-5,08_1x04_P5.08mm_Horizontal
- X701: value 7-16 V -> DC In
- moved MP1101 795.0 mm to (153.9, 883.5)
- moved X1501 783.0 mm to (228.4, 866.8)
- moved R1501 780.6 mm to (227.9, 860.4), turned to 90 degrees
- moved TP1102 779.5 mm to (180.5, 868.3), turned to -90 degrees
- moved R1503 771.5 mm to (230.6, 854.1), turned to -90 degrees
- moved C1502 771.1 mm to (226.6, 854.1), turned to -90 degrees
- moved R1102 765.0 mm to (178.1, 863.6), turned to 90 degrees
- moved LED1101 762.7 mm to (178.1, 867.3), turned to -90 degrees
- moved IC1502 753.8 mm to (228.1, 857.3)
- moved TP1501 748.1 mm to (232.8, 855.0), turned to -90 degrees
- moved R1302 746.3 mm to (150.1, 864.3), turned to 90 degrees
- moved MP1301 744.3 mm to (160.9, 883.5)
- moved MP1601 733.9 mm to (181.9, 883.5)
- moved LED1301 724.6 mm to (150.1, 868.0), turned to -90 degrees
- moved MP1201 721.1 mm to (174.9, 883.5)
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Connections:
- net /Project Architecture/Power/PowerMux-Status renamed /Project Architecture/Power/Backup-Status
- C1203 pad 1: /Project Architecture/Zigbee/+3V3 -> +1V8
- C1204 pad 1: +1V8 -> /Project Architecture/Zigbee/+3V3
- C1605 pad 1: Net-(D1601-K) -> Net-(IC1601-BOOT)
- C1605 pad 2: Net-(IC1601-BOOT) -> Net-(D1601-K)
- C1701 pad 1: Net-(X1701-MXCT1) -> /Project Architecture/Ethernet/PoE
- C1702 pad 1: Net-(X1701-MXCT3) -> GND
- C1702 pad 2: GND -> Net-(D1703-A)
- C1703 pad 1: Earth -> GND
- C1703 pad 2: GND -> Net-(D1701-A)
- C701 pad 1: +3V3 -> Net-(IC701-SS)
- C815 pad 1: GND -> V_{Backup}
- C815 pad 2: Net-(IC803-IN1) -> GND
- C816 pad 1: Net-(IC801-BIAS) -> GND
- C816 pad 2: Net-(C816-Pad2) -> Net-(IC803-IN1)
- C817 pad 1: GND -> V_{Backup}
- C817 pad 2: +5V -> GND
- C818 pad 1: Net-(IC803-SS) -> Net-(IC801-BIAS)
- C818 pad 2: GND -> Net-(C818-Pad2)
- C819 pad 2: +3V3 -> +5V
- C820 pad 1: GND -> Net-(IC803-SS)
- C820 pad 2: +5V -> GND
- C821 pad 2: +1V8 -> +3V3
- C822 pad 1: V_{Backup} -> GND
- C822 pad 2: GND -> +5V
- C823 pad 1: V_{Backup} -> GND
- C823 pad 2: GND -> +1V8
- IC1303 pad 1: +1V8 -> unconnected-(IC1303-NC-Pad1)
- IC1303 pad 2: Net-(IC1303-A1) -> /Project Architecture/System on Module/Thread.Boot
- IC1303 pad 3: Net-(IC1303-A2) -> GND
- IC1303 pad 4: Net-(IC1303-A3) -> Net-(M1301-P1.15)
- IC1303 pad 5: Net-(IC1303-A4) -> +1V8
- IC1304 pad 1: unconnected-(IC1304-NC-Pad1) -> +1V8
- IC1304 pad 2: /Project Architecture/System on Module/Thread.Boot -> Net-(IC1304-A1)
- IC1304 pad 3: GND -> Net-(IC1304-A2)
- IC1304 pad 4: Net-(M1301-P1.15) -> Net-(IC1304-A3)
- IC1304 pad 5: +1V8 -> Net-(IC1304-A4)
- IC701 pad 1: Net-(IC701-A1) -> Net-(F701-Pad1)
- IC701 pad 2: Net-(IC701-A0) -> /Project Architecture/Ethernet/PoE
- IC701 pad 3: /Project Architecture/Battery/I2C.SDA -> GND
- IC701 pad 4: /Project Architecture/Battery/I2C.SCL -> GND
- IC701 pad 5: +3V3 -> GND
- IC701 pad 7: V_{In} -> Net-(IC701-IN1)
- IC701 pad 8: Net-(IC701-IN+) -> Net-(F701-Pad1)
- LED1302 pad 1: Net-(LED1302-K) -> GND
- M1301 pad 6: Net-(LED1302-A) -> Net-(M1301-P0.05/AIN1)
- M1401 pad 1: (no net) -> Net-(M1401-P1)
- M1401 pad 10: (no net) -> Net-(M1401-P1)
- M1401 pad 11: (no net) -> Net-(M1401-P1)
- M1401 pad 12: (no net) -> Net-(M1401-P1)
- M1401 pad 13: (no net) -> Net-(M1401-P1)
- M1401 pad 14: (no net) -> Net-(M1401-P1)
- M1401 pad 2: (no net) -> Net-(M1401-P1)
- M1401 pad 20: (no net) -> Net-(M1401-P1)
- M1401 pad 21: (no net) -> Net-(M1401-P1)
- M1401 pad 22: (no net) -> Net-(M1401-P1)
- M1401 pad 23: (no net) -> Net-(M1401-P1)
- M1401 pad 3: (no net) -> Net-(M1401-P1)
- M1401 pad 4: (no net) -> Net-(M1401-P1)
- M1401 pad 6: (no net) -> Net-(M1401-P1)
- M1401 pad 8: (no net) -> Net-(M1401-P1)
- M1401 pad 9: (no net) -> Net-(M1401-P1)
- R1003 pad 2: Net-(R1003-Pad2) -> /Project Architecture/Ethernet/AT-DET
- R1004 pad 1: +1V8 -> /Project Architecture/System on Module/Ready
- R1004 pad 2: Net-(R1004-Pad2) -> GND
- R1005 pad 1: +1V8 -> Net-(LED1001-K)
- R1005 pad 2: /Project Architecture/System on Module/~{CTRL_RESET_MOCI} -> Net-(Q1001-D)
- R1006 pad 1: /Project Architecture/System on Module/~{CTRL_RESET_MICO} -> +1V8
- R1007 pad 1: /Project Architecture/System on Module/~{SoM-Peripheral-Reset} -> +1V8
- R1007 pad 2: /Project Architecture/System on Module/~{CTRL_RESET_MOCI} -> Net-(R1007-Pad2)
- R1008 pad 2: Net-(R1008-Pad2) -> /Project Architecture/System on Module/~{CTRL_RESET_MOCI}
- R1009 pad 1: GND -> /Project Architecture/System on Module/~{CTRL_RESET_MICO}
- R1009 pad 2: /Project Architecture/System on Module/~{CTRL_FORCE_OFF_MOC} -> Net-(R1009-Pad2)
- R1010 pad 1: Net-(R1010-Pad1) -> /Project Architecture/System on Module/~{SoM-Peripheral-Reset}
- R1010 pad 2: /Project Architecture/Power/PWR_1V8_MOCI -> /Project Architecture/System on Module/~{CTRL_RESET_MOCI}
- R1011 pad 1: /Project Architecture/System on Module/Ready -> +1V8
- R1011 pad 2: GND -> Net-(R1011-Pad2)
- R1012 pad 1: Net-(LED1001-K) -> GND
- R1012 pad 2: Net-(Q1001-D) -> /Project Architecture/System on Module/~{CTRL_FORCE_OFF_MOC}
- R1303 pad 1: +1V8 -> Net-(M1301-P0.05/AIN1)
- R1303 pad 2: /Project Architecture/Thread/~{RESET} -> Net-(LED1302-A)
- R1304 pad 1: /Project Architecture/Thread/Thread-CTS -> +1V8
- R1304 pad 2: Net-(IC1303-B3) -> /Project Architecture/Thread/~{RESET}
- R1305 pad 1: /Project Architecture/Thread/Thread-RTS -> /Project Architecture/Thread/Thread-CTS
- R1305 pad 2: Net-(IC1303-B4) -> Net-(IC1304-B3)
- R1306 pad 1: /Project Architecture/Thread/Thread-TxD -> /Project Architecture/Thread/Thread-RTS
- R1306 pad 2: Net-(IC1303-B1) -> Net-(IC1304-B4)
- R1307 pad 1: Net-(IC1303-B2) -> /Project Architecture/Thread/+3V3
- R1307 pad 2: /Project Architecture/Thread/Thread-RxD -> Net-(M1301-P1.15)
- R1308 pad 1: Net-(IC1303-A3) -> /Project Architecture/Thread/Thread-TxD
- R1308 pad 2: /Project Architecture/System on Module/Thread.RTS -> Net-(IC1304-B1)
- R1309 pad 1: Net-(IC1303-A4) -> Net-(IC1304-B2)
- R1309 pad 2: /Project Architecture/System on Module/Thread.CTS -> /Project Architecture/Thread/Thread-RxD
- R1310 pad 1: Net-(IC1303-A1) -> Net-(IC1304-A3)
- R1310 pad 2: /Project Architecture/System on Module/Thread.RxD -> /Project Architecture/System on Module/Thread.RTS
- R1311 pad 1: /Project Architecture/System on Module/Thread.TxD -> Net-(IC1304-A4)
- R1311 pad 2: Net-(IC1303-A2) -> /Project Architecture/System on Module/Thread.CTS
- R1312 pad 1: /Project Architecture/Thread/+3V3 -> Net-(IC1304-A1)
- R1312 pad 2: Net-(M1301-P1.15) -> /Project Architecture/System on Module/Thread.RxD
- R1313 pad 1: Net-(LED1302-K) -> /Project Architecture/System on Module/Thread.TxD
- R1313 pad 2: GND -> Net-(IC1304-A2)
- R1601 pad 1: /Project Architecture/NVMe/SSD-Power-Enable -> GND
- R1601 pad 2: GND -> Net-(IC1601-~{EN1})
- R1701 pad 1: +3V3 -> /Project Architecture/Ethernet/PoE
- R1701 pad 2: Net-(X1701-LED2+) -> Net-(M1701-ADJ)
- R1702 pad 1: +3V3 -> Net-(M1701-ADJ)
- R1702 pad 2: Net-(X1701-LED1-) -> GND
- R1703 pad 1: Earth -> +3V3
- R1703 pad 2: GND -> Net-(X1701-LED2+)
- R701 pad 1: Net-(IC701-IN+) -> Net-(IC701-ILIM)
- R701 pad 2: V_{In} -> GND
- R702 pad 1: /Project Architecture/Power Input/ADC.ADC_1 -> Net-(IC701-ST)
- R702 pad 2: V_{In} -> GND
- R703 pad 1: GND -> +1V8
- R703 pad 2: /Project Architecture/Power Input/ADC.ADC_1 -> /Project Architecture/Power Input/Input-Status
- R704 pad 1: Net-(IC701-A1) -> Net-(IC702-IN+)
- R704 pad 2: +3V3 -> V_{In}
- R705 pad 1: Net-(IC701-A1) -> Net-(IC702-A1)
- R705 pad 2: GND -> +3V3
- R706 pad 1: +3V3 -> Net-(IC702-A1)
- R706 pad 2: Net-(IC701-A0) -> GND
- R707 pad 1: GND -> +3V3
- R707 pad 2: Net-(IC701-A0) -> Net-(IC702-A0)
- R808 pad 2: Net-(C816-Pad2) -> Net-(C818-Pad2)
- SW1001 pad 1: Net-(R1006-Pad2) -> Net-(R1009-Pad2)
- TP1001 pad 1: /Project Architecture/System on Module/~{CTRL_RESET_MOCI} -> /Project Architecture/System on Module/Ready
- TP1002 pad 1: /Project Architecture/System on Module/Ready -> /Project Architecture/System on Module/~{CTRL_RESET_MOCI}
- TP1302 pad 1: /Project Architecture/System on Module/Thread.Reset -> /Project Architecture/Thread/+3V3
- TP1303 pad 1: /Project Architecture/Thread/+3V3 -> /Project Architecture/System on Module/Thread.Reset
- TP1701 pad 1: /Project Architecture/Ethernet/PoE-B -> Net-(D1703-A)
- TP1702 pad 1: /Project Architecture/Ethernet/PoE-A -> Net-(D1701-A)
- TP701 pad 1: V_{In} -> Net-(F701-Pad1)
- X1002 pad 212: Net-(R1003-Pad2) -> Net-(R1006-Pad2)
- X1002 pad 214: Net-(R1010-Pad1) -> Net-(R1013-Pad1)
- X1002 pad 216: Net-(R1004-Pad2) -> Net-(R1007-Pad2)
- X1002 pad 218: Net-(R1008-Pad2) -> Net-(R1011-Pad2)
- X1002 pad 38: unconnected-(X1002-Pad38) -> /Project Architecture/Power Input/Input-Status
- X1002 pad 48: unconnected-(X1002-Pad48) -> /Project Architecture/Ethernet/AT-DET
- X701 pad 1: Net-(F701-Pad1) -> Net-(IC701-IN1)
Other:
- board outline added: 400 x 250 mm

Commit message: Working on layout
Parts:
- removed R810, R812: 5k1, Resistor_SMD:R_0805_2012Metric
- removed R811: 21k, Resistor_SMD:R_0805_2012Metric
- removed R814: 51k1, Resistor_SMD:R_0805_2012Metric
- removed the TP1201 at (159.1, 772.6)
- removed TP1601, TP803, TP807, TP904: ~, Testpoints_Kampi:TestPoint_Pad_1.0x1.0mm
- removed the TP903 at (145.3, 450.7)
- added BT1001: Backup, Keystone:3034, F.Cu at (194.0, 736.5)
- added R711: 30k, Resistor_SMD:R_0805_2012Metric, F.Cu at (381.4, 757.4)
- added R712: 2k, Resistor_SMD:R_0805_2012Metric, F.Cu at (377.9, 757.4)
- added R819: 0R, Resistor_SMD:R_0805_2012Metric, F.Cu at (402.6, 759.2)
- added TP1201: ~, Testpoints_Kampi:TestPoint_Pad_1.0x1.0mm, F.Cu at (161.9, 852.1)
- added TP1201: ~, Testpoints_Kampi:TestPoint_Pad_1.0x1.0mm, F.Cu at (154.4, 758.7)
- added TP1705: ~, Testpoints_Kampi:TestPoint_Pad_1.0x1.0mm, F.Cu at (375.0, 755.1)
- BAT901: value Backup Power -> Backup Battery
- C816: value 22u -> ~
- R701: value 51k1 -> 33k
- R809: value 21k -> 27k
- moved C1601 514.9 mm to (370.8, 821.2), turned to -90 degrees
- moved C1602 513.4 mm to (372.8, 821.2), turned to -90 degrees
- moved C1603 508.7 mm to (368.8, 821.2), turned to -90 degrees
- moved IC1601 505.6 mm to (362.1, 821.1)
- moved C1604 505.1 mm to (366.8, 821.2), turned to -90 degrees
- moved R1601 503.5 mm to (356.7, 821.7)
- moved R1604 501.1 mm to (356.8, 824.8)
- moved R1605 500.4 mm to (360.4, 824.8)
- moved R1607 498.2 mm to (364.8, 825.6), turned to 90 degrees
- moved C1605 494.9 mm to (357.2, 818.2), turned to 90 degrees
- moved L1601 493.9 mm to (370.1, 815.5)
- moved D1601 491.1 mm to (362.1, 816.1), turned to 180 degrees
- moved TP1602 488.2 mm to (359.4, 826.9), turned to 180 degrees
- moved TP1603 484.4 mm to (376.9, 815.5)
- moved TP902 402.7 mm to (437.8, 724.4), turned to 180 degrees
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- renumbered TP802 to TP903
Connections:
- net /Project Architecture/Peripherals/SCL_{HV} renamed Net-(IC1504-B2)
- net /Project Architecture/Peripherals/SDA_{HV} renamed Net-(IC1504-B1)
- net V_{Backup} renamed Net-(D801-K)
- C1504 pad 1: +3V3 -> Net-(IC1503-VCCB)
- C1508 pad 1: +3V3 -> Net-(IC1504-VCCB)
- C1509 pad 1: +3V3 -> Net-(IC1505-VCCB)
- C1510 pad 1: +3V3 -> Net-(IC1506-VCCB)
- C809 pad 2: Net-(IC803-IN1) -> Net-(IC801-BIAS)
- C811 pad 2: Net-(IC803-IN1) -> Net-(IC801-BIAS)
- C813 pad 2: Net-(IC803-IN1) -> Net-(IC801-BIAS)
- C814 pad 2: Net-(IC803-IN1) -> Net-(IC801-BIAS)
- C816 pad 2: Net-(IC803-IN1) -> Net-(IC801-BIAS)
- C818 pad 1: Net-(IC801-BIAS) -> Net-(IC801-FB)
- IC1503 pad 19: +3V3 -> Net-(IC1503-VCCB)
- IC1504 pad 7: +3V3 -> Net-(IC1504-VCCB)
- IC1505 pad 7: +3V3 -> Net-(IC1505-VCCB)
- IC1506 pad 7: +3V3 -> Net-(IC1506-VCCB)
- IC1601 pad 2: Net-(IC1601-PG) -> unconnected-(IC1601-PG-Pad2)
- IC701 pad 1: Net-(F701-Pad1) -> Net-(IC702-IN+)
- IC701 pad 5: GND -> Net-(IC701-OV1)
- IC701 pad 8: Net-(F701-Pad1) -> Net-(IC702-IN+)
- IC801 pad 11: Net-(IC801-RT) -> Net-(IC801-SpSp)
- IC801 pad 7: Net-(IC801-BIAS) -> Net-(IC801-FB)
- IC803 pad 4: Net-(IC803-OV2) -> GND
- IC803 pad 5: Net-(IC803-OV1) -> GND
- IC803 pad 7: Net-(IC803-IN1) -> Net-(IC801-BIAS)
- L802 pad 2: Net-(IC803-IN1) -> Net-(IC801-BIAS)
- R1504 pad 1: +3V3 -> Net-(IC1504-VCCB)
- R1505 pad 1: +3V3 -> Net-(IC1506-VCCB)
- R1506 pad 1: +3V3 -> Net-(IC1504-VCCB)
- R1507 pad 1: +3V3 -> Net-(IC1506-VCCB)
- R806 pad 1: Net-(IC803-IN1) -> Net-(IC801-BIAS)
- R806 pad 2: Net-(IC801-BIAS) -> Net-(IC801-FB)
- R807 pad 1: Net-(IC801-BIAS) -> Net-(IC801-FB)
- R808 pad 1: Net-(IC803-IN1) -> Net-(IC801-BIAS)
- R809 pad 1: Net-(IC803-IN1) -> Net-(IC803-ILIM)
- R809 pad 2: Net-(IC803-OV1) -> GND
- TP701 pad 1: Net-(F701-Pad1) -> Net-(IC701-OV1)
- TP804 pad 1: Net-(IC803-IN1) -> Net-(IC801-BIAS)
- X1502 pad 1: +3V3 -> Net-(IC1503-VCCB)
- X1503 pad 1: +3V3 -> Net-(IC1504-VCCB)
- X1504 pad 1: +3V3 -> Net-(IC1505-VCCB)
- X1505 pad 1: +3V3 -> Net-(IC1506-VCCB)
Routing:
- net GND: track 0.00 -> 83.5 mm, vias 0 -> 93
- net Net-(IC801-BIAS): track 0.00 -> 44.2 mm, vias 0 -> 4
- net Net-(BT1001-+): track 0.00 -> 39.5 mm, vias 0 -> 2
- net /Project Architecture/NVMe/V_{SSD}: track 0.00 -> 23.4 mm, vias 0 -> 2
- net Net-(IC701-ST): track 0.00 -> 16.6 mm
- net V_{In}: track 0.00 -> 15.6 mm, vias 0 -> 4
- net +5V: track 0.00 -> 14.6 mm
- net /Project Architecture/Battery/REGN: track 0.00 -> 13.8 mm, vias 0 -> 2
- net /Project Architecture/System on Module/~{CTRL_RECOVERY_MICO}: track 0.00 -> 10.7 mm
- net Net-(IC702-A1): track 0.00 -> 9.93 mm
- net Net-(IC901-TS): track 0.00 -> 9.18 mm
- net Net-(D1703-A): track 0.00 -> 9.01 mm, vias 0 -> 2
- net Net-(IC801-FB): track 0.00 -> 8.24 mm
- net Net-(IC803-ST): track 0.00 -> 7.96 mm
- net Net-(IC702-A0): track 0.00 -> 7.88 mm
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- added copper zone on F.Cu, net /Project Architecture/Battery/V_{Batt}
- added copper zone on F.Cu, net /Project Architecture/Ethernet/PoE
- added copper zone on F.Cu, net /Project Architecture/Ethernet/PoE-A
- added copper zone on F.Cu, net /Project Architecture/Ethernet/PoE-B
- added copper zone on F.Cu, net Earth
- added copper zone on F.Cu, net GND
- added copper zone on In1.Cu, net GND
- added copper zone on F.Cu, net Net-(BAT901--)
- added copper zone on F.Cu, net Net-(C904-Pad1)
- added copper zone on F.Cu, net Net-(D1601-K)
- added copper zone on F.Cu, net Net-(D1701-A)
- added copper zone on F.Cu, net Net-(D1703-A)
- added copper zone on F.Cu, net Net-(D801-A)
- added copper zone on F.Cu, net Net-(D801-K)
- added copper zone on F.Cu, net Net-(IC702-IN+)
- added copper zone on F.Cu, net Net-(IC801-BIAS)
- added copper zone on F.Cu, net Net-(IC801-SW)
- added copper zone on F.Cu, net V_{In}
- added copper zone on In2.Cu, net V_{In}
