File: gateway/Gateway.kicad_pcb (KiCad board)
At the start: 4 copper layers, 400 x 250 mm, 301 parts, among them IC1101 TLV75733PDBV, IC1102 74LVC1G07, IC1201 TLV75733PDBV, IC1202 TXB0102DCT, IC1203 74LVC1G07, IC1204 74LVC1G07, IC1301 TLV75733PDBV, IC1302 74LVC1G07, IC1303 74LVC1G07, IC1304 TXB0104PWR, IC1401 TLV75733PDBV, IC1402 74LVC1G07, IC1403 TXB0102DCT, IC1501 ATECC608B-SSHDA, IC1502 TUSB320, IC1503 TXS0108EPW, IC1504 TXS0102DCU, IC1505 TXB0102DCU, IC1506 TXS0102DCU, IC1601 ST1S14PHR, IC1701 TLP293, IC701 TPS2121RUXT, IC702 INA219AxD, IC801 LM62460, IC802 ADP1614ACPZ-650-R7, IC803 TPS2121RUXT, IC804 TLV75733PDBV, IC805 TLV75733PDBV, IC901 BQ25308, IC902 MAX17048, IC903 BQ297xy, M1201 RF-BM-2652, M1301 BT40, M1401 iM891A-XL, M1701 Ag5400, Q1001 BSS123, Q701 BSS123, Q801 BSS123, Q901 Si2342DS, Q902 Si2342DS, SW1001 Reset, SW1002 On / Off, X1001 UART, X1002 SoM, X1101 LoRa, X1301 DEBUG, X1302 UART, X1501 OTG, X1502 GPIO, X1503 I2C, X1504 CAN, X1505 I2C, X1601 SSD, X1701 Ethernet, X701 DC In

Commit message: Working on layout
Parts:
- removed TP1001, TP1002, TP808, TP810: ~, Testpoints_Kampi:TestPoint_Pad_1.0x1.0mm
- removed the TP1201 at (161.9, 852.1)
- added C824: 100n, Capacitor_SMD:C_0805_2012Metric, F.Cu at (285.3, 966.1)
- added C825: 10u, Capacitor_SMD:C_0805_2012Metric, F.Cu at (282.5, 974.6)
- added R1602: 100k, Resistor_SMD:R_0805_2012Metric, F.Cu at (221.4, 1051.7)
- added R810: 5k36, Resistor_SMD:R_0805_2012Metric, F.Cu at (293.9, 969.4)
- added R811: 23k7, Resistor_SMD:R_0805_2012Metric, F.Cu at (293.9, 975.4)
- added R812: 5k36, Resistor_SMD:R_0805_2012Metric, F.Cu at (293.9, 973.4)
- added R814: 22k1, Resistor_SMD:R_0805_2012Metric, F.Cu at (293.9, 977.4)
- added R820: 93k1, Resistor_SMD:R_0805_2012Metric, F.Cu at (293.9, 965.4)
- added R821: 1M, Resistor_SMD:R_0805_2012Metric, B.Cu at (291.3, 966.1)
- added R822: 23k2, Resistor_SMD:R_0805_2012Metric, F.Cu at (287.3, 966.1)
- added R823: 10k, Resistor_SMD:R_0805_2012Metric, F.Cu at (289.3, 966.1)
- added R824: 10k, Resistor_SMD:R_0805_2012Metric, F.Cu at (279.8, 970.2)
- added R910: 5M1, Resistor_SMD:R_0805_2012Metric, F.Cu at (290.0, 1024.6)
- added R911: 5M1, Resistor_SMD:R_0805_2012Metric, F.Cu at (297.3, 1025.5)
- added REF**: MountingHole_3.2mm_M3, MountingHole:MountingHole_3.2mm_M3, F.Cu at (259.0, 1013.0)
- added REF**: MountingHole_3.2mm_M3, MountingHole:MountingHole_3.2mm_M3, F.Cu at (162.0, 943.0)
- added REF**: MountingHole_3.2mm_M3, MountingHole:MountingHole_3.2mm_M3, F.Cu at (356.0, 943.0)
- added REF**: MountingHole_3.2mm_M3, MountingHole:MountingHole_3.2mm_M3, F.Cu at (162.0, 1083.0)
- added REF**: MountingHole_3.2mm_M3, MountingHole:MountingHole_3.2mm_M3, F.Cu at (356.0, 1083.0)
- added TP802: ~, Testpoints_Kampi:TestPoint_Pad_1.0x1.0mm, F.Cu at (279.3, 973.3)
- added TP803: ~, Testpoints_Kampi:TestPoint_Pad_1.0x1.0mm, F.Cu at (285.3, 968.8)
- BT1001: footprint Keystone:3034 -> Keystone:3030TR; moved to B.Cu
- C1203, C1204, C1303, C1304, C1403, C1404, C1503, C1504, C1505, C1506, C1507, C1508, C1509, C1510, IC1202, IC1304, IC1403, IC1503, IC1504, IC1505, IC1506, R1008, R1010, R1012, R1202, R1203, R1205, R1206, R1305, R1306, R1308, R1309, R1310, R1311, R1312, R1313, R1403, R1404, R1405, R1406, R1504, R1505, R1506, R1507: moved to B.Cu
- C820: value 10n -> 220u; footprint Capacitor_SMD:C_0805_2012Metric -> Capacitor_Tantalum_SMD:CP_EIA-7343-31_Kemet-D
- Q901, Q902: value Si2342DS -> CSD16301Q2; footprint Package_TO_SOT_SMD:SOT-23 -> Package_SON:Texas_DQK
- R809: value 27k -> 23k7
- R815: value 10k -> 93k1
- R816: value 10k -> 16k5
- moved C1609 687.7 mm to (211.6, 1070.5), turned to 180 degrees
- moved C1608 684.7 mm to (211.6, 1064.5), turned to 180 degrees
- moved C1610 680.8 mm to (211.6, 1066.5), turned to 180 degrees
- moved C1611 679.8 mm to (211.6, 1068.5), turned to 180 degrees
- moved C1607 678.9 mm to (218.1, 1069.1)
- moved C1606 677.4 mm to (231.3, 1050.5), turned to 180 degrees
- moved H1601 673.6 mm to (172.3, 1060.3)
- moved R1606 672.6 mm to (193.7, 1064.3)
- moved H1001 635.9 mm to (171.5, 1039.2)
- moved H1002 632.0 mm to (236.5, 1039.2), turned to 90 degrees
- moved R818 586.3 mm to (186.3, 1016.1), turned to 90 degrees
- moved TH901 580.4 mm to (310.6, 1015.0), turned to -90 degrees
- moved R817 550.1 mm to (272.0, 976.6), turned to -90 degrees
- moved C823 544.3 mm to (277.7, 977.8), turned to -90 degrees
- moved C822 542.9 mm to (275.4, 973.6)
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- renumbered MP1601 to MP1001
Connections:
- net /Project Architecture/Zigbee/CC2652-Boot renamed Net-(M1201-DIO15)
- C820 pad 1: Net-(IC803-SS) -> +5V
- IC803 pad 3: GND -> Net-(IC803-CP2)
- IC803 pad 4: GND -> Net-(IC803-OV2)
- IC803 pad 5: GND -> Net-(IC803-OV1)
- IC803 pad 6: GND -> Net-(IC803-PR1)
- M1401 pad 1: Net-(M1401-P1) -> unconnected-(M1401-P1-Pad1)
- M1401 pad 10: Net-(M1401-P1) -> unconnected-(M1401-P10-Pad10)
- M1401 pad 11: Net-(M1401-P1) -> unconnected-(M1401-P11-Pad11)
- M1401 pad 12: Net-(M1401-P1) -> unconnected-(M1401-P12-Pad12)
- M1401 pad 13: Net-(M1401-P1) -> unconnected-(M1401-P13-Pad13)
- M1401 pad 14: Net-(M1401-P1) -> unconnected-(M1401-P14-Pad14)
- M1401 pad 2: Net-(M1401-P1) -> unconnected-(M1401-P2-Pad2)
- M1401 pad 20: Net-(M1401-P1) -> unconnected-(M1401-P20-Pad20)
- M1401 pad 21: Net-(M1401-P1) -> unconnected-(M1401-P21-Pad21)
- M1401 pad 22: Net-(M1401-P1) -> unconnected-(M1401-P22-Pad22)
- M1401 pad 23: Net-(M1401-P1) -> unconnected-(M1401-P23-Pad23)
- M1401 pad 3: Net-(M1401-P1) -> unconnected-(M1401-P3-Pad3)
- M1401 pad 4: Net-(M1401-P1) -> unconnected-(M1401-P4-Pad4)
- M1401 pad 6: Net-(M1401-P1) -> unconnected-(M1401-P6-Pad6)
- M1401 pad 8: Net-(M1401-P1) -> unconnected-(M1401-P8-Pad8)
- M1401 pad 9: Net-(M1401-P1) -> unconnected-(M1401-P9-Pad9)
- Q801 pad 3: /Project Architecture/Power/Backup-Status -> /Project Architecture/Power/PowerMux-Status
- Q901 pad 1: Net-(IC903-Cout) -> Net-(Q901-D-Pad1)
- Q901 pad 2: GND -> Net-(Q901-D-Pad1)
- Q901 pad 3: Net-(Q901-D) -> Net-(IC903-Cout)
- Q902 pad 1: Net-(IC903-Dout) -> Net-(Q901-D-Pad1)
- Q902 pad 2: Net-(BAT901--) -> Net-(Q901-D-Pad1)
- Q902 pad 3: Net-(Q901-D) -> Net-(IC903-Dout)
- R809 pad 1: Net-(IC803-ILIM) -> Net-(IC801-BIAS)
- R809 pad 2: GND -> Net-(IC803-OV1)
- R815 pad 1: Net-(IC803-ST) -> Net-(IC803-CP2)
- R816 pad 1: +1V8 -> Net-(IC801-BIAS)
- R816 pad 2: /Project Architecture/Power/Backup-Status -> Net-(IC803-PR1)
- TP806 pad 1: Net-(IC803-OV1) -> /Project Architecture/Power/PowerMux-Status
- X1002 pad 17: /Project Architecture/Peripherals/GPIO.Num0 -> /Project Architecture/Peripherals/GPIO.Num2
- X1002 pad 21: /Project Architecture/Peripherals/GPIO.Num2 -> /Project Architecture/Peripherals/GPIO.Num0
- X1002 pad 210: /Project Architecture/Power/Backup-Status -> /Project Architecture/System on Module/Backup-Status
- X1002 pad 94: /Project Architecture/Peripherals/GPIO.Num3 -> /Project Architecture/Peripherals/GPIO.Num4
- X1002 pad 96: /Project Architecture/Peripherals/GPIO.Num4 -> /Project Architecture/Peripherals/GPIO.Num3
Routing:
- net /Project Architecture/Battery/I2C.SDA: track 2.95 -> 339.7 mm, vias 0 -> 9
- net /Project Architecture/Battery/I2C.SCL: track 2.93 -> 337.8 mm, vias 0 -> 8
- net /Project Architecture/Power/SoM-Power-Enable: track 0.00 -> 266.1 mm, vias 0 -> 5
- net /Project Architecture/System on Module/~{CTRL_PWR_BTN_MICO}: track 0.00 -> 232.1 mm, vias 0 -> 1
- net /Project Architecture/System on Module/~{CTRL_RESET_MICO}: track 0.00 -> 222.1 mm, vias 0 -> 2
- net /Project Architecture/Zigbee/+3V3: track 1.96 -> 221.5 mm, vias 0 -> 5
- net GND: track 83.5 -> 301.3 mm, vias 93 -> 273
- net /Project Architecture/LoRa/+3V3: track 0.00 -> 206.6 mm, vias 0 -> 3
- net /Project Architecture/System on Module/Ready: track 0.00 -> 198.6 mm, vias 0 -> 2
- net /Project Architecture/LoRa/LoRa.Reset: track 0.00 -> 183.2 mm, vias 0 -> 6
- net /Project Architecture/LoRa/LoRa.D_P: track 0.00 -> 156.0 mm
- net /Project Architecture/LoRa/LoRa.D_N: track 0.00 -> 156.0 mm
- net /Project Architecture/System on Module/Thread.Boot: track 0.00 -> 126.9 mm, vias 0 -> 4
- net /Project Architecture/Power Input/ADC.ADC_1: track 1.68 -> 127.1 mm, vias 0 -> 2
- net /Project Architecture/LoRa/LoRa-Power-Enable: track 0.00 -> 116.9 mm, vias 0 -> 2
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- added copper zone on In2.Cu, net +1V8
- added copper zone on In2.Cu, net +3V3
- added copper zone on F.Cu, net +5V
- added copper zone on In2.Cu, net +5V
- added copper zone on In2.Cu, net /Project Architecture/Battery/V_{Batt}
- added copper zone on In2.Cu, net /Project Architecture/Ethernet/PoE
- added copper zone on F.Cu, net /Project Architecture/NVMe/V_{SSD}
- added copper zone on In2.Cu, net /Project Architecture/NVMe/V_{SSD}
- added copper zone on In2.Cu, net /Project Architecture/Peripherals/USB.VBUS
- added copper zone on B.Cu, net Net-(IC1504-VCCB)
- added copper zone on B.Cu, net Net-(IC1505-VCCB)
- added copper zone on B.Cu, net Net-(IC1506-VCCB)
- added copper zone on F.Cu, net Net-(IC701-IN1)
- added copper zone on In2.Cu, net Net-(IC701-IN1)
- added copper zone on F.Cu, net Net-(Q901-D-Pad1)
Other:
- board size 400 x 250 mm -> 204 x 150 mm

Commit message: Prepare release 1.0.0
Parts:
- moved BT1001 852.2 mm to (133.2, 150.2)
- moved C1001 852.2 mm to (282.7, 227.3)
- moved C1101 852.2 mm to (255.0, 119.3)
- moved C1102 852.2 mm to (261.3, 120.8)
- moved C1206 852.2 mm to (195.6, 144.7)
- moved C1301 852.2 mm to (236.2, 212.8)
- moved C1401 852.2 mm to (205.0, 206.4)
- moved C1502 852.2 mm to (115.9, 136.2)
- moved C1504 852.2 mm to (123.6, 221.8)
- moved C1508 852.2 mm to (200.4, 234.6)
- moved C1509 852.2 mm to (175.5, 234.6)
- moved C1510 852.2 mm to (225.4, 234.6)
- moved C1701 852.2 mm to (169.4, 135.2)
- moved C1703 852.2 mm to (172.6, 105.1)
- moved C701 852.2 mm to (255.8, 107.8)
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- renumbered R1003 to R1706
Routing:
- net /Project Architecture/System on Module/Zigbee.TxD: track 50.7 -> 46.8 mm
