File: gateway/Gateway.kicad_pcb (KiCad board)
At the start: 4 copper layers, 204 x 150 mm, 317 parts, among them IC1101 TLV75733PDBV, IC1102 74LVC1G07, IC1201 TLV75733PDBV, IC1202 TXB0102DCT, IC1203 74LVC1G07, IC1204 74LVC1G07, IC1301 TLV75733PDBV, IC1302 74LVC1G07, IC1303 74LVC1G07, IC1304 TXB0104PWR, IC1401 TLV75733PDBV, IC1402 74LVC1G07, IC1403 TXB0102DCT, IC1501 ATECC608B-SSHDA, IC1502 TUSB320, IC1503 TXS0108EPW, IC1504 TXS0102DCU, IC1505 TXB0102DCU, IC1506 TXS0102DCU, IC1601 ST1S14PHR, IC1701 TLP293, IC701 TPS2121RUXT, IC702 INA219AxD, IC801 LM62460, IC802 ADP1614ACPZ-650-R7, IC803 TPS2121RUXT, IC804 TLV75733PDBV, IC805 TLV75733PDBV, IC901 BQ25308, IC902 MAX17048, IC903 BQ297xy, M1201 RF-BM-2652, M1301 BT40, M1401 iM891A-XL, M1701 Ag5400, Q1001 BSS123, Q701 BSS123, Q801 BSS123, Q901 CSD16301Q2, Q902 CSD16301Q2, SW1001 Reset, SW1002 On / Off, X1001 UART, X1002 SoM, X1101 LoRa, X1301 DEBUG, X1302 UART, X1501 OTG, X1502 GPIO, X1503 I2C, X1504 CAN, X1505 I2C, X1601 SSD, X1701 Ethernet, X701 DC In

Commit message: Replace battery charger with BQ25300
Parts:
- IC901: value BQ25308 -> BQ25300
Connections:
- net /Project Architecture/Battery/~{Battery-Charge-Enable} renamed /Project Architecture/Battery/Battery-Charge-Enable

Commit message: Smaller changes
Parts:
- H1001, H1002: value MountingHole -> Spacer
- H1601: value MountingHole -> 2230
Changed lines of the file:
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@@
 	(property "RELEASE_TITLE_2.2.0" "Version 2.2.0 not found.")
 	(property "RELEASE_TITLE_UNRELEASED" "Version Unreleased not found.")
-	(property "REVISION" "")
+	(property "REVISION" "X.Y.Z")
 	(property "SHEET_NAME_1" "Cover Page")
 	(property "SHEET_NAME_10" "System on Module")
@@
 			)
 		)
-		(property ki_fp_filters "MountingHole*")
+		(property ki_fp_filters "Spacer*")
 		(sheetname "/Project Architecture/LoRa/")
 		(sheetfile "LoRa.kicad_sch")
@@
 			)
 		)
-		(property ki_fp_filters "MountingHole*")
+		(property ki_fp_filters "Spacer*")
 		(sheetname "/Project Architecture/LoRa/")
 		(sheetfile "LoRa.kicad_sch")
@@
 			)
 		)
-		(property "Config" ""
+		(property "Config" "+POE"
 			(at 0 0 180)
 			(unlocked yes)
@@
 			)
 		)
-		(property "Value" "MountingHole"
+		(property "Value" "Spacer"
 			(at 0 0 90)
 			(layer "F.SilkS")
@@
 			)
 		)
-		(property "Description" "Mounting Hole without connection"
+		(property "Description" ""
 			(at 0 0 90)
 			(layer "F.Fab")
@@
 			)
 		)
-		(property ki_fp_filters "MountingHole*")
+		(property ki_fp_filters "Spacer*")
 		(sheetname "/Project Architecture/System on Module/")
 		(sheetfile "SoM.kicad_sch")
@@
 			)
 		)
-		(attr through_hole exclude_from_pos_files exclude_from_bom)
+		(attr through_hole)
 		(duplicate_pad_numbers_are_jumpers no)
 		(fp_line
@@
 			)
 		)
-		(property "Config" ""
+		(property "Config" "+POE"
 			(at 0 0 90)
 			(unlocked yes)
@@
 			)
 		)
-		(property "Value" "MountingHole"
+		(property "Value" "2230"
 			(at 0 0 0)
 			(layer "F.SilkS")
@@
 			)
 		)
-		(property "Description" "Mounting Hole without connection"
+		(property "Description" ""
 			(at 0 0 0)
 			(layer "F.Fab")
@@
 			)
 		)
-		(property ki_fp_filters "MountingHole*")
+		(property ki_fp_filters "Spacer*")
 		(sheetname "/Project Architecture/NVMe/")
 		(sheetfile "NVMe.kicad_sch")
@@
 			)
 		)
-		(attr through_hole exclude_from_pos_files exclude_from_bom)
+		(attr through_hole)
 		(duplicate_pad_numbers_are_jumpers no)
 		(fp_line
@@
 			)
 		)
-		(property "Value" "MountingHole"
+		(property "Value" "Spacer"
 			(at 0 0 0)
 			(layer "F.SilkS")
@@
 			)
 		)
-		(property "Description" "Mounting Hole without connection"
+		(property "Description" ""
 			(at 0 0 0)
 			(layer "F.Fab")
@@
 			)
 		)
-		(property ki_fp_filters "MountingHole*")
+		(property ki_fp_filters "Spacer*")
 		(sheetname "/Project Architecture/System on Module/")
 		(sheetfile "SoM.kicad_sch")
@@
 			)
 		)
-		(attr through_hole exclude_from_pos_files exclude_from_bom)
+		(attr through_hole)
 		(duplicate_pad_numbers_are_jumpers no)
 		(fp_line
@@
 	)
 	(segment
+		(start 172.525 174)
+		(end 172.525 162.4)
+		(width 0.2)
+		(layer "F.Cu")
+		(net "/Project Architecture/Battery/Battery-Charge-Enable")
+	)
+	(segment
+		(start 229.5 157.149998)
+		(end 228.625 157.149998)
+		(width 0.2)
+		(layer "F.Cu")
+		(net "/Project Architecture/Battery/Battery-Charge-Enable")
+	)
+	(segment
+		(start 230.255 157.149998)
+		(end 229.5 157.149998)
+		(width 0.2)
+		(layer "F.Cu")
+		(net "/Project Architecture/Battery/Battery-Charge-Enable")
+	)
+	(via
+		(at 229.5 157.149998)
+		(size 0.45)
+		(drill 0.25)
+		(layers "F.Cu" "B.Cu")
+		(net "/Project Architecture/Battery/Battery-Charge-Enable")
+	)
+	(via
+		(at 172.525 174)
+		(size 0.45)
+		(drill 0.25)
+		(layers "F.Cu" "B.Cu")
+		(net "/Project Architecture/Battery/Battery-Charge-Enable")
+	)
+	(segment
+		(start 227.4 160.7)
+		(end 224.4 163.7)
+		(width 0.2)
+		(layer "B.Cu")
+		(net "/Project Architecture/Battery/Battery-Charge-Enable")
+	)
+	(segment
+		(start 227.4 158.6)
+		(end 227.4 160.7)
+		(width 0.2)
+		(layer "B.Cu")
+		(net "/Project Architecture/Battery/Battery-Charge-Enable")
+	)
+	(segment
+		(start 224.4 172.4)
+		(end 222.8 174)
+		(width 0.2)
+		(layer "B.Cu")
+		(net "/Project Architecture/Battery/Battery-Charge-Enable")
+	)
+	(segment
+		(start 228.850002 157.149998)
+		(end 227.4 158.6)
+		(width 0.2)
+		(layer "B.Cu")
+		(net "/Project Architecture/Battery/Battery-Charge-Enable")
+	)
+	(segment
+		(start 222.8 174)
+		(end 172.525 174)
+		(width 0.2)
+		(layer "B.Cu")
+		(net "/Project Architecture/Battery/Battery-Charge-Enable")
+	)
+	(segment
+		(start 229.5 157.149998)
+		(end 228.850002 157.149998)
+		(width 0.2)
+		(layer "B.Cu")
+		(net "/Project Architecture/Battery/Battery-Charge-Enable")
+	)
+	(segment
+		(start 224.4 163.7)
+		(end 224.4 172.4)
+		(width 0.2)
+		(layer "B.Cu")
+		(net "/Project Architecture/Battery/Battery-Charge-Enable")
+	)
+	(segment
 		(start 230.412501 154.887499)
 		(end 228.625 153.099998)
@@
 		(net "Net-(IC1202-A1)")
 	)
-	(segment
-		(start 172.525 174)
-		(end 172.525 162.4)
-		(width 0.2)
-		(layer "F.Cu")
-		(net "/Project Architecture/Battery/Battery-Charge-Enable")
-	)
-	(segment
-		(start 229.5 157.149998)
-		(end 228.625 157.149998)
-		(width 0.2)
-		(layer "F.Cu")
-		(net "/Project Architecture/Battery/Battery-Charge-Enable")
-	)
-	(segment
-		(start 230.255 157.149998)
-		(end 229.5 157.149998)
-		(width 0.2)
-		(layer "F.Cu")
-		(net "/Project Architecture/Battery/Battery-Charge-Enable")
-	)
-	(via
-		(at 229.5 157.149998)
-		(size 0.45)
-		(drill 0.25)
-		(layers "F.Cu" "B.Cu")
-		(net "/Project Architecture/Battery/Battery-Charge-Enable")
-	)
-	(via
-		(at 172.525 174)
-		(size 0.45)
-		(drill 0.25)
-		(layers "F.Cu" "B.Cu")
-		(net "/Project Architecture/Battery/Battery-Charge-Enable")
-	)
-	(segment
-		(start 227.4 160.7)
-		(end 224.4 163.7)
-		(width 0.2)
-		(layer "B.Cu")
-		(net "/Project Architecture/Battery/Battery-Charge-Enable")
-	)
-	(segment
-		(start 227.4 158.6)
-		(end 227.4 160.7)
-		(width 0.2)
-		(layer "B.Cu")
-		(net "/Project Architecture/Battery/Battery-Charge-Enable")
-	)
-	(segment
-		(start 224.4 172.4)
-		(end 222.8 174)
-		(width 0.2)
-		(layer "B.Cu")
-		(net "/Project Architecture/Battery/Battery-Charge-Enable")
-	)
-	(segment
-		(start 228.850002 157.149998)
-		(end 227.4 158.6)
-		(width 0.2)
-		(layer "B.Cu")
-		(net "/Project Architecture/Battery/Battery-Charge-Enable")
-	)
-	(segment
-		(start 222.8 174)
-		(end 172.525 174)
-		(width 0.2)
-		(layer "B.Cu")
-		(net "/Project Architecture/Battery/Battery-Charge-Enable")
-	)
-	(segment
-		(start 229.5 157.149998)
-		(end 228.850002 157.149998)
-		(width 0.2)
-		(layer "B.Cu")
-		(net "/Project Architecture/Battery/Battery-Charge-Enable")
-	)
-	(segment
-		(start 224.4 163.7)
-		(end 224.4 172.4)
-		(width 0.2)
-		(layer "B.Cu")
-		(net "/Project Architecture/Battery/Battery-Charge-Enable")
-	)
 	(zone
