File: gateway/Battery.kicad_sch (KiCad schematic)
At the start: 29 parts, among them IC801 BQ25308, IC802 MAX17048, IC803 BQ297xy, Q801 Si2342DS, Q802 Si2342DS

Commit message: Working on first version
Parts:
- added R801: 100k, Resistor_SMD:R_0402_1005Metric, symbol Device:R
- R802: renamed from R801; value 10k -> 0R; footprint Resistor_SMD:R_0402_1005Metric -> Resistor_SMD:R_0805_2012Metric; manf# CR0402-JW-103GLF -> CR0805-J/-000ELF; mouser# 652-CR0402-JW-103GLF -> 652-CR0805-J/-000ELF
- R804: renamed from R803; now not fitted; now left out of the parts list
- R808: renamed from R813; now not fitted; now left out of the parts list
- renumbered L802 to L801, R802 to R803, R804 to R805, R811 to R806, R812 to R807, R814 to R809, TP803 to TP802, TP804 to TP803, TP805 to TP804, TP811 to TP805
Connections:
- net GND: now also IC801.5 (POL), R801.2
- net ~{Battery-Charge-Enable}: now reaches IC801.6 (~{EN})
- net ~{Battery-Charge-Enable}: now also R801.1
- no-connect marks 2 -> 0
Other:
- moved on the sheet: TP801, TP805

Commit message: Working on version 1.0
Parts:
- C802, C803: manf TAIYO YUDEN -> KYOCERA AVX; manf# MCJCT21GCB7225MTPA1J -> 0805ZC225JAT2A; mouser# 963-T21GCB7225MTPA1J -> 581-0805ZC225JAT2A
- C804: footprint Capacitor_SMD:C_0402_1005Metric -> Capacitor_SMD:C_0805_2012Metric; manf# 04023C473KAT4A -> 08053C473K4T2A; mouser# 581-04023C473KAT4A -> 581-08053C473K4T2A
- C806, C807: footprint Capacitor_SMD:C_0402_1005Metric -> Capacitor_SMD:C_0805_2012Metric; manf# 04025C104JAT2A -> 08053C104M4T4A; mouser# 581-04025C104JAT2A -> 581-08053C104M4T4A
- C808: footprint Capacitor_SMD:C_0603_1608Metric -> Capacitor_SMD:C_0805_2012Metric; manf TAIYO YUDEN -> KYOCERA AVX; manf# MBASE168BB5475KTNA01 -> 08055D475KAT4A; mouser# 963-BASE168BB5475KT -> 581-08055D475KAT4A
- R801, R804, R808: manf# CR0402-JW-104GLF -> CR0805-JW-104GLF; mouser# 652-CR0402-JW-104GLF -> 652-CR0805-JW-104GLF
- R803: footprint Resistor_SMD:R_0402_1005Metric -> Resistor_SMD:R_0805_2012Metric; manf# CR0402-JW-183GLF -> CR0805-JW-183GLF; mouser# 652-CR0402-JW-183GLF -> 652-CR0805-JW-183GLF
- R805: footprint Resistor_SMD:R_0402_1005Metric -> Resistor_SMD:R_0805_2012Metric; manf# CR0402-FX-4531GLF -> CR0805-FX-4531GLF; mouser# 652-CR0402-FX-4531GLF -> 652-CR0805-FX-4531GLF
- R806: footprint Resistor_SMD:R_0402_1005Metric -> Resistor_SMD:R_0805_2012Metric; manf# CR0402-FX-2262GLF -> CR0805-FX-2262GLF; mouser# 652-CR0402-FX-2262GLF -> 652-CR0805-FX-2262GLF
- R807: footprint Resistor_SMD:R_0402_1005Metric -> Resistor_SMD:R_0805_2012Metric; manf# CR0402-JW-222GLF -> CR0805-JW-222GLF; mouser# 652-CR0402-JW-222GLF -> 652-CR0805-JW-222GLF
- R809: footprint Resistor_SMD:R_0402_1005Metric -> Resistor_SMD:R_0805_2012Metric; manf# CR0402-JW-331GLF -> CR0805-JW-331GLF; mouser# 652-CR0402-JW-331GLF -> 652-CR0805-JW-331GLF
- TH801: footprint Resistor_SMD:R_0402_1005Metric -> Resistor_SMD:R_0805_2012Metric; manf TDK -> Bourns; manf# NTCG103JF103HTDS -> CR0805-JW-103GLF; mouser# 810-NTCG103JF103HTDS -> 652-CR0805-JW-103GLF
Changed lines of the file:
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@@
 	(text_box "Battery Charger"
 		(exclude_from_sim no)
-		(at 88.9 162.56 0)
-		(size 130.81 7.62)
+		(at 55.88 162.56 0)
+		(size 163.83 7.62)
 		(margins 1.9049 1.9049 1.9049 1.9049)
 		(stroke
@@
 			)
 		)
-		(property "Footprint" "Capacitor_SMD:C_0402_1005Metric"
+		(property "Footprint" "Capacitor_SMD:C_0805_2012Metric"
 			(at 251.7648 161.29 0)
 			(hide yes)
@@
 			)
 		)
-		(property "Datasheet" "https://datasheets.kyocera-avx.com/KGM_X7R.pdf"
+		(property "Datasheet" "https://datasheets.kyocera-avx.com/AutoMLCC.pdf"
 			(at 252.73 157.48 0)
 			(hide yes)
@@
 			)
 		)
-		(property "manf#" "04025C104JAT2A"
+		(property "manf#" "08053C104M4T4A"
 			(at 252.73 157.48 0)
 			(hide yes)
@@
 			)
 		)
-		(property "mouser#" "581-04025C104JAT2A"
+		(property "mouser#" "581-08053C104M4T4A"
 			(at 252.73 157.48 0)
 			(hide yes)
@@
 		(dnp no)
 		(property "Reference" "IC803"
-			(at 260.35 104.14 0)
+			(at 261.62 104.14 0)
 			(show_name no)
 			(do_not_autoplace no)
@@
 			)
 		)
-		(property "Footprint" "Resistor_SMD:R_0402_1005Metric"
+		(property "Footprint" "Resistor_SMD:R_0805_2012Metric"
 			(at 192.532 115.57 90)
 			(hide yes)
@@
 			)
 		)
-		(property "manf#" "CR0402-FX-2262GLF"
+		(property "manf#" "CR0805-FX-2262GLF"
 			(at 194.31 115.57 0)
 			(hide yes)
@@
 			)
 		)
-		(property "mouser#" "652-CR0402-FX-2262GLF"
+		(property "mouser#" "652-CR0805-FX-2262GLF"
 			(at 194.31 115.57 0)
 			(hide yes)
@@
 			)
 		)
-		(property "Footprint" "Resistor_SMD:R_0402_1005Metric"
+		(property "Footprint" "Resistor_SMD:R_0805_2012Metric"
 			(at 192.532 104.14 90)
 			(hide yes)
@@
 			)
 		)
-		(property "manf#" "CR0402-FX-4531GLF"
+		(property "manf#" "CR0805-FX-4531GLF"
 			(at 194.31 104.14 0)
 			(hide yes)
@@
 			)
 		)
-		(property "mouser#" "652-CR0402-FX-4531GLF"
+		(property "mouser#" "652-CR0805-FX-4531GLF"
 			(at 194.31 104.14 0)
 			(hide yes)
@@
 			)
 		)
-		(property "manf#" "CR0402-JW-104GLF"
+		(property "manf#" "CR0805-JW-104GLF"
 			(at 85.09 115.57 0)
 			(hide yes)
@@
 			)
 		)
-		(property "mouser#" "652-CR0402-JW-104GLF"
+		(property "mouser#" "652-CR0805-JW-104GLF"
 			(at 85.09 115.57 0)
 			(hide yes)
@@
 		(in_bom no)
 		(on_board yes)
-		(in_pos_files yes)
+		(in_pos_files no)
 		(dnp yes)
 		(property "Reference" "C808"
@@
 			)
 		)
-		(property "Footprint" "Capacitor_SMD:C_0603_1608Metric"
+		(property "Footprint" "Capacitor_SMD:C_0805_2012Metric"
 			(at 332.4352 113.03 0)
 			(hide yes)
@@
 			)
 		)
-		(property "Datasheet" ""
+		(property "Datasheet" "https://datasheets.kyocera-avx.com/cx5r.pdf"
 			(at 331.47 109.22 0)
 			(hide yes)
@@
 			)
 		)
-		(property "manf" "TAIYO YUDEN"
+		(property "manf" "KYOCERA AVX"
 			(at 331.47 109.22 0)
 			(hide yes)
@@
 			)
 		)
-		(property "manf#" "MBASE168BB5475KTNA01"
+		(property "manf#" "08055D475KAT4A"
 			(at 331.47 109.22 0)
 			(hide yes)
@@
 			)
 		)
-		(property "mouser#" "963-BASE168BB5475KT"
+		(property "mouser#" "581-08055D475KAT4A"
 			(at 331.47 109.22 0)
 			(hide yes)
@@
 			)
 		)
-		(property "Footprint" "Resistor_SMD:R_0402_1005Metric"
+		(property "Footprint" "Resistor_SMD:R_0805_2012Metric"
 			(at 158.242 116.84 90)
 			(hide yes)
@@
 			)
 		)
-		(property "manf#" "CR0402-JW-183GLF"
+		(property "manf#" "CR0805-JW-183GLF"
 			(at 160.02 116.84 0)
 			(hide yes)
@@
 			)
 		)
-		(property "mouser#" "652-CR0402-JW-183GLF"
+		(property "mouser#" "652-CR0805-JW-183GLF"
 			(at 160.02 116.84 0)
 			(hide yes)
@@
 			)
 		)
-		(property "Footprint" "Capacitor_SMD:C_0402_1005Metric"
+		(property "Footprint" "Capacitor_SMD:C_0805_2012Metric"
 			(at 172.4152 85.09 0)
 			(hide yes)
@@
 			)
 		)
-		(property "Datasheet" "https://datasheets.kyocera-avx.com/KGM_X7R.pdf"
+		(property "Datasheet" "https://datasheets.kyocera-avx.com/AutoMLCC.pdf"
 			(at 171.45 81.28 0)
 			(hide yes)
@@
 			)
 		)
-		(property "manf#" "04023C473KAT4A"
+		(property "manf#" "08053C473K4T2A"
 			(at 171.45 81.28 0)
 			(hide yes)
@@
 			)
 		)
-		(property "mouser#" "581-04023C473KAT4A"
+		(property "mouser#" "581-08053C473K4T2A"
 			(at 171.45 81.28 0)
 			(hide yes)
@@
 			)
 		)
-		(property "Datasheet" "https://www.mouser.com/catalog/specsheets/Taiyo%20Yuden_1102023_MC_mlcc_all_e.pdf"
+		(property "Datasheet" "https://www.mouser.de/datasheet/3/5926/1/X7RDielectric.pdf"
 			(at 129.54 68.58 0)
 			(hide yes)
@@
 			)
 		)
-		(property "manf" "TAIYO YUDEN"
+		(property "manf" "KYOCERA AVX"
 			(at 129.54 68.58 0)
 			(hide yes)
@@
 			)
 		)
-		(property "manf#" "MCJCT21GCB7225MTPA1J"
+		(property "manf#" "0805ZC225JAT2A"
 			(at 129.54 68.58 0)
 			(hide yes)
@@
 			)
 		)
-		(property "mouser#" "963-T21GCB7225MTPA1J"
+		(property "mouser#" "581-0805ZC225JAT2A"
 			(at 129.54 68.58 0)
 			(hide yes)
@@
 			)
 		)
-		(property "Footprint" "Resistor_SMD:R_0402_1005Metric"
+		(property "Footprint" "Resistor_SMD:R_0805_2012Metric"
 			(at 286.512 100.33 90)
 			(hide yes)
@@
 			)
 		)
-		(property "manf#" "CR0402-JW-331GLF"
+		(property "manf#" "CR0805-JW-331GLF"
 			(at 288.29 100.33 0)
 			(hide yes)
@@
 			)
 		)
-		(property "mouser#" "652-CR0402-JW-331GLF"
+		(property "mouser#" "652-CR0805-JW-331GLF"
 			(at 288.29 100.33 0)
 			(hide yes)
@@
 			)
 		)
-		(property "Footprint" "Resistor_SMD:R_0402_1005Metric"
+		(property "Footprint" "Resistor_SMD:R_0805_2012Metric"
 			(at 234.188 111.76 90)
 			(hide yes)
@@
 			)
 		)
-		(property "manf#" "CR0402-JW-222GLF"
+		(property "manf#" "CR0805-JW-222GLF"
 			(at 232.41 111.76 0)
 			(hide yes)
@@
 			)
 		)
-		(property "mouser#" "652-CR0402-JW-222GLF"
+		(property "mouser#" "652-CR0805-JW-222GLF"
 			(at 232.41 111.76 0)
 			(hide yes)
@@
 			)
 		)
-		(property "manf#" "CR0402-JW-104GLF"
+		(property "manf#" "CR0805-JW-104GLF"
 			(at 172.72 116.84 0)
 			(hide yes)
@@
 			)
 		)
-		(property "mouser#" "652-CR0402-JW-104GLF"
+		(property "mouser#" "652-CR0805-JW-104GLF"
 			(at 172.72 116.84 0)
 			(hide yes)
@@
 			)
 		)
-		(property "Footprint" "Capacitor_SMD:C_0402_1005Metric"
+		(property "Footprint" "Capacitor_SMD:C_0805_2012Metric"
 			(at 289.2552 116.84 0)
 			(hide yes)
@@
 			)
 		)
-		(property "Datasheet" "https://datasheets.kyocera-avx.com/KGM_X7R.pdf"
+		(property "Datasheet" "https://datasheets.kyocera-avx.com/AutoMLCC.pdf"
 			(at 288.29 113.03 0)
 			(hide yes)
@@
 			)
 		)
-		(property "manf#" "04025C104JAT2A"
+		(property "manf#" "08053C104M4T4A"
 			(at 288.29 113.03 0)
 			(hide yes)
@@
 			)
 		)
-		(property "mouser#" "581-04025C104JAT2A"
+		(property "mouser#" "581-08053C104M4T4A"
 			(at 288.29 113.03 0)
 			(hide yes)
@@
 			)
 		)
-		(property "Footprint" "Resistor_SMD:R_0402_1005Metric"
+		(property "Footprint" "Resistor_SMD:R_0805_2012Metric"
 			(at 209.55 115.57 0)
 			(hide yes)
@@
 			)
 		)
-		(property "Datasheet" "https://product.tdk.com/system/files/dam/doc/product/sensor/ntc/chip-ntc-thermistor/catalog/tpd_automotive_ntc-thermistor_ntcg_en.pdf?ref_disty=mouser"
+		(property "Datasheet" "https://www.mouser.de/datasheet/3/40/1/cr.pdf"
 			(at 209.55 115.57 0)
 			(hide yes)
@@
 			)
 		)
-		(property "manf" "TDK"
+		(property "manf" "Bourns"
 			(at 209.55 116.84 0)
 			(hide yes)
@@
 			)
 		)
-		(property "manf#" "NTCG103JF103HTDS"
+		(property "manf#" "CR0805-JW-103GLF"
 			(at 209.55 116.84 0)
 			(hide yes)
@@
 			)
 		)
-		(property "mouser#" "810-NTCG103JF103HTDS"
+		(property "mouser#" "652-CR0805-JW-103GLF"
 			(at 209.55 116.84 0)
 			(hide yes)
@@
 			)
 		)
-		(property "manf#" "CR0402-JW-104GLF"
+		(property "manf#" "CR0805-JW-104GLF"
 			(at 269.24 173.99 0)
 			(hide yes)
@@
 			)
 		)
-		(property "mouser#" "652-CR0402-JW-104GLF"
+		(property "mouser#" "652-CR0805-JW-104GLF"
 			(at 269.24 173.99 0)
 			(hide yes)
@@
 			)
 		)
-		(property "Datasheet" "https://www.mouser.com/catalog/specsheets/Taiyo%20Yuden_1102023_MC_mlcc_all_e.pdf"
+		(property "Datasheet" "https://www.mouser.de/datasheet/3/5926/1/X7RDielectric.pdf"
 			(at 113.03 115.57 0)
 			(hide yes)
@@
 			)
 		)
-		(property "manf" "TAIYO YUDEN"
+		(property "manf" "KYOCERA AVX"
 			(at 113.03 115.57 0)
 			(hide yes)
@@
 			)
 		)
-		(property "manf#" "MCJCT21GCB7225MTPA1J"
+		(property "manf#" "0805ZC225JAT2A"
 			(at 113.03 115.57 0)
 			(hide yes)
@@
 			)
 		)
-		(property "mouser#" "963-T21GCB7225MTPA1J"
+		(property "mouser#" "581-0805ZC225JAT2A"
 			(at 113.03 115.57 0)
 			(hide yes)

Commit message: Working on PCB
Changed lines of the file:
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@@
 		)
 	)
-	(hierarchical_label "I2C{SDA SCL}"
+	(hierarchical_label "I2C{I2C}"
 		(shape bidirectional)
 		(at 209.55 176.53 180)

Commit message: Adding level shifter, update documentation
Parts:
- TP801, TP802, TP803, TP804, TP805: value (none) -> ~
Changed lines of the file:
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@@
 			)
 		)
-		(property "Value" ""
+		(property "Value" "~"
 			(at 252.73 94.615 0)
 			(show_name no)
@@
 			)
 		)
-		(property "Value" ""
+		(property "Value" "~"
 			(at 238.76 94.615 0)
 			(show_name no)
@@
 			)
 		)
-		(property "Value" ""
+		(property "Value" "~"
 			(at 269.24 186.055 0)
 			(show_name no)
@@
 			)
 		)
-		(property "Value" ""
+		(property "Value" "~"
 			(at 209.55 103.505 0)
 			(show_name no)
@@
 			)
 		)
-		(property "Value" ""
+		(property "Value" "~"
 			(at 168.91 130.175 0)
 			(show_name no)

Commit message: Replace level shifter, replace CC2530 with CC2652, fix wrong part numbers
Parts:
- C808: manf# 08055D475KAT4A -> 08053D475MAT2A
- R801, R804, R808: footprint Resistor_SMD:R_0402_1005Metric -> Resistor_SMD:R_0805_2012Metric
Changed lines of the file:
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@@
 			)
 		)
-		(property "Footprint" "Resistor_SMD:R_0402_1005Metric"
+		(property "Footprint" "Resistor_SMD:R_0805_2012Metric"
 			(at 86.868 115.57 90)
 			(hide yes)
@@
 			)
 		)
-		(property "manf#" "08055D475KAT4A"
+		(property "manf#" "08053D475MAT2A"
 			(at 331.47 109.22 0)
 			(hide yes)
@@
 			)
 		)
-		(property "Footprint" "Resistor_SMD:R_0402_1005Metric"
+		(property "Footprint" "Resistor_SMD:R_0805_2012Metric"
 			(at 170.942 116.84 90)
 			(hide yes)
@@
 			)
 		)
-		(property "Footprint" "Resistor_SMD:R_0402_1005Metric"
+		(property "Footprint" "Resistor_SMD:R_0805_2012Metric"
 			(at 267.462 173.99 90)
 			(hide yes)
