File: gateway/Battery.kicad_sch (KiCad schematic)
At the start: 30 parts, among them IC801 BQ25308, IC802 MAX17048, IC803 BQ297xy, Q801 Si2342DS, Q802 Si2342DS

Commit message: Add INA219 for current measurement
Parts:
- renumbered BAT801 to BAT901, C801 to C901, C802 to C902, C803 to C903, C804 to C904, C805 to C905, C806 to C906, C807 to C907, C808 to C908, IC801 to IC901, IC802 to IC902, IC803 to IC903, L801 to L901, Q801 to Q901, Q802 to Q902, R801 to R901, R802 to R902, R803 to R903, R804 to R904, R805 to R905, R806 to R906, R807 to R907, R808 to R908, R809 to R909, TH801 to TH901, TP801 to TP901, TP802 to TP902, TP803 to TP903, TP804 to TP904, TP805 to TP905
Connections:
- net +BATT renamed V_{Batt}

Commit message: Improving Thread
- Add boot signal for Thread MCU
- Add debug LED for nRF5340
Parts:
- TP901, TP902, TP903, TP904, TP905: value ~ -> (none)
Changed lines of the file:
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@@
 			)
 		)
-		(property "Value" "~"
+		(property "Value" ""
 			(at 252.73 94.615 0)
 			(show_name no)
@@
 			)
 		)
-		(property "Value" "~"
+		(property "Value" ""
 			(at 238.76 94.615 0)
 			(show_name no)
@@
 			)
 		)
-		(property "Value" "~"
+		(property "Value" ""
 			(at 269.24 186.055 0)
 			(show_name no)
@@
 			)
 		)
-		(property "Value" "~"
+		(property "Value" ""
 			(at 209.55 103.505 0)
 			(show_name no)
@@
 			)
 		)
-		(property "Value" "~"
+		(property "Value" ""
 			(at 168.91 130.175 0)
 			(show_name no)
