File: gateway/Battery.kicad_sch (KiCad schematic)
At the start: 30 parts, among them IC901 BQ25308, IC902 MAX17048, IC903 BQ297xy, Q901 Si2342DS, Q902 Si2342DS

Commit message: Working on PCB
Parts:
- BAT901: value Backup Power -> Backup Battery
- TP901, TP902, TP903, TP904, TP905: value (none) -> ~
Other:
- moved on the sheet: BAT901, C901, C902, C903, C904, C905, C906, C907, C908, IC901, IC902, IC903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

Commit message: Working on layout
Parts:
- removed TP904: ~, Testpoints_Kampi:TestPoint_Pad_1.0x1.0mm, symbol Connector:TestPoint
Connections:
- net V_{Batt}: now also TP903.1
- net at IC903.2 (Cout), Q901.1 (G): no longer TP903.1
Changed lines of the file:
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@@
-	)
-	(junction
-		(at 224.79 115.57)
-		(diameter 0)
-		(color 0 0 0 0)
 	)
 	(junction
@@
 		(color 0 0 0 0)
 	)
-	(junction
-		(at 238.76 120.65)
-		(diameter 0)
-		(color 0 0 0 0)
-	)
 	(bus_entry
 		(at 196.85 185.42)
@@
 		)
 	)
-	(wire
-		(pts
-			(xy 224.79 107.95) (xy 224.79 115.57)
-		)
-		(stroke
-			(width 0)
-			(type default)
-		)
-	)
 	(polyline
 		(pts
@@
 	(wire
 		(pts
-			(xy 238.76 107.95) (xy 238.76 120.65)
-		)
-		(stroke
-			(width 0)
-			(type default)
-		)
-	)
-	(wire
-		(pts
 			(xy 99.06 127) (xy 99.06 132.08)
 		)
@@
 		(pts
 			(xy 262.89 129.54) (xy 262.89 130.81)
+		)
+		(stroke
+			(width 0)
+			(type default)
+		)
+	)
+	(wire
+		(pts
+			(xy 191.77 82.55) (xy 191.77 83.82)
 		)
 		(stroke
@@
 	)
 	(symbol
-		(lib_id "Connector:TestPoint")
-		(at 238.76 107.95 0)
-		(unit 1)
-		(body_style 1)
-		(exclude_from_sim no)
-		(in_bom no)
-		(on_board yes)
-		(in_pos_files no)
-		(dnp no)
-		(property "Reference" "TP904"
-			(at 238.76 100.33 0)
-			(show_name no)
-			(do_not_autoplace no)
-			(effects
-				(font
-					(size 1.27 1.27)
-				)
-			)
-		)
-		(property "Value" "~"
-			(at 238.76 102.235 0)
-			(show_name no)
-			(do_not_autoplace no)
-			(effects
-				(font
-					(size 1.27 1.27)
-				)
-			)
-		)
-		(property "Footprint" "Testpoints_Kampi:TestPoint_Pad_1.0x1.0mm"
-			(at 243.84 107.95 0)
-			(hide yes)
-			(show_name no)
-			(do_not_autoplace no)
-			(effects
-				(font
-					(size 1.27 1.27)
-				)
-			)
-		)
-		(property "Datasheet" ""
-			(at 243.84 107.95 0)
-			(hide yes)
-			(show_name no)
-			(do_not_autoplace no)
-			(effects
-				(font
-					(size 1.27 1.27)
-				)
-			)
-		)
-		(property "Description" "test point"
-			(at 238.76 107.95 0)
-			(hide yes)
-			(show_name no)
-			(do_not_autoplace no)
-			(effects
-				(font
-					(size 1.27 1.27)
-				)
-			)
-		)
-		(property "manf" ""
-			(at 238.76 107.95 0)
-			(hide yes)
-			(show_name no)
-			(do_not_autoplace no)
-			(effects
-				(font
-					(size 1.27 1.27)
-				)
-			)
-		)
-		(property "manf#" ""
-			(at 238.76 107.95 0)
-			(hide yes)
-			(show_name no)
-			(do_not_autoplace no)
-			(effects
-				(font
-					(size 1.27 1.27)
-				)
-			)
-		)
-		(property "mouser#" ""
-			(at 238.76 107.95 0)
-			(hide yes)
-			(show_name no)
-			(do_not_autoplace no)
-			(effects
-				(font
-					(size 1.27 1.27)
-				)
-			)
-		)
-		(pin "1"
-		)
-		(instances
-			(project "Gateway"
-				(path "/d5742f03-3b1a-42e5-a384-018bd4b919aa/c5103ceb-5325-4a84-a025-9638a412984e/a382d3a7-1839-425a-ad98-cfb69b49aae1"
-					(reference "TP904")
-					(unit 1)
-				)
-			)
-		)
-	)
-	(symbol
 		(lib_id "power:GND")
 		(at 195.58 132.08 0)
@@
 				(path "/d5742f03-3b1a-42e5-a384-018bd4b919aa/c5103ceb-5325-4a84-a025-9638a412984e/a382d3a7-1839-425a-ad98-cfb69b49aae1"
 					(reference "#PWR0912")
-					(unit 1)
-				)
-			)
-		)
-	)
-	(symbol
-		(lib_id "Connector:TestPoint")
-		(at 224.79 107.95 0)
-		(unit 1)
-		(body_style 1)
-		(exclude_from_sim no)
-		(in_bom no)
-		(on_board yes)
-		(in_pos_files no)
-		(dnp no)
-		(property "Reference" "TP903"
-			(at 224.79 100.33 0)
-			(show_name no)
-			(do_not_autoplace no)
-			(effects
-				(font
-					(size 1.27 1.27)
-				)
-			)
-		)
-		(property "Value" "~"
-			(at 224.79 102.235 0)
-			(show_name no)
-			(do_not_autoplace no)
-			(effects
-				(font
-					(size 1.27 1.27)
-				)
-			)
-		)
-		(property "Footprint" "Testpoints_Kampi:TestPoint_Pad_1.0x1.0mm"
-			(at 229.87 107.95 0)
-			(hide yes)
-			(show_name no)
-			(do_not_autoplace no)
-			(effects
-				(font
-					(size 1.27 1.27)
-				)
-			)
-		)
-		(property "Datasheet" ""
-			(at 229.87 107.95 0)
-			(hide yes)
-			(show_name no)
-			(do_not_autoplace no)
-			(effects
-				(font
-					(size 1.27 1.27)
-				)
-			)
-		)
-		(property "Description" "test point"
-			(at 224.79 107.95 0)
-			(hide yes)
-			(show_name no)
-			(do_not_autoplace no)
-			(effects
-				(font
-					(size 1.27 1.27)
-				)
-			)
-		)
-		(property "manf" ""
-			(at 224.79 107.95 0)
-			(hide yes)
-			(show_name no)
-			(do_not_autoplace no)
-			(effects
-				(font
-					(size 1.27 1.27)
-				)
-			)
-		)
-		(property "manf#" ""
-			(at 224.79 107.95 0)
-			(hide yes)
-			(show_name no)
-			(do_not_autoplace no)
-			(effects
-				(font
-					(size 1.27 1.27)
-				)
-			)
-		)
-		(property "mouser#" ""
-			(at 224.79 107.95 0)
-			(hide yes)
-			(show_name no)
-			(do_not_autoplace no)
-			(effects
-				(font
-					(size 1.27 1.27)
-				)
-			)
-		)
-		(pin "1"
-		)
-		(instances
-			(project "Gateway"
-				(path "/d5742f03-3b1a-42e5-a384-018bd4b919aa/c5103ceb-5325-4a84-a025-9638a412984e/a382d3a7-1839-425a-ad98-cfb69b49aae1"
-					(reference "TP903")
 					(unit 1)
 				)
@@
 					(unit 1)
 				)
+			)
+		)
+	)
+	(symbol
+		(lib_id "Connector:TestPoint")
+		(at 191.77 82.55 0)
+		(unit 1)
+		(body_style 1)
+		(exclude_from_sim no)
+		(in_bom no)
+		(on_board yes)
+		(in_pos_files no)
+		(dnp no)
+		(property "Reference" "TP903"
+			(at 191.77 74.93 0)
+			(show_name no)
+			(do_not_autoplace no)
+			(effects
+				(font
+					(size 1.27 1.27)
+				)
+			)
+		)
+		(property "Value" "~"
+			(at 191.77 76.835 0)
+			(show_name no)
+			(do_not_autoplace no)
+			(effects
+				(font
+					(size 1.27 1.27)
+				)
+			)
+		)
+		(property "Footprint" "Testpoints_Kampi:TestPoint_Pad_1.0x1.0mm"
+			(at 196.85 82.55 0)
+			(hide yes)
+			(show_name no)
+			(do_not_autoplace no)
+			(effects
+				(font
+					(size 1.27 1.27)
+				)
+			)
+		)
+		(property "Datasheet" ""
+			(at 196.85 82.55 0)
+			(hide yes)
+			(show_name no)
+			(do_not_autoplace no)
+			(effects
+				(font
+					(size 1.27 1.27)
+				)
+			)
+		)
+		(property "Description" "test point"
+			(at 191.77 82.55 0)
+			(hide yes)
+			(show_name no)
+			(do_not_autoplace no)
+			(effects
+				(font
+					(size 1.27 1.27)
+				)
+			)
+		)
+		(property "manf" ""
+			(at 191.77 82.55 0)
+			(hide yes)
+			(show_name no)
+			(do_not_autoplace no)
+			(effects
+				(font
+					(size 1.27 1.27)
+				)
+			)
+		)
+		(property "manf#" ""
+			(at 191.77 82.55 0)
+			(hide yes)
+			(show_name no)
+			(do_not_autoplace no)
+			(effects
+				(font
+					(size 1.27 1.27)
+				)
+			)
+		)
+		(property "mouser#" ""
+			(at 191.77 82.55 0)
+			(hide yes)
+			(show_name no)
+			(do_not_autoplace no)
+			(effects
+				(font
+					(size 1.27 1.27)
+				)
+			)
+		)
+		(pin "1"
+		)
+		(instances
+			(project "Gateway"
+				(path "/d5742f03-3b1a-42e5-a384-018bd4b919aa/c5103ceb-5325-4a84-a025-9638a412984e/a382d3a7-1839-425a-ad98-cfb69b49aae1"
+					(reference "TP903")
+					(unit 1)
+				)

Commit message: Working on layout
Parts:
- removed Q901, Q902: Si2342DS, Package_TO_SOT_SMD:SOT-23, symbol Vishay:Si2342DS
- added Q901, Q902: CSD16301Q2, Package_SON:Texas_DQK, symbol Transistor_FET:CSD16301Q2
- added R910, R911: 5M1, Resistor_SMD:R_0402_1005Metric, symbol Device:R
- R907: footprint Resistor_SMD:R_0805_2012Metric -> Resistor_SMD:R_0402_1005Metric; manf# CR0805-JW-222GLF -> CR0402-JW-222GLF; mouser# 652-CR0805-JW-222GLF -> 652-CR0402-JW-222GLF
Connections:
- net GND: now also Q901.4 (S), Q901.7 (S), R910.1
- net at IC903.2 (Cout): now also Q901.3 (G), R910.2
- net at IC903.3 (Dout): now also Q902.3 (G), R911.2
- net at BAT901.2 (-), C907.2, C908.2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: now also Q902.4 (S), Q902.7 (S), R911.1
- new net: Q901.1 (D), Q901.2 (D), Q901.5 (D), Q901.6 (D), Q901.8 (D), Q902.1 (D), Q902.2 (D), Q902.5 (D), Q902.6 (D), Q902.8 (D)
Other:
- moved on the sheet: C901, C902, C903, C904, C905, IC901, L901, R901, R902, R903, R904, R905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

Commit message: Working on layout
Parts:
- R907: footprint Resistor_SMD:R_0402_1005Metric -> Resistor_SMD:R_0805_2012Metric; manf# CR0402-JW-222GLF -> CR0805-JW-222ELF; mouser# 652-CR0402-JW-222GLF -> 652-CR0805-JW-222ELF
- R910, R911: footprint Resistor_SMD:R_0402_1005Metric -> Resistor_SMD:R_0805_2012Metric; manf# RC0402JR-075M1L -> RC0805JR-075M1L; mouser# 603-RC0402JR-075M1L -> 603-RC0805JR-075M1L
Other:
- moved on the sheet: BAT901, C901, C902, C903, C904, C905, C906, C907, C908, IC901, IC902, IC903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

Commit message: Replace battery charger with BQ25300
Parts:
- IC901: value BQ25308 -> BQ25300; symbol Texas Instruments:BQ25308 -> Texas Instruments:BQ25300; manf# BQ25308RTER -> BQ25300RTER; mouser# 595-BQ25308RTER -> 595-BQ25300RTER
Connections:
- net ~{Battery-Charge-Enable} renamed Battery-Charge-Enable
Changed lines of the file:
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@@
 		)
 	)
-	(hierarchical_label "~{Battery-Charge-Enable}"
+	(hierarchical_label "Battery-Charge-Enable"
 		(shape input)
 		(at 50.8 93.98 180)
@@
 	)
 	(symbol
-		(lib_id "Texas Instruments:BQ25308")
+		(lib_id "Texas Instruments:BQ25300")
 		(at 100.33 107.95 0)
 		(unit 1)
@@
 			)
 		)
-		(property "Value" "BQ25308"
+		(property "Value" "BQ25300"
 			(at 94.615 123.19 0)
 			(show_name no)
@@
 			)
 		)
-		(property "Datasheet" "https://www.ti.com/lit/ds/symlink/bq25308.pdf?ts=1719898702995&ref_url=https%253A%252F%252Fwww.mouser.in%252F"
+		(property "Datasheet" "https://www.ti.com/lit/ds/symlink/bq25300.pdf"
 			(at 127 292.71 0)
 			(hide yes)
@@
 			)
 		)
-		(property "Description" "Battery Management Standalone, 1-cell 17V 3A battery charger with dead-battery charge inhibit feature"
+		(property "Description" "Battery Management Standalone, 1-cell 17V 3A battery charger"
 			(at 100.33 107.95 0)
 			(hide yes)
@@
 			)
 		)
-		(property "manf#" "BQ25308RTER"
+		(property "manf#" "BQ25300RTER"
 			(at 100.33 107.95 0)
 			(hide yes)
@@
 			)
 		)
-		(property "mouser#" "595-BQ25308RTER"
+		(property "mouser#" "595-BQ25300RTER"
 			(at 100.33 107.95 0)
 			(hide yes)

Commit message: Working on revision 1.0.0
Parts:
- added C909: 220p, Capacitor_SMD:C_0805_2012Metric, symbol Device:C
- added IC904: TPS22965, Package_SON:WSON-8-1EP_2x2mm_P0.5mm_EP0.9x1.6mm_ThermalVias, symbol Texas Instruments:TPS22965
- added R912: 100k, Resistor_SMD:R_0805_2012Metric, symbol partdb:RT0805FRE13100KL
- C901, C905: symbol Device:C -> partdb:0805X7R106KT1AT; Category (none) -> Kondensator/MLCC; MPN (none) -> 0805X7R106KT1AT; Manufacturer (none) -> KYOCERA AVX; Manufacturing Status (none) -> Active; Mouser SPN (none) -> 581-0805X7R106KT1AT; Part-DB Footprint (none) -> 0805; Part-DB ID (none) -> 331; Part-DB URL (none) -> https://inventory.lan/de/part/331/info; Stock (none) -> 0
- C902, C903: symbol Device:C -> partdb:MCJCT21GCB7225MTPA1J; Category (none) -> Kondensator/MLCC; MPN (none) -> MCJCT21GCB7225MTPA1J; Manufacturer (none) -> TAIYO YUDEN; Manufacturing Status (none) -> Active; Mouser SPN (none) -> 963-T21GCB7225MTPA1J; Part-DB Footprint (none) -> 0805; Part-DB ID (none) -> 328; Part-DB URL (none) -> https://inventory.lan/de/part/328/info; Stock (none) -> 0; manf KYOCERA AVX -> TAIYO YUDEN; manf# 0805ZC225JAT2A -> MCJCT21GCB7225MTPA1J; mouser# 581-0805ZC225JAT2A -> 963-T21GCB7225MTPA1J
- C906, C907: symbol Device:C -> partdb:08055C104K4Z4A; Category (none) -> Kondensator/MLCC; MPN (none) -> 08055C104K4Z4A; Manufacturer (none) -> KYOCERA AVX; Manufacturing Status (none) -> Active; Mass (none) -> 0.006 g; Mouser SPN (none) -> 581-08055C104K4Z4A; Part-DB Footprint (none) -> 0805; Part-DB ID (none) -> 109; Part-DB URL (none) -> https://inventory.lan/de/part/109/info; Stock (none) -> 6; Storage Location (none) -> Sortierregal; manf# 08053C104M4T4A -> 08055C104K4Z4A; mouser# 581-08053C104M4T4A -> 581-08055C104K4Z4A
- R901, R904, R908: symbol Device:R -> partdb:RT0805FRE13100KL; Category (none) -> Widerstand/Dünnfilmwiderstand; MPN (none) -> RT0805FRE13100KL; Manufacturer (none) -> YAGEO; Manufacturing Status (none) -> Active; Mass (none) -> 0.006 g; Mouser SPN (none) -> 603-RT0805FRE13100KL; Part-DB Footprint (none) -> 0805; Part-DB ID (none) -> 66; Part-DB URL (none) -> https://inventory.lan/de/part/66/info; Stock (none) -> 4; Storage Location (none) -> Sortierregal; manf Bourns -> YAGEO; manf# CR0805-JW-104GLF -> RT0805FRE13100KL; mouser# 652-CR0805-JW-104GLF -> 603-RT0805FRE13100KL
- R902: symbol Device:R -> partdb:CR0805-J/-000ELF; Category (none) -> Widerstand/Dickfilmwiderstand; MPN (none) -> CR0805-J/-000ELF; Manufacturer (none) -> Bourns; Manufacturing Status (none) -> Active; Mass (none) -> 0.006 g; Mouser SPN (none) -> 652-CR0805-J/-000ELF; Part-DB Footprint (none) -> 0805; Part-DB ID (none) -> 322; Part-DB URL (none) -> https://inventory.lan/de/part/322/info; Stock (none) -> 0
- R907: symbol Device:R -> partdb:CR0805-JW-222ELF; Category (none) -> Widerstand/Dickfilmwiderstand; MPN (none) -> CR0805-JW-222ELF; Manufacturer (none) -> Bourns; Manufacturing Status (none) -> Active; Mass (none) -> 0.006 g; Mouser SPN (none) -> 652-CR0805JW-222ELF; Part-DB Footprint (none) -> 0805; Part-DB ID (none) -> 72; Part-DB URL (none) -> https://inventory.lan/de/part/72/info; Stock (none) -> 50; Storage Location (none) -> Sortierregal; mouser# 652-CR0805-JW-222ELF -> 652-CR0805JW-222ELF
- R909: symbol Device:R -> partdb:CR0805-JW-331ELF; Category (none) -> Widerstand/Dickfilmwiderstand; MPN (none) -> CR0805-JW-331ELF; Manufacturer (none) -> Bourns; Manufacturing Status (none) -> Active; Mass (none) -> 0.006 g; Mouser SPN (none) -> 652-CR0805JW-331ELF; Part-DB Footprint (none) -> 0805; Part-DB ID (none) -> 323; Part-DB URL (none) -> https://inventory.lan/de/part/323/info; Stock (none) -> 0; manf# CR0805-JW-331GLF -> CR0805-JW-331ELF; mouser# 652-CR0805-JW-331GLF -> 652-CR0805JW-331ELF
Connections:
- net GND: now also C909.2, IC904.5 (GND), IC904.9 (PAD), R912.2
- net V_{Batt}: now also IC904.7 (VOUT), IC904.8 (VOUT); no longer BAT901.1 (+), C905.1, C906.1, C908.1, IC901.10 (BAT), IC902.2 (CELL), IC902.3 (VDD), L901.2, R909.1
- new net: BAT901.1 (+), C905.1, C906.1, C908.1, IC901.10 (BAT), IC902.2 (CELL), IC902.3 (VDD), IC904.1 (VIN), IC904.2 (VIN), IC904.4 (VBIAS), L901.2, R909.1
- new net: C909.1, IC904.6 (CT)
- new net Battery-Backup-Enable: IC904.3 (ON), R912.1
Other:
- moved on the sheet: C904, C905, C906, IC902, L901, Q901, Q902, R907, R908, R910, R911, TP903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
