File: gateway/Battery.kicad_sch (KiCad schematic)
At the start: 34 parts, among them IC901 BQ25300, IC902 MAX17048, IC903 BQ297xy, IC904 TPS22965, Q901 CSD16301Q2, Q902 CSD16301Q2

Commit message: Prepare Release 1.0.0
Co-Authored-By: Claude Opus 5.5 <noreply@anthropic.com>
Parts:
- R803: renamed from R903; mouser# 652-CR0805-JW-183GLF -> 652-CR0805JW-183GLF
- R806: renamed from R905; mouser# 652-CR0805-FX-4531GLF -> 652-CR0805FX-4531GLF
- R807: renamed from R906; mouser# 652-CR0805-FX-2262GLF -> 652-CR0805FX-2262GLF
- TH801: renamed from TH901; mouser# 652-CR0805-JW-103GLF -> 652-CR0805JW-103GLF
- renumbered BAT901 to BAT801, C901 to C801, C902 to C802, C903 to C803, C904 to C804, C905 to C805, C909 to C806, C906 to C807, C907 to C808, C908 to C809, IC901 to IC801, IC904 to IC802, IC902 to IC803, IC903 to IC804, L901 to L801, Q901 to Q801, Q902 to Q802, R901 to R801, R902 to R802, R904 to R804, R912 to R805, R907 to R808, R910 to R809, R911 to R810, R908 to R811, R909 to R812, TP901 to TP801, TP902 to TP802, TP903 to TP803, TP905 to TP804
