File: gateway/Power.kicad_sch (KiCad schematic)
At the start: 62 parts, among them IC701 LM62460, IC702 ADP1614ACPZ-R7, IC703 TPS2121RUXT, IC704 MIC5317-3.3xM5, IC705 MIC5317-1.8xM5, Q701 BSS123, X701 7-16 V

Commit message: Add INA219 for current measurement
Parts:
- removed F701: 3 A, symbol Device:Fuse
- removed TP706: ~, Testpoints_Kampi:TestPoint_Pad_1.0x1.0mm, symbol Connector:TestPoint
- removed X701: 7-16 V, Connector_BarrelJack:BarrelJack_Wuerth_6941xx301002, symbol Connector:Barrel_Jack
- renumbered C701 to C801, C702 to C802, C703 to C803, C704 to C804, C705 to C805, C706 to C806, C707 to C807, C708 to C808, C709 to C809, C710 to C810, C711 to C811, C712 to C812, C713 to C813, C714 to C814, C715 to C815, C716 to C816, C717 to C817, C718 to C818, C719 to C819, C720 to C820, C721 to C821, D701 to D801, IC701 to IC801, IC702 to IC802, IC703 to IC803, IC704 to IC804, IC705 to IC805, L701 to L801, L702 to L802, Q701 to Q801, R701 to R801, R702 to R802, R703 to R803, R704 to R804, R705 to R805, R706 to R806, R707 to R807, R708 to R808, R709 to R809, R710 to R810, R711 to R811, R712 to R812, R713 to R813, R714 to R814, R715 to R815, R716 to R816, R717 to R817, R718 to R818, TP701 to TP801, TP702 to TP802, TP703 to TP803, TP704 to TP804, TP705 to TP805, TP707 to TP806, TP708 to TP807, TP709 to TP808, TP710 to TP809, TP711 to TP810, TP712 to TP811
Connections:
- net +BATT renamed V_{Batt}
Other:
- moved on the sheet: TP805
