File: gateway/Power.kicad_sch (KiCad schematic)
At the start: 66 parts, among them IC801 LM62460, IC802 ADP1614ACPZ-650-R7, IC803 TPS2121RUXT, IC804 TLV75733PDBV, IC805 TLV75733PDBV, Q801 BSS123

Commit message: Working on revision 1.0.0
Parts:
- C801, C802, C807, C815, C817, C825: symbol Device:C -> partdb:0805X7R106KT1AT; Category (none) -> Kondensator/MLCC; MPN (none) -> 0805X7R106KT1AT; Manufacturer (none) -> KYOCERA AVX; Manufacturing Status (none) -> Active; Mouser SPN (none) -> 581-0805X7R106KT1AT; Part-DB Footprint (none) -> 0805; Part-DB ID (none) -> 331; Part-DB URL (none) -> https://inventory.lan/de/part/331/info; Stock (none) -> 0
- C803, C819, C821, C822, C823: symbol Device:C -> partdb:08053G105MAT2A; Category (none) -> Kondensator/MLCC; MPN (none) -> 08053G105MAT2A; Manufacturer (none) -> KYOCERA AVX; Manufacturing Status (none) -> Active; Mass (none) -> 0.006 g; Mouser SPN (none) -> 581-08053G105MAT2A; Part-DB Footprint (none) -> 0805; Part-DB ID (none) -> 349; Part-DB URL (none) -> https://inventory.lan/de/part/349/info; Stock (none) -> 0; manf# 08056C105MAT2A -> 08053G105MAT2A; mouser# 581-08056C105MAT2A -> 581-08053G105MAT2A
- C805, C806: symbol Device:C -> partdb:08055C474K4Z2A; Category (none) -> Kondensator/MLCC; MPN (none) -> 08055C474K4Z2A; Manufacturer (none) -> KYOCERA AVX; Manufacturing Status (none) -> Active; Mass (none) -> 0.006 g; Mouser SPN (none) -> 581-08055C474K4Z2A; Part-DB Footprint (none) -> 0805; Part-DB ID (none) -> 329; Part-DB URL (none) -> https://inventory.lan/de/part/329/info; Stock (none) -> 0; manf# 08053C474K4T4A -> 08055C474K4Z2A; mouser# 581-08053C474K4T4A -> 581-08055C474K4Z2A
- C808, C824: symbol Device:C -> partdb:08055C104K4Z4A; Category (none) -> Kondensator/MLCC; MPN (none) -> 08055C104K4Z4A; Manufacturer (none) -> KYOCERA AVX; Manufacturing Status (none) -> Active; Mass (none) -> 0.006 g; Mouser SPN (none) -> 581-08055C104K4Z4A; Part-DB Footprint (none) -> 0805; Part-DB ID (none) -> 109; Part-DB URL (none) -> https://inventory.lan/de/part/109/info; Stock (none) -> 6; Storage Location (none) -> Sortierregal; manf# 08053C104M4T4A -> 08055C104K4Z4A; mouser# 581-08053C104M4T4A -> 581-08055C104K4Z4A
- C809, C811, C813, C814: symbol Device:C -> partdb:MLAST21GBB5226MTNC12; Category (none) -> Kondensator/MLCC; MPN (none) -> MLAST21GBB5226MTNC12; Manufacturer (none) -> TAIYO YUDEN; Manufacturing Status (none) -> Active; Mouser SPN (none) -> 963-MLAST21GBB5226MT; Part-DB Footprint (none) -> 0805; Part-DB ID (none) -> 330; Part-DB URL (none) -> https://inventory.lan/de/part/330/info; Stock (none) -> 0; manf KYOCERA AVX -> TAIYO YUDEN; manf# KGM21AR51A226MU -> MLAST21GBB5226MTNC12; mouser# 581-KGM21AR51A226MU -> 963-MLAST21GBB5226MT
- Q801: value BSS123 -> BSS138; symbol Transistor_FET:BSS123 -> partdb:BSS138; Category (none) -> Transistor/N-Kanal; MPN (none) -> BSS138; Manufacturer (none) -> onsemi / Fairchild; Manufacturing Status (none) -> Active; Mass (none) -> 0.008 g; Mouser SPN (none) -> 512-BSS138; Part-DB Footprint (none) -> SOT-23-3; Part-DB ID (none) -> 353; Part-DB URL (none) -> https://inventory.lan/de/part/353/info; Stock (none) -> 0; manf onsemi -> onsemi / Fairchild; manf# BSS123 -> BSS138; mouser# 512-BSS123 -> 512-BSS138
- R801, R805, R813, R823, R824: symbol Device:R -> partdb:CR0805-FX-1002ELF; Category (none) -> Widerstand/Dickfilmwiderstand; MPN (none) -> CR0805-FX-1002ELF; Manufacturer (none) -> Bourns; Manufacturing Status (none) -> Active; Mass (none) -> 0.006 g; Mouser SPN (none) -> 652-CR0805FX-1002ELF; Part-DB Footprint (none) -> 0805; Part-DB ID (none) -> 343; Part-DB URL (none) -> https://inventory.lan/de/part/343/info; Stock (none) -> 0; manf# CR0805-JW-103GLF -> CR0805-FX-1002ELF; mouser# 652-CR0805-JW-103GLF -> 652-CR0805FX-1002ELF
- R806: symbol Device:R -> partdb:RT0805FRE13100KL; Category (none) -> Widerstand/Dünnfilmwiderstand; MPN (none) -> RT0805FRE13100KL; Manufacturer (none) -> YAGEO; Manufacturing Status (none) -> Active; Mass (none) -> 0.006 g; Mouser SPN (none) -> 603-RT0805FRE13100KL; Part-DB Footprint (none) -> 0805; Part-DB ID (none) -> 66; Part-DB URL (none) -> https://inventory.lan/de/part/66/info; Stock (none) -> 4; Storage Location (none) -> Sortierregal; manf Bourns -> YAGEO; manf# CR0805-JW-104GLF -> RT0805FRE13100KL; mouser# 652-CR0805-JW-104GLF -> 603-RT0805FRE13100KL
- R817: symbol Device:R -> partdb:CR0805-FX-1002ELF; Category (none) -> Widerstand/Dickfilmwiderstand; MPN (none) -> CR0805-FX-1002ELF; Manufacturer (none) -> Bourns; Manufacturing Status (none) -> Active; Mass (none) -> 0.006 g; Mouser SPN (none) -> 652-CR0805FX-1002ELF; Part-DB Footprint (none) -> 0805; Part-DB ID (none) -> 343; Part-DB URL (none) -> https://inventory.lan/de/part/343/info; Stock (none) -> 0; manf# CR0805-FX-1002GLF -> CR0805-FX-1002ELF; mouser# 652-CR0805-FX-1002GLF -> 652-CR0805FX-1002ELF
- R818, R819: symbol Device:R -> partdb:CR0805-J/-000ELF; Category (none) -> Widerstand/Dickfilmwiderstand; MPN (none) -> CR0805-J/-000ELF; Manufacturer (none) -> Bourns; Manufacturing Status (none) -> Active; Mass (none) -> 0.006 g; Mouser SPN (none) -> 652-CR0805-J/-000ELF; Part-DB Footprint (none) -> 0805; Part-DB ID (none) -> 322; Part-DB URL (none) -> https://inventory.lan/de/part/322/info; Stock (none) -> 0
- R821: symbol Device:R -> partdb:RC0805FR-071ML; Category (none) -> Widerstand/Dickfilmwiderstand; MPN (none) -> RC0805FR-071ML; Manufacturer (none) -> YAGEO; Manufacturing Status (none) -> Active; Mass (none) -> 0.0055 g; Mouser SPN (none) -> 603-RC0805FR-071ML; Part-DB Footprint (none) -> 0805; Part-DB ID (none) -> 370; Part-DB URL (none) -> https://inventory.lan/de/part/370/info; Stock (none) -> 0
Other:
- moved on the sheet: C821, TP809
