File: gateway/Power.kicad_sch (KiCad schematic)
At the start: 59 parts, among them IC801 LM62460, IC802 ADP1614ACPZ-R7, IC803 TPS2121RUXT, IC804 MIC5317-3.3xM5, IC805 MIC5317-1.8xM5, Q801 BSS123

Commit message: Push outputs from CI/CD (2026-07-09 20:18:55)
Parts:
- removed TP805: ~, Testpoints_Kampi:TestPoint_Pad_1.0x1.0mm, symbol Connector:TestPoint
- added C822, C823: 10u, Capacitor_SMD:C_0805_2012Metric, symbol Device:C
- added TP812: (no value), Testpoints_Kampi:TestPoint_Pad_1.0x1.0mm, symbol Connector:TestPoint
- IC802: value ADP1614ACPZ-R7 -> ADP1614ACPZ-650-R7; manf# ADP1614ACPZ-R7 -> ADP1614ACPZ-650-R7; mouser# 584-ADP1614ACPZ-R7 -> 584-ADP1614ACPZ-650-R7
- R802: value 0R -> 66k5; manf Bourns -> YAGEO; manf# CR0805-J/-000ELF -> RT0805BRD0766K5L; mouser# 652-CR0805-J/-000ELF -> 603-RT0805BRD0766K5L
Connections:
- net GND: now also C822.2, C823.2
- net V_{Backup}: now also C822.1, C823.1, TP812.1

Commit message: Improving Thread
- Add boot signal for Thread MCU
- Add debug LED for nRF5340
Parts:
- TP801, TP802, TP803, TP804, TP806, TP807, TP808, TP809, TP810, TP811: value ~ -> (none)
Changed lines of the file:
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@@
 			)
 		)
-		(property "Value" "~"
+		(property "Value" ""
 			(at 102.87 117.3479 0)
 			(show_name no)
@@
 			)
 		)
-		(property "Datasheet" "https://www.mouser.de/datasheet/3/5926/1/X7RDielectric.pdf"
+		(property "Datasheet" "https://datasheets.kyocera-avx.com/C0GNP0-KGM.pdf"
 			(at 113.03 234.95 0)
 			(hide yes)
@@
 			)
 		)
-		(property "Value" "~"
+		(property "Value" ""
 			(at 397.51 207.5179 0)
 			(show_name no)
@@
 			)
 		)
-		(property "Value" "~"
+		(property "Value" ""
 			(at 314.96 203.7079 0)
 			(show_name no)
@@
 			)
 		)
-		(property "Value" "~"
+		(property "Value" ""
 			(at 257.81 153.035 0)
 			(show_name no)
@@
 			)
 		)
-		(property "Value" "~"
+		(property "Value" ""
 			(at 339.09 137.6679 0)
 			(show_name no)
@@
 			)
 		)
-		(property "Value" "~"
+		(property "Value" ""
 			(at 46.99 197.485 0)
 			(show_name no)
@@
 			)
 		)
-		(property "Value" "~"
+		(property "Value" ""
 			(at 60.96 89.4079 0)
 			(show_name no)
@@
 			)
 		)
-		(property "Value" "~"
+		(property "Value" ""
 			(at 257.81 123.825 0)
 			(show_name no)
@@
 			)
 		)
-		(property "Value" "~"
+		(property "Value" ""
 			(at 24.13 130.3019 0)
 			(show_name no)
@@
 			)
 		)
-		(property "Value" "~"
+		(property "Value" ""
 			(at 290.83 107.315 0)
 			(show_name no)

Commit message: Working on PCB
Parts:
- removed IC804: MIC5317-3.3xM5, Package_TO_SOT_SMD:SOT-23-5, symbol Regulator_Linear:MIC5317-3.3xM5
- removed IC805: MIC5317-1.8xM5, Package_TO_SOT_SMD:SOT-23-5, symbol Regulator_Linear:MIC5317-1.8xM5
- added IC804, IC805: TLV75733PDBV, Package_TO_SOT_SMD:SOT-23-5, symbol Regulator_Linear:TLV75733PDBV
- TP801, TP802, TP803, TP804, TP806, TP807, TP808, TP809, TP810, TP811: value (none) -> ~
- TP805: renamed from TP812; value (none) -> ~
- renumbered C822 to C815, C815 to C816, C823 to C817, C816 to C818, C817 to C819, C818 to C820, C819 to C821, C820 to C822, C821 to C823
Connections:
- net +1V8: now also IC805.5 (OUT)
- net +3V3: now also IC804.5 (OUT)
- net +5V: now also IC804.1 (IN), IC805.1 (IN)
- net GND: now also IC804.2 (GND), IC805.2 (GND)
- net SoM-Power-Enable: now also IC804.3 (EN), IC805.3 (EN)
- net PowerMux-Status renamed Backup-Status

Commit message: Working on layout
Parts:
- removed R810, R812: 5k1, Resistor_SMD:R_0805_2012Metric, symbol Device:R
- removed R811: 21k, Resistor_SMD:R_0805_2012Metric, symbol Device:R
- removed R814: 51k1, Resistor_SMD:R_0805_2012Metric, symbol Device:R
- removed TP802, TP803, TP806, TP807: ~, Testpoints_Kampi:TestPoint_Pad_1.0x1.0mm, symbol Connector:TestPoint
- added R819: 0R, Resistor_SMD:R_0805_2012Metric, symbol Device:R
- C816: value 22u -> (none); manf KYOCERA AVX -> (none); manf# KGM21AR51A226MU -> (none); mouser# 581-KGM21AR51A226MU -> (none); now not fitted; now left out of the parts list
- R809: value 21k -> 27k; manf# CR0805-FX-2102GLF -> CR0805-JW-273ELF; mouser# 652-CR0805-FX-2102GLF -> 652-CR0805-JW-273ELF
Connections:
- net GND: now also IC803.4 (OV2), IC803.5 (OV1), R809.2, R819.1
- net at C818.1, IC801.7 (FB), R806.2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: no longer IC801.5 (BIAS)
- net at C809.2, C811.2, C813.2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: now also IC801.5 (BIAS); no longer R809.1
- net at IC803.10 (ILIM): now also R809.1
- net at C803.2, IC801.6 (VCC), IC801.9 (RT): no longer IC801.11 (SpSp)
- net V_{Backup}: no longer names the net of C815.1, C817.1, D801.1 (K), IC803.2 (IN2), R804.1, TP805.1
- new net: IC801.11 (SpSp), R819.2
Other:
- moved on the sheet: C802, C803, C805, C806, C807, C808, C809, C811, C813, C814, C818, IC801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

Commit message: Working on layout
Parts:
- removed C820: 10n, Capacitor_SMD:C_0805_2012Metric, symbol Device:C
- removed TP808, TP810: ~, Testpoints_Kampi:TestPoint_Pad_1.0x1.0mm, symbol Connector:TestPoint
- added C820: 220u, Capacitor_Tantalum_SMD:CP_EIA-7343-31_Kemet-D, symbol Device:C_Polarized
- added C824: 100n, Capacitor_SMD:C_0402_1005Metric, symbol Device:C
- added C825: 10u, Capacitor_SMD:C_0805_2012Metric, symbol Device:C
- added R810, R812: 5k36, Resistor_SMD:R_0402_1005Metric, symbol Device:R
- added R811: 23k7, Resistor_SMD:R_0402_1005Metric, symbol Device:R
- added R814: 22k1, Resistor_SMD:R_0402_1005Metric, symbol Device:R
- added R820: 93k1, Resistor_SMD:R_0402_1005Metric, symbol Device:R
- added R821: 1M, Resistor_SMD:R_0402_1005Metric, symbol Device:R
- added R822: 23k2, Resistor_SMD:R_0402_1005Metric, symbol Device:R
- added R823, R824: 10k, Resistor_SMD:R_0402_1005Metric, symbol Device:R
- added TP802: (no value), Testpoints_Kampi:TestPoint_Pad_1.0x1.0mm, symbol Connector:TestPoint
- added TP803, TP806: ~, Testpoints_Kampi:TestPoint_Pad_1.0x1.0mm, symbol Connector:TestPoint
- R809: value 27k -> 23k7; footprint Resistor_SMD:R_0805_2012Metric -> Resistor_SMD:R_0402_1005Metric; manf Bourns -> YAGEO; manf# CR0805-JW-273ELF -> RC0402FR-0723K7L; mouser# 652-CR0805-JW-273ELF -> 603-RC0402FR-0723K7L
- R815: value 10k -> 93k1; footprint Resistor_SMD:R_0805_2012Metric -> Resistor_SMD:R_0402_1005Metric; manf Bourns -> YAGEO; manf# CR0805-JW-103GLF -> RT0402BRD0793K1L; mouser# 652-CR0805-JW-103GLF -> 603-RT0402BRD0793K1L
- R816: value 10k -> 16k5; footprint Resistor_SMD:R_0805_2012Metric -> Resistor_SMD:R_0402_1005Metric; manf Bourns -> YAGEO; manf# CR0805-JW-103GLF -> RT0402BRD0716K5L; mouser# 652-CR0805-JW-103GLF -> 603-RT0402BRD0716K5L
Connections:
- net +1V8: now also R824.1; no longer R816.1
- net +5V: now also C820.1, C825.1, R823.1, TP802.1
- net GND: now also C820.2, C824.2, C825.2, R810.2, R812.2, R820.2, R822.2; no longer IC803.3 (CP2), IC803.4 (OV2), IC803.5 (OV1), IC803.6 (PR1), R809.2
- net at C809.2, C811.2, C813.2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: now also R809.1, R816.1
- net at C815.1, C817.1, D801.1 (K)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: now also R811.1, R814.1
- net at IC803.10 (ILIM): now also R822.1; no longer R809.1
- net at IC803.11 (SS): now also C824.1
- net at IC803.9 (ST), Q801.1 (G): now also R821.2, R823.2, TP803.1; no longer R815.1
- net Backup-Status: no longer names the net of R816.2
- net Backup-Status: now also IC803.6 (PR1), R820.1, R821.1; no longer Q801.3 (D)
- new net: IC803.3 (CP2), R814.2, R815.1
- new net: IC803.4 (OV2), R811.2, R812.1
- new net: IC803.5 (OV1), R809.2, R810.1
- new net PowerMux-Status: Q801.3 (D), R824.2, TP806.1

Commit message: Working on layout
Parts:
- C824: footprint Capacitor_SMD:C_0402_1005Metric -> Capacitor_SMD:C_0805_2012Metric; manf# 04025C104JAT2A -> 08053C104M4T4A; mouser# 581-04025C104JAT2A -> 581-08053C104M4T4A
- R803: manf# CR0805-JW-202GLF -> CR0805-FX-2001ELF; mouser# 652-CR0805-JW-202GLF -> 652-CR0805-FX-2001ELF
- R809, R811: footprint Resistor_SMD:R_0402_1005Metric -> Resistor_SMD:R_0805_2012Metric; manf# RC0402FR-0723K7L -> RC0805FR-0723K7L; mouser# 603-RC0402FR-0723K7L -> 603-RC0805FR-0723K7L
- R810, R812: footprint Resistor_SMD:R_0402_1005Metric -> Resistor_SMD:R_0805_2012Metric; manf# RT0402BRD075K36L -> RT0805BRD075K36L; mouser# 603-RT0402BRD075K36L -> 603-RT0805BRD075K36L
- R814: footprint Resistor_SMD:R_0402_1005Metric -> Resistor_SMD:R_0805_2012Metric; manf# RT0402BRD0722K1L -> RT0805BRD0722K1L; mouser# 603-RT0402BRD0722K1L -> 603-RT0805BRD0722K1L
- R815, R820: footprint Resistor_SMD:R_0402_1005Metric -> Resistor_SMD:R_0805_2012Metric; manf# RT0402BRD0793K1L -> RT0805BRD0793K1L; mouser# 603-RT0402BRD0793K1L -> 603-RT0805BRD0793K1L
- R816: footprint Resistor_SMD:R_0402_1005Metric -> Resistor_SMD:R_0805_2012Metric; manf# RT0402BRD0716K5L -> RT0805BRD0716K5L; mouser# 603-RT0402BRD0716K5L -> 603-RT0805BRD0716K5L
- R821: footprint Resistor_SMD:R_0402_1005Metric -> Resistor_SMD:R_0805_2012Metric; manf# RC0402FR-071ML -> RC0805FR-071ML; mouser# 603-RC0402FR-071ML -> 603-RC0805FR-071ML
- R822: footprint Resistor_SMD:R_0402_1005Metric -> Resistor_SMD:R_0805_2012Metric; manf# RT0402BRE0723K2L -> RT0805BRD0723K2L; mouser# 603-RT0402BRE0723K2L -> 603-RT0805BRD0723K2L
- R823, R824: footprint Resistor_SMD:R_0402_1005Metric -> Resistor_SMD:R_0805_2012Metric; manf# CR0402-JW-103GLF -> CR0805-JW-103GLF; mouser# 652-CR0402-JW-103GLF -> 652-CR0805-JW-103GLF
Changed lines of the file:
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@@
 		(exclude_from_sim no)
 		(at 217.17 176.53 0)
-		(size 195.58 7.62)
+		(size 186.69 7.62)
 		(margins 1.9049 1.9049 1.9049 1.9049)
 		(stroke
@@
 			)
 		)
-		(property "Footprint" "Resistor_SMD:R_0402_1005Metric"
+		(property "Footprint" "Resistor_SMD:R_0805_2012Metric"
 			(at 295.91 78.232 90)
 			(hide yes)
@@
 			)
 		)
-		(property "manf#" "RC0402FR-071ML"
+		(property "manf#" "RC0805FR-071ML"
 			(at 295.91 80.01 0)
 			(hide yes)
@@
 			)
 		)
-		(property "mouser#" "603-RC0402FR-071ML"
+		(property "mouser#" "603-RC0805FR-071ML"
 			(at 295.91 80.01 0)
 			(hide yes)
@@
 			)
 		)
-		(property "Footprint" "Resistor_SMD:R_0402_1005Metric"
+		(property "Footprint" "Resistor_SMD:R_0805_2012Metric"
 			(at 320.802 135.89 90)
 			(hide yes)
@@
 			)
 		)
-		(property "manf#" "RT0402BRE0723K2L"
+		(property "manf#" "RT0805BRD0723K2L"
 			(at 322.58 135.89 0)
 			(hide yes)
@@
 			)
 		)
-		(property "mouser#" "603-RT0402BRE0723K2L"
+		(property "mouser#" "603-RT0805BRD0723K2L"
 			(at 322.58 135.89 0)
 			(hide yes)
@@
 			)
 		)
-		(property "Footprint" "Resistor_SMD:R_0402_1005Metric"
+		(property "Footprint" "Resistor_SMD:R_0805_2012Metric"
 			(at 272.288 138.43 90)
 			(hide yes)
@@
 			)
 		)
-		(property "manf#" "RT0402BRD0722K1L"
+		(property "manf#" "RT0805BRD0722K1L"
 			(at 270.51 138.43 0)
 			(hide yes)
@@
 			)
 		)
-		(property "mouser#" "603-RT0402BRD0722K1L"
+		(property "mouser#" "603-RT0805BRD0722K1L"
 			(at 270.51 138.43 0)
 			(hide yes)
@@
 			)
 		)
-		(property "manf#" "CR0805-JW-202GLF"
+		(property "manf#" "CR0805-FX-2001ELF"
 			(at 100.33 226.06 0)
 			(hide yes)
@@
 			)
 		)
-		(property "mouser#" "652-CR0805-JW-202GLF"
+		(property "mouser#" "652-CR0805-FX-2001ELF"
 			(at 100.33 226.06 0)
 			(hide yes)
@@
 			)
 		)
-		(property "Footprint" "Resistor_SMD:R_0402_1005Metric"
+		(property "Footprint" "Resistor_SMD:R_0805_2012Metric"
 			(at 365.252 111.76 90)
 			(hide yes)
@@
 			)
 		)
-		(property "manf#" "CR0402-JW-103GLF"
+		(property "manf#" "CR0805-JW-103GLF"
 			(at 367.03 111.76 0)
 			(hide yes)
@@
 			)
 		)
-		(property "mouser#" "652-CR0402-JW-103GLF"
+		(property "mouser#" "652-CR0805-JW-103GLF"
 			(at 367.03 111.76 0)
 			(hide yes)
@@
 			)
 		)
-		(property "Footprint" "Resistor_SMD:R_0402_1005Metric"
+		(property "Footprint" "Resistor_SMD:R_0805_2012Metric"
 			(at 272.288 148.59 90)
 			(hide yes)
@@
 			)
 		)
-		(property "manf#" "RT0402BRD0793K1L"
+		(property "manf#" "RT0805BRD0793K1L"
 			(at 270.51 148.59 0)
 			(hide yes)
@@
 			)
 		)
-		(property "mouser#" "603-RT0402BRD0793K1L"
+		(property "mouser#" "603-RT0805BRD0793K1L"
 			(at 270.51 148.59 0)
 			(hide yes)
@@
 			)
 		)
-		(property "Footprint" "Resistor_SMD:R_0402_1005Metric"
+		(property "Footprint" "Resistor_SMD:R_0805_2012Metric"
 			(at 245.618 138.43 90)
 			(hide yes)
@@
 			)
 		)
-		(property "manf#" "RT0402BRD075K36L"
+		(property "manf#" "RT0805BRD075K36L"
 			(at 243.84 138.43 0)
 			(hide yes)
@@
 			)
 		)
-		(property "mouser#" "603-RT0402BRD075K36L"
+		(property "mouser#" "603-RT0805BRD075K36L"
 			(at 243.84 138.43 0)
 			(hide yes)
@@
 			)
 		)
-		(property "Footprint" "Resistor_SMD:R_0402_1005Metric"
+		(property "Footprint" "Resistor_SMD:R_0805_2012Metric"
 			(at 274.828 85.09 90)
 			(hide yes)
@@
 			)
 		)
-		(property "manf#" "RT0402BRD0793K1L"
+		(property "manf#" "RT0805BRD0793K1L"
 			(at 273.05 85.09 0)
 			(hide yes)
@@
 			)
 		)
-		(property "mouser#" "603-RT0402BRD0793K1L"
+		(property "mouser#" "603-RT0805BRD0793K1L"
 			(at 273.05 85.09 0)
 			(hide yes)
@@
 			)
 		)
-		(property "Footprint" "Resistor_SMD:R_0402_1005Metric"
+		(property "Footprint" "Resistor_SMD:R_0805_2012Metric"
 			(at 334.518 102.87 90)
 			(hide yes)
@@
 			)
 		)
-		(property "manf#" "CR0402-JW-103GLF"
+		(property "manf#" "CR0805-JW-103GLF"
 			(at 332.74 102.87 0)
 			(hide yes)
@@
 			)
 		)
-		(property "mouser#" "652-CR0402-JW-103GLF"
+		(property "mouser#" "652-CR0805-JW-103GLF"
 			(at 332.74 102.87 0)
 			(hide yes)
@@
 			)
 		)
-		(property "Footprint" "Resistor_SMD:R_0402_1005Metric"
+		(property "Footprint" "Resistor_SMD:R_0805_2012Metric"
 			(at 231.648 113.03 90)
 			(hide yes)
@@
 			)
 		)
-		(property "manf#" "RC0402FR-0723K7L"
+		(property "manf#" "RC0805FR-0723K7L"
 			(at 229.87 113.03 0)
 			(hide yes)
@@
 			)
 		)
-		(property "mouser#" "603-RC0402FR-0723K7L"
+		(property "mouser#" "603-RC0805FR-0723K7L"
 			(at 229.87 113.03 0)
 			(hide yes)
@@
 			)
 		)
-		(property "Footprint" "Resistor_SMD:R_0402_1005Metric"
+		(property "Footprint" "Resistor_SMD:R_0805_2012Metric"
 			(at 231.648 128.27 90)
 			(hide yes)
@@
 			)
 		)
-		(property "manf#" "RT0402BRD075K36L"
+		(property "manf#" "RT0805BRD075K36L"
 			(at 229.87 128.27 0)
 			(hide yes)
@@
 			)
 		)
-		(property "mouser#" "603-RT0402BRD075K36L"
+		(property "mouser#" "603-RT0805BRD075K36L"
 			(at 229.87 128.27 0)
 			(hide yes)
@@
 			)
 		)
-		(property "Footprint" "Capacitor_SMD:C_0402_1005Metric"
+		(property "Footprint" "Capacitor_SMD:C_0805_2012Metric"
 			(at 309.5752 139.7 0)
 			(hide yes)
@@
 			)
 		)
-		(property "Datasheet" "https://datasheets.kyocera-avx.com/KGM_X7R.pdf"
+		(property "Datasheet" "https://datasheets.kyocera-avx.com/AutoMLCC.pdf"
 			(at 308.61 135.89 0)
 			(hide yes)
@@
 			)
 		)
-		(property "manf#" "04025C104JAT2A"
+		(property "manf#" "08053C104M4T4A"
 			(at 308.61 135.89 0)
 			(hide yes)
@@
 			)
 		)
-		(property "mouser#" "581-04025C104JAT2A"
+		(property "mouser#" "581-08053C104M4T4A"
 			(at 308.61 135.89 0)
 			(hide yes)
@@
 			)
 		)
-		(property "Footprint" "Resistor_SMD:R_0402_1005Metric"
+		(property "Footprint" "Resistor_SMD:R_0805_2012Metric"
 			(at 245.618 128.27 90)
 			(hide yes)
@@
 			)
 		)
-		(property "manf#" "RC0402FR-0723K7L"
+		(property "manf#" "RC0805FR-0723K7L"
 			(at 243.84 128.27 0)
 			(hide yes)
@@
 			)
 		)
-		(property "mouser#" "603-RC0402FR-0723K7L"
+		(property "mouser#" "603-RC0805FR-0723K7L"
 			(at 243.84 128.27 0)
 			(hide yes)
@@
 			)
 		)
-		(property "Footprint" "Resistor_SMD:R_0402_1005Metric"
+		(property "Footprint" "Resistor_SMD:R_0805_2012Metric"
 			(at 274.828 74.93 90)
 			(hide yes)
@@
 			)
 		)
-		(property "manf#" "RT0402BRD0716K5L"
+		(property "manf#" "RT0805BRD0716K5L"
 			(at 273.05 74.93 0)
 			(hide yes)
@@
 			)
 		)
-		(property "mouser#" "603-RT0402BRD0716K5L"
+		(property "mouser#" "603-RT0805BRD0716K5L"
 			(at 273.05 74.93 0)
 			(hide yes)

Commit message: Working on revision 1.0.0
Parts:
- C801, C802, C807, C815, C817, C825: symbol Device:C -> partdb:0805X7R106KT1AT; Category (none) -> Kondensator/MLCC; MPN (none) -> 0805X7R106KT1AT; Manufacturer (none) -> KYOCERA AVX; Manufacturing Status (none) -> Active; Mouser SPN (none) -> 581-0805X7R106KT1AT; Part-DB Footprint (none) -> 0805; Part-DB ID (none) -> 331; Part-DB URL (none) -> https://inventory.lan/de/part/331/info; Stock (none) -> 0
- C803, C819, C821, C822, C823: symbol Device:C -> partdb:08053G105MAT2A; Category (none) -> Kondensator/MLCC; MPN (none) -> 08053G105MAT2A; Manufacturer (none) -> KYOCERA AVX; Manufacturing Status (none) -> Active; Mass (none) -> 0.006 g; Mouser SPN (none) -> 581-08053G105MAT2A; Part-DB Footprint (none) -> 0805; Part-DB ID (none) -> 349; Part-DB URL (none) -> https://inventory.lan/de/part/349/info; Stock (none) -> 0; manf# 08056C105MAT2A -> 08053G105MAT2A; mouser# 581-08056C105MAT2A -> 581-08053G105MAT2A
- C805, C806: symbol Device:C -> partdb:08055C474K4Z2A; Category (none) -> Kondensator/MLCC; MPN (none) -> 08055C474K4Z2A; Manufacturer (none) -> KYOCERA AVX; Manufacturing Status (none) -> Active; Mass (none) -> 0.006 g; Mouser SPN (none) -> 581-08055C474K4Z2A; Part-DB Footprint (none) -> 0805; Part-DB ID (none) -> 329; Part-DB URL (none) -> https://inventory.lan/de/part/329/info; Stock (none) -> 0; manf# 08053C474K4T4A -> 08055C474K4Z2A; mouser# 581-08053C474K4T4A -> 581-08055C474K4Z2A
- C808, C824: symbol Device:C -> partdb:08055C104K4Z4A; Category (none) -> Kondensator/MLCC; MPN (none) -> 08055C104K4Z4A; Manufacturer (none) -> KYOCERA AVX; Manufacturing Status (none) -> Active; Mass (none) -> 0.006 g; Mouser SPN (none) -> 581-08055C104K4Z4A; Part-DB Footprint (none) -> 0805; Part-DB ID (none) -> 109; Part-DB URL (none) -> https://inventory.lan/de/part/109/info; Stock (none) -> 6; Storage Location (none) -> Sortierregal; manf# 08053C104M4T4A -> 08055C104K4Z4A; mouser# 581-08053C104M4T4A -> 581-08055C104K4Z4A
- C809, C811, C813, C814: symbol Device:C -> partdb:MLAST21GBB5226MTNC12; Category (none) -> Kondensator/MLCC; MPN (none) -> MLAST21GBB5226MTNC12; Manufacturer (none) -> TAIYO YUDEN; Manufacturing Status (none) -> Active; Mouser SPN (none) -> 963-MLAST21GBB5226MT; Part-DB Footprint (none) -> 0805; Part-DB ID (none) -> 330; Part-DB URL (none) -> https://inventory.lan/de/part/330/info; Stock (none) -> 0; manf KYOCERA AVX -> TAIYO YUDEN; manf# KGM21AR51A226MU -> MLAST21GBB5226MTNC12; mouser# 581-KGM21AR51A226MU -> 963-MLAST21GBB5226MT
- R801, R805, R813, R823, R824: symbol Device:R -> partdb:CR0805-FX-1002ELF; Category (none) -> Widerstand/Dickfilmwiderstand; MPN (none) -> CR0805-FX-1002ELF; Manufacturer (none) -> Bourns; Manufacturing Status (none) -> Active; Mass (none) -> 0.006 g; Mouser SPN (none) -> 652-CR0805FX-1002ELF; Part-DB Footprint (none) -> 0805; Part-DB ID (none) -> 343; Part-DB URL (none) -> https://inventory.lan/de/part/343/info; Stock (none) -> 0; manf# CR0805-JW-103GLF -> CR0805-FX-1002ELF; mouser# 652-CR0805-JW-103GLF -> 652-CR0805FX-1002ELF
- R806: symbol Device:R -> partdb:RT0805FRE13100KL; Category (none) -> Widerstand/Dünnfilmwiderstand; MPN (none) -> RT0805FRE13100KL; Manufacturer (none) -> YAGEO; Manufacturing Status (none) -> Active; Mass (none) -> 0.006 g; Mouser SPN (none) -> 603-RT0805FRE13100KL; Part-DB Footprint (none) -> 0805; Part-DB ID (none) -> 66; Part-DB URL (none) -> https://inventory.lan/de/part/66/info; Stock (none) -> 4; Storage Location (none) -> Sortierregal; manf Bourns -> YAGEO; manf# CR0805-JW-104GLF -> RT0805FRE13100KL; mouser# 652-CR0805-JW-104GLF -> 603-RT0805FRE13100KL
- R817: symbol Device:R -> partdb:CR0805-FX-1002ELF; Category (none) -> Widerstand/Dickfilmwiderstand; MPN (none) -> CR0805-FX-1002ELF; Manufacturer (none) -> Bourns; Manufacturing Status (none) -> Active; Mass (none) -> 0.006 g; Mouser SPN (none) -> 652-CR0805FX-1002ELF; Part-DB Footprint (none) -> 0805; Part-DB ID (none) -> 343; Part-DB URL (none) -> https://inventory.lan/de/part/343/info; Stock (none) -> 0; manf# CR0805-FX-1002GLF -> CR0805-FX-1002ELF; mouser# 652-CR0805-FX-1002GLF -> 652-CR0805FX-1002ELF
- R818, R819: symbol Device:R -> partdb:CR0805-J/-000ELF; Category (none) -> Widerstand/Dickfilmwiderstand; MPN (none) -> CR0805-J/-000ELF; Manufacturer (none) -> Bourns; Manufacturing Status (none) -> Active; Mass (none) -> 0.006 g; Mouser SPN (none) -> 652-CR0805-J/-000ELF; Part-DB Footprint (none) -> 0805; Part-DB ID (none) -> 322; Part-DB URL (none) -> https://inventory.lan/de/part/322/info; Stock (none) -> 0
- R821: symbol Device:R -> partdb:RC0805FR-071ML; Category (none) -> Widerstand/Dickfilmwiderstand; MPN (none) -> RC0805FR-071ML; Manufacturer (none) -> YAGEO; Manufacturing Status (none) -> Active; Mass (none) -> 0.0055 g; Mouser SPN (none) -> 603-RC0805FR-071ML; Part-DB Footprint (none) -> 0805; Part-DB ID (none) -> 370; Part-DB URL (none) -> https://inventory.lan/de/part/370/info; Stock (none) -> 0
Other:
- moved on the sheet: C821, TP809
