File: gateway/Power.kicad_sch (KiCad schematic)
At the start: 66 parts, among them IC801 LM62460, IC802 ADP1614ACPZ-650-R7, IC803 TPS2121RUXT, IC804 TLV75733PDBV, IC805 TLV75733PDBV, Q801 BSS138

Commit message: Prepare Release 1.0.0
Co-Authored-By: Claude Opus 5.5 <noreply@anthropic.com>
Parts:
- IC701: renamed from IC801; manf# LM62460 -> LM62460RPHR; mouser# 595-LM62460 -> 595-LM62460RPHR
- IC702: renamed from IC802; mouser# 584-ADP1614ACPZ-650-R7 -> 584-ADP1614ACPZ650R7
- R704: renamed from R803; mouser# 652-CR0805-FX-2001ELF -> 652-CR0805FX-2001ELF
- R705: renamed from R804; mouser# 652-CR0805-FX-3092GLF -> 652-CR0805FX-3092GLF
- R708: renamed from R807; mouser# 652-CR0805-FX-2492ELF -> 652-CR0805FX-2492ELF
- R709: renamed from R808; mouser# 652-CR0805-FX-4991ELF -> 652-CR0805FX-4991ELF
- renumbered C801 to C701, C803 to C702, C802 to C703, C804 to C704, C805 to C705, C806 to C706, C807 to C707, C816 to C708, C808 to C709, C810 to C710, C809 to C711, C812 to C712, C811 to C713, C813 to C714, C815 to C715, C814 to C716, C817 to C717, C818 to C718, C819 to C719, C820 to C720, C824 to C721, C821 to C722, C825 to C723, C822 to C724, C823 to C725, D801 to D701, IC804 to IC703, IC803 to IC704, IC805 to IC705, L801 to L701, L802 to L702, Q801 to Q701, R819 to R701, R801 to R702, R802 to R703, R805 to R706, R806 to R707, R809 to R710, R810 to R711, R811 to R712, R812 to R713, R814 to R714, R815 to R715, R816 to R716, R820 to R717, R813 to R718, R821 to R719, R822 to R720, R823 to R721, R817 to R722, R824 to R723, R818 to R724, TP801 to TP701, TP804 to TP702, TP805 to TP703, TP802 to TP704, TP809 to TP705, TP803 to TP706, TP806 to TP707, TP811 to TP708
