File: gateway/Peripherals.kicad_sch (KiCad schematic)
At the start: 29 parts, among them IC1401 ATECC608B-SSHDA, IC1402 TUSB320, IC1403 TXB0102DCU, IC1404 TXS0102DCU, IC1405 TXS0102DCU, X1401 OTG, X1402 GPIO, X1403 CAN, X1404 I2C, X1405 I2C

Commit message: Add INA219 for current measurement
Parts:
- gave numbers to parts that had none: 1
- renumbered C1401 to C1501, C1402 to C1502, C1409 to C1503, C1410 to C1504, C1404 to C1505, C1403 to C1506, C1405 to C1507, C1407 to C1508, C1406 to C1509, C1408 to C1510, IC1401 to IC1501, IC1402 to IC1502, IC1404 to IC1504, IC1403 to IC1505, IC1405 to IC1506, R1407 to R1501, R1401 to R1502, R1402 to R1503, R1403 to R1504, R1404 to R1505, R1405 to R1506, R1406 to R1507, TP1401 to TP1501, X1401 to X1501, X1402 to X1502, X1404 to X1503, X1403 to X1504, X1405 to X1505
Connections:
- net SCL_{HV}: now reaches IC1504.1 (B2), R1506.2, X1503.3 (Pin_3)
- net SDA_{HV}: now reaches IC1504.8 (B1), R1504.2, X1503.2 (Pin_2)
Other:
- moved on the sheet: C1505, C1506, C1508, C1509, IC1504, IC1505, R1504, R1506, X1503, X1504
