File: gateway/Peripherals.kicad_sch (KiCad schematic)
At the start: 29 parts, among them IC1501 ATECC608B-SSHDA, IC1502 TUSB320, IC1503 TXS0108EPW, IC1504 TXS0102DCU, IC1505 TXB0102DCU, IC1506 TXS0102DCU, X1501 OTG, X1502 GPIO, X1503 I2C, X1504 CAN, X1505 I2C

Commit message: Prepare Release 1.0.0
Co-Authored-By: Claude Opus 5.5 <noreply@anthropic.com>
Parts:
- R1401: renamed from R1501; manf YAGEO -> Bourns; manf# RC0805FR-07887KL -> CR0805-FX-8873ELF; mouser# 603-RC0805FR-07887KL -> 652-CR0805FX-8873ELF
- R1404: renamed from R1504; Mouser SPN 652-CR0805-JW-332ELF -> 652-CR0805JW-332ELF; mouser# 652-CR0805-JW-332ELF -> 652-CR0805JW-332ELF
- R1405: renamed from R1505; Mouser SPN 652-CR0805-JW-332ELF -> 652-CR0805JW-332ELF; mouser# 652-CR0805-JW-332ELF -> 652-CR0805JW-332ELF
- R1406: renamed from R1506; Mouser SPN 652-CR0805-JW-332ELF -> 652-CR0805JW-332ELF; mouser# 652-CR0805-JW-332ELF -> 652-CR0805JW-332ELF
- R1407: renamed from R1507; Mouser SPN 652-CR0805-JW-332ELF -> 652-CR0805JW-332ELF; mouser# 652-CR0805-JW-332ELF -> 652-CR0805JW-332ELF
- renumbered C1501 to C1401, C1502 to C1402, C1503 to C1403, C1504 to C1404, C1505 to C1405, C1506 to C1406, C1507 to C1407, C1508 to C1408, C1509 to C1409, C1510 to C1410, IC1501 to IC1401, IC1502 to IC1402, IC1503 to IC1403, IC1504 to IC1404, IC1505 to IC1405, IC1506 to IC1406, R1502 to R1402, R1503 to R1403, TP1501 to TP1401, X1501 to X1401, X1502 to X1402, X1503 to X1403, X1504 to X1404, X1505 to X1405

Commit message: Update schematic and board
- Use Part-DB symbols, BT901 changed to Keystone 3030TR
- Add the revision text to the board
- Include more parts in BOM and position files

Co-Authored-By: Claude Opus 5.5 <noreply@anthropic.com>
Parts:
- X1401: footprint Connector_USB:USB_C_Receptacle_GCT_USB4110 -> GCT:USB4110; symbol Connector:USB_C_Receptacle_USB2.0_14P -> partdb:USB4110-GF-A
Connections:
- no-connect marks 5 -> 7
Changed lines of the file:
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@@
 		(at 96.52 193.04)
 	)
+	(no_connect
+		(at 49.53 254)
+	)
+	(no_connect
+		(at 49.53 256.54)
+	)
 	(bus_entry
 		(at 134.62 223.52)
@@
 	)
 	(symbol
-		(lib_id "Connector:USB_C_Receptacle_USB2.0_14P")
+		(lib_id "partdb:USB4110-GF-A")
 		(at 34.29 241.3 0)
 		(unit 1)
@@
 			)
 		)
-		(property "Footprint" "Connector_USB:USB_C_Receptacle_GCT_USB4110"
+		(property "Footprint" "GCT:USB4110"
 			(at 38.1 241.3 0)
 			(hide yes)
@@
 			)
 		)
+		(property "Config" ""
+			(at 34.29 241.3 0)
+			(hide yes)
+			(show_name no)
+			(do_not_autoplace no)
+			(effects
+				(font
+					(size 1.27 1.27)
+				)
+			)
+		)
 		(pin "A1"
 		)
@@
 		(pin "SH"
 		)
+		(pin "A8"
+		)
+		(pin "B8"
+		)
 		(instances
