File: gateway/Ethernet.kicad_sch (KiCad schematic)
At the start: 9 parts, among them X1601 Ethernet

Commit message: Add INA219 for current measurement
Parts:
- renumbered C1601 to C1701, C1602 to C1702, C1603 to C1703, R1601 to R1701, R1602 to R1702, R1603 to R1703, TP1601 to TP1701, TP1602 to TP1702, X1601 to X1701
Changed lines of the file:
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@@
 	(title_block
 		(title "Ethernet")
-		(date "2025-06-05")
+		(date "2026-07-09")
 		(rev "${REVISION}")
 		(company "${COMPANY}")
@@
 		(in_pos_files yes)
 		(dnp no)
-		(property "Reference" "R1603"
+		(property "Reference" "R1703"
 			(at 257.81 182.8799 0)
 			(show_name no)
@@
 			(project "Gateway"
 				(path "/d5742f03-3b1a-42e5-a384-018bd4b919aa/c5103ceb-5325-4a84-a025-9638a412984e/86891732-a753-4dcc-a58c-71e3fc99b0cd"
-					(reference "R1603")
+					(reference "R1703")
 					(unit 1)
 				)
@@
 		(in_pos_files no)
 		(dnp no)
-		(property "Reference" "TP1602"
+		(property "Reference" "TP1702"
 			(at 227.33 95.25 0)
 			(show_name no)
@@
 			(project "Gateway"
 				(path "/d5742f03-3b1a-42e5-a384-018bd4b919aa/c5103ceb-5325-4a84-a025-9638a412984e/86891732-a753-4dcc-a58c-71e3fc99b0cd"
-					(reference "TP1602")
+					(reference "TP1702")
 					(unit 1)
 				)
@@
 		(in_pos_files yes)
 		(dnp no)
-		(property "Reference" "C1603"
+		(property "Reference" "C1703"
 			(at 246.38 182.8799 0)
 			(show_name no)
@@
 			(project "Gateway"
 				(path "/d5742f03-3b1a-42e5-a384-018bd4b919aa/c5103ceb-5325-4a84-a025-9638a412984e/86891732-a753-4dcc-a58c-71e3fc99b0cd"
-					(reference "C1603")
+					(reference "C1703")
 					(unit 1)
 				)
@@
 		(in_pos_files yes)
 		(dnp no)
-		(property "Reference" "#PWR01601"
+		(property "Reference" "#PWR01701"
 			(at 185.42 187.96 0)
 			(hide yes)
@@
 			(project "Gateway"
 				(path "/d5742f03-3b1a-42e5-a384-018bd4b919aa/c5103ceb-5325-4a84-a025-9638a412984e/86891732-a753-4dcc-a58c-71e3fc99b0cd"
-					(reference "#PWR01601")
+					(reference "#PWR01701")
 					(unit 1)
 				)
@@
 		(dnp no)
 		(fields_autoplaced yes)
-		(property "Reference" "#PWR01606"
+		(property "Reference" "#PWR01706"
 			(at 269.24 196.85 0)
 			(hide yes)
@@
 			(project "Gateway"
 				(path "/d5742f03-3b1a-42e5-a384-018bd4b919aa/c5103ceb-5325-4a84-a025-9638a412984e/86891732-a753-4dcc-a58c-71e3fc99b0cd"
-					(reference "#PWR01606")
+					(reference "#PWR01706")
 					(unit 1)
 				)
@@
 		(dnp no)
 		(fields_autoplaced yes)
-		(property "Reference" "#FLG01601"
+		(property "Reference" "#FLG01701"
 			(at 269.24 175.895 0)
 			(hide yes)
@@
 			(project "Gateway"
 				(path "/d5742f03-3b1a-42e5-a384-018bd4b919aa/c5103ceb-5325-4a84-a025-9638a412984e/86891732-a753-4dcc-a58c-71e3fc99b0cd"
-					(reference "#FLG01601")
+					(reference "#FLG01701")
 					(unit 1)
 				)
@@
 		(in_pos_files yes)
 		(dnp no)
-		(property "Reference" "C1601"
+		(property "Reference" "C1701"
 			(at 181.61 176.5299 0)
 			(show_name no)
@@
 			(project "Gateway"
 				(path "/d5742f03-3b1a-42e5-a384-018bd4b919aa/c5103ceb-5325-4a84-a025-9638a412984e/86891732-a753-4dcc-a58c-71e3fc99b0cd"
-					(reference "C1601")
+					(reference "C1701")
 					(unit 1)
 				)
@@
 		(dnp no)
 		(fields_autoplaced yes)
-		(property "Reference" "#PWR01603"
+		(property "Reference" "#PWR01703"
 			(at 207.01 180.34 0)
 			(hide yes)
@@
 			(project "Gateway"
 				(path "/d5742f03-3b1a-42e5-a384-018bd4b919aa/c5103ceb-5325-4a84-a025-9638a412984e/86891732-a753-4dcc-a58c-71e3fc99b0cd"
-					(reference "#PWR01603")
+					(reference "#PWR01703")
 					(unit 1)
 				)
@@
 		(in_pos_files no)
 		(dnp no)
-		(property "Reference" "TP1601"
+		(property "Reference" "TP1701"
 			(at 227.33 74.93 0)
 			(show_name no)
@@
 			(project "Gateway"
 				(path "/d5742f03-3b1a-42e5-a384-018bd4b919aa/c5103ceb-5325-4a84-a025-9638a412984e/86891732-a753-4dcc-a58c-71e3fc99b0cd"
-					(reference "TP1601")
+					(reference "TP1701")
 					(unit 1)
 				)
@@
 		(dnp no)
 		(fields_autoplaced yes)
-		(property "Reference" "#PWR01604"
+		(property "Reference" "#PWR01704"
 			(at 217.17 105.41 0)
 			(hide yes)
@@
 			(project "Gateway"
 				(path "/d5742f03-3b1a-42e5-a384-018bd4b919aa/c5103ceb-5325-4a84-a025-9638a412984e/86891732-a753-4dcc-a58c-71e3fc99b0cd"
-					(reference "#PWR01604")
+					(reference "#PWR01704")
 					(unit 1)
 				)
@@
 		(in_pos_files yes)
 		(dnp no)
-		(property "Reference" "C1602"
+		(property "Reference" "C1702"
 			(at 194.31 176.5299 0)
 			(show_name no)
@@
 			(project "Gateway"
 				(path "/d5742f03-3b1a-42e5-a384-018bd4b919aa/c5103ceb-5325-4a84-a025-9638a412984e/86891732-a753-4dcc-a58c-71e3fc99b0cd"
-					(reference "C1602")
+					(reference "C1702")
 					(unit 1)
 				)
@@
 		(in_pos_files yes)
 		(dnp no)
-		(property "Reference" "R1601"
+		(property "Reference" "R1701"
 			(at 209.55 180.3399 0)
 			(show_name no)
@@
 			(project "Gateway"
 				(path "/d5742f03-3b1a-42e5-a384-018bd4b919aa/c5103ceb-5325-4a84-a025-9638a412984e/86891732-a753-4dcc-a58c-71e3fc99b0cd"
-					(reference "R1601")
+					(reference "R1701")
 					(unit 1)
 				)
@@
 		(in_pos_files yes)
 		(dnp no)
-		(property "Reference" "R1602"
+		(property "Reference" "R1702"
 			(at 214.63 106.6799 0)
 			(show_name no)
@@
 			(project "Gateway"
 				(path "/d5742f03-3b1a-42e5-a384-018bd4b919aa/c5103ceb-5325-4a84-a025-9638a412984e/86891732-a753-4dcc-a58c-71e3fc99b0cd"
-					(reference "R1602")
+					(reference "R1702")
 					(unit 1)
 				)
@@
 		(in_pos_files yes)
 		(dnp no)
-		(property "Reference" "#PWR01605"
+		(property "Reference" "#PWR01705"
 			(at 252.73 196.85 0)
 			(hide yes)
@@
 			(project "Gateway"
 				(path "/d5742f03-3b1a-42e5-a384-018bd4b919aa/c5103ceb-5325-4a84-a025-9638a412984e/86891732-a753-4dcc-a58c-71e3fc99b0cd"
-					(reference "#PWR01605")
+					(reference "#PWR01705")
 					(unit 1)
 				)
@@
 		(in_pos_files yes)
 		(dnp no)
-		(property "Reference" "#PWR01602"
+		(property "Reference" "#PWR01702"
 			(at 190.5 187.96 0)
 			(hide yes)
@@
 			(project "Gateway"
 				(path "/d5742f03-3b1a-42e5-a384-018bd4b919aa/c5103ceb-5325-4a84-a025-9638a412984e/86891732-a753-4dcc-a58c-71e3fc99b0cd"
-					(reference "#PWR01602")
+					(reference "#PWR01702")
 					(unit 1)
 				)
@@
 		(dnp no)
 		(fields_autoplaced yes)
-		(property "Reference" "X1601"
+		(property "Reference" "X1701"
 			(at 254 138.4299 0)
 			(show_name no)
@@
 			(project "Gateway"
 				(path "/d5742f03-3b1a-42e5-a384-018bd4b919aa/c5103ceb-5325-4a84-a025-9638a412984e/86891732-a753-4dcc-a58c-71e3fc99b0cd"
-					(reference "X1601")
+					(reference "X1701")
 					(unit 1)
 				)

Commit message: Improving Thread
- Add boot signal for Thread MCU
- Add debug LED for nRF5340
Parts:
- TP1701, TP1702: value ~ -> (none)
Changed lines of the file:
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@@
 			)
 		)
-		(property "Value" "~"
+		(property "Value" ""
 			(at 227.33 93.345 0)
 			(show_name no)
@@
 			)
 		)
-		(property "Value" "~"
+		(property "Value" ""
 			(at 227.33 76.835 0)
 			(show_name no)

Commit message: Working on PCB
Parts:
- added C1701: 470u, Capacitor_SMD:CP_Elec_6.3x7.7, symbol Device:C_Polarized
- added C1702, C1703: 4n7, Capacitor_SMD:C_1206_3216Metric, symbol Device:C
- added C1704: 10n, Capacitor_SMD:C_0805_2012Metric, symbol Device:C
- added D1701, D1702, D1703, D1704: SS36, Diode_SMD:D_SMA, symbol Diode:SS36
- added IC1701: TLP293, Toshiba:TLP293(TPL,E, symbol Isolator:TLP293
- added M1701: Ag5400, Silvertel:Ag5400, symbol Silvertel:Ag5400
- added R1701, R1702: ~, Resistor_SMD:R_0805_2012Metric, symbol Device:R
- added TP1703, TP1704: ~, Testpoints_Kampi:TestPoint_Pad_1.0x1.0mm, symbol Connector:TestPoint
- C1707: renamed from C1703; value 1n / 2 kV -> 1n
- R1705: renamed from R1703; footprint Resistor_SMD:R_1206_3216Metric -> Resistor_SMD:R_2010_5025Metric; manf YAGEO -> Vishay / Techno; manf# RC1206JR-071ML -> CRMA2010AF1M00DKEF; mouser# 603-RC1206JR-071ML -> 71-CRMA2010AF1M00DKF
- TP1701, TP1702: value (none) -> ~
- renumbered C1701 to C1705, C1702 to C1706, R1701 to R1703, R1702 to R1704
Connections:
- net GND: now also C1701.2, C1702.1, C1703.1, IC1701.3, M1701.10 (V_{DC}-), M1701.7 (V_{DC}-), R1702.2
- net PoE-A: now also D1701.1 (K), D1703.1 (K), TP1703.1; no longer TP1702.1
- net PoE-B: now also D1702.2 (A), D1704.2 (A), TP1704.1; no longer TP1701.1
- new net: C1703.2, C1704.2, D1701.2 (A), D1702.1 (K), M1701.2 (V_{IN}-), TP1702.1
- new net: M1701.9 (ADJ), R1701.2, R1702.1
- new net: C1702.2, C1704.1, D1703.2 (A), D1704.1 (K), IC1701.1, M1701.1 (V_{IN}+), TP1701.1
- new net: IC1701.2, M1701.3 (AT-DET)
- new net: M1701.4 (IC), M1701.5 (IC), M1701.6 (IC)
- new net AT-DET: IC1701.4
- new net PoE: C1701.1, M1701.8 (V_{DC}+), R1701.1
Other:
- moved on the sheet: C1705, C1706, C1707, R1703, R1704, R1705, X1701
