File: gateway/Ethernet.kicad_sch (KiCad schematic)
At the start: 23 parts, among them IC1701 TLP293, M1701 Ag5400, X1701 Ethernet

Commit message: Working on layout
Parts:
- added TP1705: ~, Testpoints_Kampi:TestPoint_Pad_1.0x1.0mm, symbol Connector:TestPoint
Connections:
- net PoE: now also TP1705.1
Other:
- moved on the sheet: C1701, C1702, C1703, C1704, D1701, D1702, D1703, D1704, IC1701, M1701, R1701, R1702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

Commit message: Prepare release 1.0.0
Parts:
- added R1706: 1k8, Resistor_SMD:R_0805_2012Metric, symbol Device:R
- C1701, C1702, C1703, C1704, D1702, D1703, D1704, M1701: Config (none) -> +POE
Connections:
- net AT-DET: now also R1706.2
- new net +1V8: R1706.1

Commit message: Smaller changes
Parts:
- D1701, IC1701: Config (none) -> +POE
Changed lines of the file:
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@@
 			)
 		)
-		(property "Config" ""
+		(property "Config" "+POE"
 			(at -13.97 13.97 0)
+			(hide yes)
 			(show_name no)
 			(do_not_autoplace no)
@@
 			)
 		)
-		(property "Config" ""
+		(property "Config" "+POE"
 			(at 0 0 0)
+			(hide yes)
 			(show_name no)
 			(do_not_autoplace no)
@@
 		(property "Config" "+POE"
 			(at -153.67 153.67 0)
+			(hide yes)
 			(show_name no)
 			(do_not_autoplace no)
@@
 		(property "Config" "+POE"
 			(at 139.7 0 0)
+			(hide yes)
 			(show_name no)
 			(do_not_autoplace no)
@@
 		(property "Config" "+POE"
 			(at -26.67 26.67 0)
+			(hide yes)
 			(show_name no)
 			(do_not_autoplace no)
@@
 		(property "Config" "+POE"
 			(at 389.89 8.89 0)
+			(hide yes)
 			(show_name no)
 			(do_not_autoplace no)
@@
 		(property "Config" "+POE"
 			(at 402.59 21.59 0)
+			(hide yes)
 			(show_name no)
 			(do_not_autoplace no)
@@
 		(property "Config" "+POE"
 			(at 0 0 0)
+			(hide yes)
 			(show_name no)
 			(do_not_autoplace no)
@@
 		(property "Config" "+POE"
 			(at -160.02 299.72 0)
+			(hide yes)
 			(show_name no)
 			(do_not_autoplace no)

Commit message: Working on revision 1.0.0
Parts:
- C1705, C1706: symbol Device:C -> partdb:08055C104K4Z4A; Category (none) -> Kondensator/MLCC; MPN (none) -> 08055C104K4Z4A; Manufacturer (none) -> KYOCERA AVX; Manufacturing Status (none) -> Active; Mass (none) -> 0.006 g; Mouser SPN (none) -> 581-08055C104K4Z4A; Part-DB Footprint (none) -> 0805; Part-DB ID (none) -> 109; Part-DB URL (none) -> https://inventory.lan/de/part/109/info; Stock (none) -> 6; Storage Location (none) -> Sortierregal; manf# 08053C104M4T4A -> 08055C104K4Z4A; mouser# 581-08053C104M4T4A -> 581-08055C104K4Z4A
- R1703, R1704: symbol Device:R -> partdb:CR0805-JW-471ELF; Category (none) -> Widerstand/Dickfilmwiderstand; MPN (none) -> CR0805-JW-471ELF; Manufacturer (none) -> Bourns; Manufacturing Status (none) -> Active; Mass (none) -> 0.006 g; Mouser SPN (none) -> 652-CR0805JW-471ELF; Part-DB Footprint (none) -> 0805; Part-DB ID (none) -> 307; Part-DB URL (none) -> https://inventory.lan/de/part/307/info; Stock (none) -> 25; Storage Location (none) -> Sortierregal; manf# CR0805-JW-471GLF -> CR0805-JW-471ELF; mouser# 652-CR0805-JW-471GLF -> 652-CR0805JW-471ELF
- R1706: symbol Device:R -> partdb:CR0805-JW-182ELF; Category (none) -> Widerstand/Dickfilmwiderstand; MPN (none) -> CR0805-JW-182ELF; Manufacturer (none) -> Bourns; Manufacturing Status (none) -> Active; Mass (none) -> 0.0055 g; Mouser SPN (none) -> 652-CR0805JW-182ELF; Part-DB Footprint (none) -> 0805; Part-DB ID (none) -> 350; Part-DB URL (none) -> https://inventory.lan/de/part/350/info; Stock (none) -> 0; manf# CR0805-FX-1801GLF -> CR0805-JW-182ELF; mouser# 652-CR0805-FX-1801GLF -> 652-CR0805JW-182ELF
