File: gateway/Ethernet.kicad_sch (KiCad schematic)
At the start: 25 parts, among them IC1701 TLP293, M1701 Ag5400, X1701 Ethernet

Commit message: Working on revision 1.0.0
Parts:
- C1705, C1706: symbol Device:C -> partdb:08055C104K4Z4A; Category (none) -> Kondensator/MLCC; MPN (none) -> 08055C104K4Z4A; Manufacturer (none) -> KYOCERA AVX; Manufacturing Status (none) -> Active; Mass (none) -> 0.006 g; Mouser SPN (none) -> 581-08055C104K4Z4A; Part-DB Footprint (none) -> 0805; Part-DB ID (none) -> 109; Part-DB URL (none) -> https://inventory.lan/de/part/109/info; Stock (none) -> 6; Storage Location (none) -> Sortierregal; manf# 08053C104M4T4A -> 08055C104K4Z4A; mouser# 581-08053C104M4T4A -> 581-08055C104K4Z4A
- R1703, R1704: symbol Device:R -> partdb:CR0805-JW-471ELF; Category (none) -> Widerstand/Dickfilmwiderstand; MPN (none) -> CR0805-JW-471ELF; Manufacturer (none) -> Bourns; Manufacturing Status (none) -> Active; Mass (none) -> 0.006 g; Mouser SPN (none) -> 652-CR0805JW-471ELF; Part-DB Footprint (none) -> 0805; Part-DB ID (none) -> 307; Part-DB URL (none) -> https://inventory.lan/de/part/307/info; Stock (none) -> 25; Storage Location (none) -> Sortierregal; manf# CR0805-JW-471GLF -> CR0805-JW-471ELF; mouser# 652-CR0805-JW-471GLF -> 652-CR0805JW-471ELF
- R1706: symbol Device:R -> partdb:CR0805-JW-182ELF; Category (none) -> Widerstand/Dickfilmwiderstand; MPN (none) -> CR0805-JW-182ELF; Manufacturer (none) -> Bourns; Manufacturing Status (none) -> Active; Mass (none) -> 0.0055 g; Mouser SPN (none) -> 652-CR0805JW-182ELF; Part-DB Footprint (none) -> 0805; Part-DB ID (none) -> 350; Part-DB URL (none) -> https://inventory.lan/de/part/350/info; Stock (none) -> 0; manf# CR0805-FX-1801GLF -> CR0805-JW-182ELF; mouser# 652-CR0805-FX-1801GLF -> 652-CR0805JW-182ELF
