File: gateway/Ethernet.kicad_sch (KiCad schematic)
At the start: 25 parts, among them IC1701 TLP293, M1701 Ag5400, X1701 Ethernet

Commit message: Prepare Release 1.0.0
Co-Authored-By: Claude Opus 5.5 <noreply@anthropic.com>
Parts:
- renumbered C1701 to C1601, C1702 to C1602, C1703 to C1603, C1704 to C1604, C1705 to C1605, C1706 to C1606, C1707 to C1607, D1701 to D1601, D1702 to D1602, D1703 to D1603, D1704 to D1604, IC1701 to IC1601, M1701 to M1601, R1701 to R1601, R1702 to R1602, R1706 to R1603, R1703 to R1604, R1704 to R1605, R1705 to R1606, TP1705 to TP1601, TP1701 to TP1602, TP1702 to TP1603, TP1703 to TP1604, TP1704 to TP1605, X1701 to X1601
