File: gateway/Interfaces.kicad_sch (KiCad schematic)
At the start: 4 parts, among them X703 USB_C_Plug_USB2.0

Commit message: Working on layout
Parts:
- R707: footprint (none) -> Resistor_SMD:R_0805_2012Metric; manf (none) -> YAGEO; manf# (none) -> RC0805FR-075K1L; mouser# (none) -> 603-RC0805FR-075K1L
- R810: footprint (none) -> Resistor_SMD:R_0805_2012Metric; manf (none) -> YAGEO; manf# (none) -> RC0805FR-073KL; mouser# (none) -> 603-RC0805FR-073KL
Changed lines of the file:
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@@
 			)
 		)
-		(property "Footprint" ""
+		(property "Footprint" "Resistor_SMD:R_0805_2012Metric"
 			(at 55.372 262.89 90)
 			(hide yes)
@@
 			)
 		)
-		(property "Datasheet" ""
+		(property "Datasheet" "https://www.mouser.com/catalog/specsheets/YAGEO_PYu_RC_Group_51_RoHS_L_12.pdf"
 			(at 57.15 262.89 0)
 			(hide yes)
@@
 			)
 		)
-		(property "manf" ""
-			(at 57.15 262.89 0)
-			(hide yes)
-			(show_name no)
-			(do_not_autoplace no)
-			(effects
-				(font
-					(size 1.27 1.27)
-				)
-			)
-		)
-		(property "manf#" ""
-			(at 57.15 262.89 0)
-			(hide yes)
-			(show_name no)
-			(do_not_autoplace no)
-			(effects
-				(font
-					(size 1.27 1.27)
-				)
-			)
-		)
-		(property "mouser#" ""
+		(property "manf" "YAGEO"
+			(at 57.15 262.89 0)
+			(hide yes)
+			(show_name no)
+			(do_not_autoplace no)
+			(effects
+				(font
+					(size 1.27 1.27)
+				)
+			)
+		)
+		(property "manf#" "RC0805FR-075K1L"
+			(at 57.15 262.89 0)
+			(hide yes)
+			(show_name no)
+			(do_not_autoplace no)
+			(effects
+				(font
+					(size 1.27 1.27)
+				)
+			)
+		)
+		(property "mouser#" "603-RC0805FR-075K1L"
 			(at 57.15 262.89 0)
 			(hide yes)
@@
 			)
 		)
-		(property "Footprint" ""
+		(property "Footprint" "Resistor_SMD:R_0805_2012Metric"
 			(at 212.598 261.62 90)
 			(hide yes)
@@
 			)
 		)
-		(property "Datasheet" ""
+		(property "Datasheet" "https://www.mouser.com/catalog/specsheets/YAGEO_PYu_RC_Group_51_RoHS_L_12.pdf"
 			(at 210.82 261.62 0)
 			(hide yes)
@@
 			)
 		)
-		(property "manf" ""
-			(at 210.82 261.62 0)
-			(hide yes)
-			(show_name no)
-			(do_not_autoplace no)
-			(effects
-				(font
-					(size 1.27 1.27)
-				)
-			)
-		)
-		(property "manf#" ""
-			(at 210.82 261.62 0)
-			(hide yes)
-			(show_name no)
-			(do_not_autoplace no)
-			(effects
-				(font
-					(size 1.27 1.27)
-				)
-			)
-		)
-		(property "mouser#" ""
-			(at 210.82 261.62 0)
-			(hide yes)
+		(property "manf" "YAGEO"
+			(at 210.82 261.62 0)
+			(hide yes)
+			(show_name no)
+			(do_not_autoplace no)
+			(effects
+				(font
+					(size 1.27 1.27)
+				)
+			)
+		)
+		(property "manf#" "RC0805FR-073KL"
+			(at 210.82 261.62 0)
+			(hide yes)
+			(show_name no)
+			(do_not_autoplace no)
+			(effects
+				(font
+					(size 1.27 1.27)
+				)
+			)
+		)
+		(property "mouser#" "603-RC0805FR-073KL"
+			(at 210.82 261.62 0)
+			(hide yes)
