File: gateway/WmBus.kicad_sch (KiCad schematic)
At the start: 24 parts, among them IC1401 MIC5317-3.3xM5, IC1402 74LVC1G07, IC1403 TXB0102DCT, M1401 iM891A-XL

Commit message: Working on PCB
Parts:
- removed IC1401: MIC5317-3.3xM5, Package_TO_SOT_SMD:SOT-23-5, symbol Regulator_Linear:MIC5317-3.3xM5
- removed TP1404, TP1405, TP1406: (no value), Testpoints_Kampi:TestPoint_Pad_1.0x1.0mm, symbol Connector:TestPoint
- added IC1401: TLV75733PDBV, Package_TO_SOT_SMD:SOT-23-5, symbol Regulator_Linear:TLV75733PDBV
- TP1401, TP1402, TP1403: value (none) -> ~
Connections:
- net +3V3: now also IC1401.5 (OUT)
- net +5V: now also IC1401.1 (IN)
- net GND: now also IC1401.2 (GND)
- net wM-Bus-Power-Enable: now also IC1401.3 (EN)
- new net: M1401.1 (P1), M1401.10 (P10), M1401.11 (P11), M1401.12 (P12), M1401.13 (P13), M1401.14 (P14), M1401.2 (P2), M1401.20 (P20), M1401.21 (P21), M1401.22 (P22), M1401.23 (P23), M1401.3 (P3), M1401.4 (P4), M1401.6 (P6), M1401.8 (P8), M1401.9 (P9)
