File: gateway/LoRa.kicad_sch (KiCad schematic)
At the start: 16 parts, among them IC1001 MIC5317-3.3xM5, IC1002 74LVC1G07, X1001 LoRa

Commit message: Add INA219 for current measurement
Parts:
- renumbered AE1001 to AE1101, C1001 to C1101, C1002 to C1102, H1001 to H1101, H1002 to H1102, IC1001 to IC1101, IC1002 to IC1102, LED1001 to LED1101, MP1001 to MP1101, R1001 to R1101, R1002 to R1102, R1003 to R1103, TP1001 to TP1101, TP1002 to TP1102, TP1003 to TP1103, X1001 to X1101
Changed lines of the file:
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@@
 	(title_block
 		(title "LoRa")
-		(date "2025-06-05")
+		(date "2026-07-09")
 		(rev "${REVISION}")
 		(company "${COMPANY}")
@@
 		(in_pos_files yes)
 		(dnp no)
-		(property "Reference" "#PWR01009"
+		(property "Reference" "#PWR01109"
 			(at 201.93 172.72 0)
 			(hide yes)
@@
 			(project "Gateway"
 				(path "/d5742f03-3b1a-42e5-a384-018bd4b919aa/c5103ceb-5325-4a84-a025-9638a412984e/3c9d5f3c-b2fb-4756-9da0-aea6b09e18b6"
-					(reference "#PWR01009")
+					(reference "#PWR01109")
 					(unit 1)
 				)
@@
 		(dnp no)
 		(fields_autoplaced yes)
-		(property "Reference" "R1002"
+		(property "Reference" "R1102"
 			(at 99.06 256.5399 0)
 			(show_name no)
@@
 			(project "Gateway"
 				(path "/d5742f03-3b1a-42e5-a384-018bd4b919aa/c5103ceb-5325-4a84-a025-9638a412984e/3c9d5f3c-b2fb-4756-9da0-aea6b09e18b6"
-					(reference "R1002")
+					(reference "R1102")
 					(unit 1)
 				)
@@
 		(dnp no)
 		(fields_autoplaced yes)
-		(property "Reference" "IC1001"
+		(property "Reference" "IC1101"
 			(at 67.31 237.49 0)
 			(show_name no)
@@
 			(project "Gateway"
 				(path "/d5742f03-3b1a-42e5-a384-018bd4b919aa/c5103ceb-5325-4a84-a025-9638a412984e/3c9d5f3c-b2fb-4756-9da0-aea6b09e18b6"
-					(reference "IC1001")
+					(reference "IC1101")
 					(unit 1)
 				)
@@
 		(dnp no)
 		(fields_autoplaced yes)
-		(property "Reference" "#PWR01004"
+		(property "Reference" "#PWR01104"
 			(at 67.31 269.24 0)
 			(hide yes)
@@
 			(project "Gateway"
 				(path "/d5742f03-3b1a-42e5-a384-018bd4b919aa/c5103ceb-5325-4a84-a025-9638a412984e/3c9d5f3c-b2fb-4756-9da0-aea6b09e18b6"
-					(reference "#PWR01004")
+					(reference "#PWR01104")
 					(unit 1)
 				)
@@
 		(dnp no)
 		(fields_autoplaced yes)
-		(property "Reference" "#PWR01001"
+		(property "Reference" "#PWR01101"
 			(at 39.37 246.38 0)
 			(hide yes)
@@
 			(project "Gateway"
 				(path "/d5742f03-3b1a-42e5-a384-018bd4b919aa/c5103ceb-5325-4a84-a025-9638a412984e/3c9d5f3c-b2fb-4756-9da0-aea6b09e18b6"
-					(reference "#PWR01001")
+					(reference "#PWR01101")
 					(unit 1)
 				)
@@
 		(dnp no)
 		(fields_autoplaced yes)
-		(property "Reference" "AE1001"
+		(property "Reference" "AE1101"
 			(at 203.2 274.9549 0)
 			(show_name no)
@@
 			(project "Gateway"
 				(path "/d5742f03-3b1a-42e5-a384-018bd4b919aa/c5103ceb-5325-4a84-a025-9638a412984e/3c9d5f3c-b2fb-4756-9da0-aea6b09e18b6"
-					(reference "AE1001")
+					(reference "AE1101")
 					(unit 1)
 				)
@@
 		(dnp no)
 		(fields_autoplaced yes)
-		(property "Reference" "#PWR01005"
+		(property "Reference" "#PWR01105"
 			(at 86.36 269.24 0)
 			(hide yes)
@@
 			(project "Gateway"
 				(path "/d5742f03-3b1a-42e5-a384-018bd4b919aa/c5103ceb-5325-4a84-a025-9638a412984e/3c9d5f3c-b2fb-4756-9da0-aea6b09e18b6"
-					(reference "#PWR01005")
+					(reference "#PWR01105")
 					(unit 1)
 				)
@@
 		(in_pos_files no)
 		(dnp no)
-		(property "Reference" "TP1001"
+		(property "Reference" "TP1101"
 			(at 52.07 237.9979 0)
 			(show_name no)
@@
 			(project "Gateway"
 				(path "/d5742f03-3b1a-42e5-a384-018bd4b919aa/c5103ceb-5325-4a84-a025-9638a412984e/3c9d5f3c-b2fb-4756-9da0-aea6b09e18b6"
-					(reference "TP1001")
+					(reference "TP1101")
 					(unit 1)
 				)
@@
 		(dnp no)
 		(fields_autoplaced yes)
-		(property "Reference" "#PWR01003"
+		(property "Reference" "#PWR01103"
 			(at 54.61 269.24 0)
 			(hide yes)
@@
 			(project "Gateway"
 				(path "/d5742f03-3b1a-42e5-a384-018bd4b919aa/c5103ceb-5325-4a84-a025-9638a412984e/3c9d5f3c-b2fb-4756-9da0-aea6b09e18b6"
-					(reference "#PWR01003")
+					(reference "#PWR01103")
 					(unit 1)
 				)
@@
 		(in_pos_files yes)
 		(dnp no)
-		(property "Reference" "C1001"
+		(property "Reference" "C1101"
 			(at 35.56 250.1899 0)
 			(show_name no)
@@
 			(project "Gateway"
 				(path "/d5742f03-3b1a-42e5-a384-018bd4b919aa/c5103ceb-5325-4a84-a025-9638a412984e/3c9d5f3c-b2fb-4756-9da0-aea6b09e18b6"
-					(reference "C1001")
+					(reference "C1101")
 					(unit 1)
 				)
@@
 		(in_pos_files no)
 		(dnp no)
-		(property "Reference" "TP1003"
+		(property "Reference" "TP1103"
 			(at 128.27 164.5921 0)
 			(show_name no)
@@
 			(project "Gateway"
 				(path "/d5742f03-3b1a-42e5-a384-018bd4b919aa/c5103ceb-5325-4a84-a025-9638a412984e/3c9d5f3c-b2fb-4756-9da0-aea6b09e18b6"
-					(reference "TP1003")
+					(reference "TP1103")
 					(unit 1)
 				)
@@
 		(dnp no)
 		(fields_autoplaced yes)
-		(property "Reference" "#PWR01006"
+		(property "Reference" "#PWR01106"
 			(at 101.6 269.24 0)
 			(hide yes)
@@
 			(project "Gateway"
 				(path "/d5742f03-3b1a-42e5-a384-018bd4b919aa/c5103ceb-5325-4a84-a025-9638a412984e/3c9d5f3c-b2fb-4756-9da0-aea6b09e18b6"
-					(reference "#PWR01006")
+					(reference "#PWR01106")
 					(unit 1)
 				)
@@
 		(in_pos_files yes)
 		(dnp no)
-		(property "Reference" "C1002"
+		(property "Reference" "C1102"
 			(at 82.55 250.1899 0)
 			(show_name no)
@@
 			(project "Gateway"
 				(path "/d5742f03-3b1a-42e5-a384-018bd4b919aa/c5103ceb-5325-4a84-a025-9638a412984e/3c9d5f3c-b2fb-4756-9da0-aea6b09e18b6"
-					(reference "C1002")
+					(reference "C1102")
 					(unit 1)
 				)
@@
 		(dnp no)
 		(fields_autoplaced yes)
-		(property "Reference" "H1002"
+		(property "Reference" "H1102"
 			(at 182.88 276.8599 0)
 			(show_name no)
@@
 			(project "Gateway"
 				(path "/d5742f03-3b1a-42e5-a384-018bd4b919aa/c5103ceb-5325-4a84-a025-9638a412984e/3c9d5f3c-b2fb-4756-9da0-aea6b09e18b6"
-					(reference "H1002")
+					(reference "H1102")
 					(unit 1)
 				)
@@
 		(in_pos_files yes)
 		(dnp no)
-		(property "Reference" "X1001"
+		(property "Reference" "X1101"
 			(at 185.42 101.6 0)
 			(show_name no)
@@
 			(project "Gateway"
 				(path "/d5742f03-3b1a-42e5-a384-018bd4b919aa/c5103ceb-5325-4a84-a025-9638a412984e/3c9d5f3c-b2fb-4756-9da0-aea6b09e18b6"
-					(reference "X1001")
+					(reference "X1101")
 					(unit 1)
 				)
@@
 		(dnp no)
 		(fields_autoplaced yes)
-		(property "Reference" "#PWR01002"
+		(property "Reference" "#PWR01102"
 			(at 39.37 269.24 0)
 			(hide yes)
@@
 			(project "Gateway"
 				(path "/d5742f03-3b1a-42e5-a384-018bd4b919aa/c5103ceb-5325-4a84-a025-9638a412984e/3c9d5f3c-b2fb-4756-9da0-aea6b09e18b6"
-					(reference "#PWR01002")
+					(reference "#PWR01102")
 					(unit 1)
 				)
@@
 		(in_pos_files no)
 		(dnp yes)
-		(property "Reference" "R1001"
+		(property "Reference" "R1101"
 			(at 52.07 250.1899 0)
 			(show_name no)
@@
 			(project "Gateway"
 				(path "/d5742f03-3b1a-42e5-a384-018bd4b919aa/c5103ceb-5325-4a84-a025-9638a412984e/3c9d5f3c-b2fb-4756-9da0-aea6b09e18b6"
-					(reference "R1001")
+					(reference "R1101")
 					(unit 1)
 				)
@@
 		(in_pos_files yes)
 		(dnp no)
-		(property "Reference" "R1003"
+		(property "Reference" "R1103"
 			(at 170.18 128.2699 0)
 			(show_name no)
@@
 			(project "Gateway"
 				(path "/d5742f03-3b1a-42e5-a384-018bd4b919aa/c5103ceb-5325-4a84-a025-9638a412984e/3c9d5f3c-b2fb-4756-9da0-aea6b09e18b6"
-					(reference "R1003")
+					(reference "R1103")
 					(unit 1)
 				)
@@
 		(dnp no)
 		(fields_autoplaced yes)
-		(property "Reference" "#PWR01008"
+		(property "Reference" "#PWR01108"
 			(at 143.51 176.53 0)
 			(hide yes)
@@
 			(project "Gateway"
 				(path "/d5742f03-3b1a-42e5-a384-018bd4b919aa/c5103ceb-5325-4a84-a025-9638a412984e/3c9d5f3c-b2fb-4756-9da0-aea6b09e18b6"
-					(reference "#PWR01008")
+					(reference "#PWR01108")
 					(unit 1)
 				)
@@
 		(dnp no)
 		(fields_autoplaced yes)
-		(property "Reference" "#PWR01007"
+		(property "Reference" "#PWR01107"
 			(at 143.51 151.13 0)
 			(hide yes)
@@
 			(project "Gateway"
 				(path "/d5742f03-3b1a-42e5-a384-018bd4b919aa/c5103ceb-5325-4a84-a025-9638a412984e/3c9d5f3c-b2fb-4756-9da0-aea6b09e18b6"
-					(reference "#PWR01007")
+					(reference "#PWR01107")
 					(unit 1)
 				)
@@
 		(in_pos_files no)
 		(dnp no)
-		(property "Reference" "H1001"
+		(property "Reference" "H1101"
 			(at 171.45 276.8599 0)
 			(show_name no)
@@
 			(project "Gateway"
 				(path "/d5742f03-3b1a-42e5-a384-018bd4b919aa/c5103ceb-5325-4a84-a025-9638a412984e/3c9d5f3c-b2fb-4756-9da0-aea6b09e18b6"
-					(reference "H1001")
+					(reference "H1101")
 					(unit 1)
 				)
@@
 		(dnp no)
 		(fields_autoplaced yes)
-		(property "Reference" "IC1002"
+		(property "Reference" "IC1102"
 			(at 160.02 152.3298 0)
 			(show_name no)
@@
 			(project "Gateway"
 				(path "/d5742f03-3b1a-42e5-a384-018bd4b919aa/c5103ceb-5325-4a84-a025-9638a412984e/3c9d5f3c-b2fb-4756-9da0-aea6b09e18b6"
-					(reference "IC1002")
+					(reference "IC1102")
 					(unit 1)
 				)
@@
 		(dnp no)
 		(fields_autoplaced yes)
-		(property "Reference" "TP1002"
+		(property "Reference" "TP1102"
 			(at 88.9 237.9979 0)
 			(show_name no)
@@
 			(project "Gateway"
 				(path "/d5742f03-3b1a-42e5-a384-018bd4b919aa/c5103ceb-5325-4a84-a025-9638a412984e/3c9d5f3c-b2fb-4756-9da0-aea6b09e18b6"
-					(reference "TP1002")
+					(reference "TP1102")
 					(unit 1)
 				)
@@
 		(in_pos_files no)
 		(dnp no)
-		(property "Reference" "MP1001"
+		(property "Reference" "MP1101"
 			(at 145.034 274.32 0)
 			(show_name no)
@@
 			(project "Gateway"
 				(path "/d5742f03-3b1a-42e5-a384-018bd4b919aa/c5103ceb-5325-4a84-a025-9638a412984e/3c9d5f3c-b2fb-4756-9da0-aea6b09e18b6"
-					(reference "MP1001")
+					(reference "MP1101")
 					(unit 1)
 				)
@@
 		(dnp no)
 		(fields_autoplaced yes)
-		(property "Reference" "LED1001"
+		(property "Reference" "LED1101"
 			(at 97.79 249.2374 90)
 			(show_name no)
@@
 			(project "Gateway"
 				(path "/d5742f03-3b1a-42e5-a384-018bd4b919aa/c5103ceb-5325-4a84-a025-9638a412984e/3c9d5f3c-b2fb-4756-9da0-aea6b09e18b6"
-					(reference "LED1001")
+					(reference "LED1101")
 					(unit 1)
 				)

Commit message: Improving Thread
- Add boot signal for Thread MCU
- Add debug LED for nRF5340
Parts:
- TP1101, TP1102, TP1103: value ~ -> (none)
Changed lines of the file:
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@@
 	)
 	(rectangle
+		(start 86.36 74.93)
+		(end 261.62 203.2)
+		(stroke
+			(width 1)
+			(type default)
+			(color 200 200 200 1)
+		)
+		(fill
+			(type none)
+		)
+	)
+	(rectangle
 		(start 13.97 223.5199)
 		(end 119.38 283.0697)
@@
 		)
 	)
+	(text_box "LoRa Concentrator"
+		(exclude_from_sim no)
+		(at 87.63 193.04 0)
+		(size 172.72 8.89)
+		(margins 1.9049 1.9049 1.9049 1.9049)
+		(stroke
+			(width -0.0001)
+			(type solid)
+		)
+		(fill
+			(type none)
+		)
+		(effects
+			(font
+				(face "Times New Roman")
+				(size 2.54 2.54)
+				(thickness 0.508)
+				(bold yes)
+				(color 162 22 34 1)
+			)
+			(justify bottom)
+		)
+	)
 	(junction
 		(at 39.37 243.84)
@@
 			)
 		)
-		(property "Value" "~"
+		(property "Value" ""
 			(at 52.07 240.5379 0)
 			(show_name no)
@@
 			)
 		)
-		(property "Value" "~"
+		(property "Value" ""
 			(at 128.27 162.0521 0)
 			(hide yes)
@@
 			)
 		)
-		(property "Value" "~"
+		(property "Value" ""
 			(at 88.9 240.5379 0)
 			(show_name no)

Commit message: Working on PCB
Parts:
- removed IC1101: MIC5317-3.3xM5, Package_TO_SOT_SMD:SOT-23-5, symbol Regulator_Linear:MIC5317-3.3xM5
- added IC1101: TLV75733PDBV, Package_TO_SOT_SMD:SOT-23-5, symbol Regulator_Linear:TLV75733PDBV
- TP1101, TP1102, TP1103: value (none) -> ~
Connections:
- net +3V3: now also IC1101.5 (OUT)
- net +5V: now also IC1101.1 (IN)
- net GND: now also IC1101.2 (GND)
- net LoRa-Power-Enable: now also IC1101.3 (EN)
Changed lines of the file:
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@@
-	)
-	(symbol
-		(lib_id "Regulator_Linear:MIC5317-3.3xM5")
-		(at 67.31 246.38 0)
-		(unit 1)
-		(body_style 1)
-		(exclude_from_sim no)
-		(in_bom yes)
-		(on_board yes)
-		(in_pos_files yes)
-		(dnp no)
-		(fields_autoplaced yes)
-		(property "Reference" "IC1101"
-			(at 67.31 237.49 0)
-			(show_name no)
-			(do_not_autoplace no)
-			(effects
-				(font
-					(size 1.27 1.27)
-				)
-			)
-		)
-		(property "Value" "MIC5317-3.3xM5"
-			(at 67.31 240.03 0)
-			(show_name no)
-			(do_not_autoplace no)
-			(effects
-				(font
-					(size 1.27 1.27)
-				)
-			)
-		)
-		(property "Footprint" "Package_TO_SOT_SMD:SOT-23-5"
-			(at 67.31 237.49 0)
-			(hide yes)
-			(show_name no)
-			(do_not_autoplace no)
-			(effects
-				(font
-					(size 1.27 1.27)
-				)
-			)
-		)
-		(property "Datasheet" "https://ww1.microchip.com/downloads/aemDocuments/documents/OTH/ProductDocuments/DataSheets/MIC5317-High-Performance-Single-150mA-LDO-DS20006195B.pdf"
-			(at 59.69 226.06 0)
-			(hide yes)
-			(show_name no)
-			(do_not_autoplace no)
-			(effects
-				(font
-					(size 1.27 1.27)
-				)
-			)
-		)
-		(property "Description" "150mA Low-dropout Voltage Regulator, Vout 3.3V, Vin up to 6V, SOT23-5"
-			(at 67.31 246.38 0)
-			(hide yes)
-			(show_name no)
-			(do_not_autoplace no)
-			(effects
-				(font
-					(size 1.27 1.27)
-				)
-			)
-		)
-		(property "manf" "Microchip Technology"
-			(at 67.31 246.38 0)
-			(hide yes)
-			(show_name no)
-			(do_not_autoplace no)
-			(effects
-				(font
-					(size 1.27 1.27)
-				)
-			)
-		)
-		(property "manf#" "MIC5317-3.3YM5-TR"
-			(at 67.31 246.38 0)
-			(hide yes)
-			(show_name no)
-			(do_not_autoplace no)
-			(effects
-				(font
-					(size 1.27 1.27)
-				)
-			)
-		)
-		(property "mouser#" "998-MIC5317-3.3YM5-TR"
-			(at 67.31 246.38 0)
-			(hide yes)
-			(show_name no)
-			(do_not_autoplace no)
-			(effects
-				(font
-					(size 1.27 1.27)
-				)
-			)
-		)
-		(pin "1"
-		)
-		(pin "3"
-		)
-		(pin "2"
-		)
-		(pin "4"
-		)
-		(pin "5"
-		)
-		(instances
-			(project "Gateway"
-				(path "/d5742f03-3b1a-42e5-a384-018bd4b919aa/c5103ceb-5325-4a84-a025-9638a412984e/3c9d5f3c-b2fb-4756-9da0-aea6b09e18b6"
-					(reference "IC1101")
-					(unit 1)
-				)
-			)
-		)
 	)
 	(symbol
@@
 			)
 		)
-		(property "Value" ""
+		(property "Value" "~"
 			(at 52.07 240.5379 0)
 			(show_name no)
@@
 			)
 		)
-		(property "Value" ""
+		(property "Value" "~"
 			(at 128.27 162.0521 0)
 			(hide yes)
@@
 	)
 	(symbol
+		(lib_id "Regulator_Linear:TLV75733PDBV")
+		(at 67.31 246.38 0)
+		(unit 1)
+		(body_style 1)
+		(exclude_from_sim no)
+		(in_bom yes)
+		(on_board yes)
+		(in_pos_files yes)
+		(dnp no)
+		(fields_autoplaced yes)
+		(property "Reference" "IC1101"
+			(at 67.31 237.49 0)
+			(show_name no)
+			(do_not_autoplace no)
+			(effects
+				(font
+					(size 1.27 1.27)
+				)
+			)
+		)
+		(property "Value" "TLV75733PDBV"
+			(at 67.31 240.03 0)
+			(show_name no)
+			(do_not_autoplace no)
+			(effects
+				(font
+					(size 1.27 1.27)
+				)
+			)
+		)
+		(property "Footprint" "Package_TO_SOT_SMD:SOT-23-5"
+			(at 67.31 238.125 0)
+			(hide yes)
+			(show_name no)
+			(do_not_autoplace no)
+			(effects
+				(font
+					(size 1.27 1.27)
+					(italic yes)
+				)
+			)
+		)
+		(property "Datasheet" "https://www.ti.com/lit/ds/symlink/tlv757p.pdf"
+			(at 67.31 245.11 0)
+			(hide yes)
+			(show_name no)
+			(do_not_autoplace no)
+			(effects
+				(font
+					(size 1.27 1.27)
+				)
+			)
+		)
+		(property "Description" "1A Low IQ Small Size Low Dropout Voltage Regulator, Fixed Output 3.3V, SOT-23-5"
+			(at 67.31 246.38 0)
+			(hide yes)
+			(show_name no)
+			(do_not_autoplace no)
+			(effects
+				(font
+					(size 1.27 1.27)
+				)
+			)
+		)
+		(property "manf" "Texas Instruments"
+			(at 67.31 246.38 0)
+			(hide yes)
+			(show_name no)
+			(do_not_autoplace no)
+			(effects
+				(font
+					(size 1.27 1.27)
+				)
+			)
+		)
+		(property "manf#" "TLV75733PDBVR"
+			(at 67.31 246.38 0)
+			(hide yes)
+			(show_name no)
+			(do_not_autoplace no)
+			(effects
+				(font
+					(size 1.27 1.27)
+				)
+			)
+		)
+		(property "mouser#" "595-TLV75733PDBVR"
+			(at 67.31 246.38 0)
+			(hide yes)
+			(show_name no)
+			(do_not_autoplace no)
+			(effects
+				(font
+					(size 1.27 1.27)
+				)
+			)
+		)
+		(pin "2"
+		)
+		(pin "3"
+		)
+		(pin "5"
+		)
+		(pin "1"
+		)
+		(pin "4"
+		)
+		(instances
+			(project "Gateway"
+				(path "/d5742f03-3b1a-42e5-a384-018bd4b919aa/c5103ceb-5325-4a84-a025-9638a412984e/3c9d5f3c-b2fb-4756-9da0-aea6b09e18b6"
+					(reference "IC1101")
+					(unit 1)
+				)
+			)
+		)
+	)
+	(symbol
 		(lib_id "power:+1V8")
 		(at 143.51 147.32 0)
@@
 			)
 		)
-		(property "Value" ""
+		(property "Value" "~"
 			(at 88.9 240.5379 0)
 			(show_name no)
@@
 			(at 101.6 248.92 0)
 			(hide yes)
-			(show_name no)
-			(do_not_autoplace no)
-			(effects
-				(font
-					(size 1.27 1.27)
-				)
-			)
-		)
-		(property "Sim.Pins" "1=K 2=A"
-			(at 101.6 248.92 0)
-			(hide yes)

Commit message: Smaller changes
Parts:
- H1101, H1102: symbol Mechanical_Kampi:MountingHole -> Mechanical:Spacer
Changed lines of the file:
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@@
 	)
 	(symbol
-		(lib_id "Mechanical_Kampi:MountingHole")
+		(lib_id "Mechanical:Spacer")
 		(at 180.34 278.13 0)
 		(unit 1)
@@
 	)
 	(symbol
-		(lib_id "Mechanical_Kampi:MountingHole")
+		(lib_id "Mechanical:Spacer")
 		(at 173.99 278.13 0)
 		(mirror y)
