File: gateway/LoRa.kicad_sch (KiCad schematic)
At the start: 16 parts, among them IC1101 TLV75733PDBV, IC1102 74LVC1G07, X1101 LoRa

Commit message: Working on revision 1.0.0
Parts:
- C1101, C1102: symbol Device:C -> partdb:08053G105MAT2A; Category (none) -> Kondensator/MLCC; MPN (none) -> 08053G105MAT2A; Manufacturer (none) -> KYOCERA AVX; Manufacturing Status (none) -> Active; Mass (none) -> 0.006 g; Mouser SPN (none) -> 581-08053G105MAT2A; Part-DB Footprint (none) -> 0805; Part-DB ID (none) -> 349; Part-DB URL (none) -> https://inventory.lan/de/part/349/info; Stock (none) -> 0; manf# 08056C105MAT2A -> 08053G105MAT2A; mouser# 581-08056C105MAT2A -> 581-08053G105MAT2A
- H1101, H1102: symbol Mechanical:Spacer -> partdb:9774015151R; Category (none) -> Mechanik/Abstandshalter; MPN (none) -> 9774015151R; Manufacturer (none) -> Wurth Elektronik; Manufacturing Status (none) -> Active; Mass (none) -> 0.238 g; Mouser SPN (none) -> 710-9774015151R; Part-DB Footprint (none) -> WA-SMSI M2.5; Part-DB ID (none) -> 384; Part-DB URL (none) -> https://inventory.lan/de/part/384/info; Stock (none) -> 0; now in the parts list
- LED1101: symbol Device:LED -> partdb:SM0805YC; Category (none) -> Diode/LED/Gelb; MPN (none) -> SM0805YC; Manufacturer (none) -> Bivar; Manufacturing Status (none) -> Active; Mass (none) -> 0.004 g; Mouser SPN (none) -> 749-SM0805YC; Part-DB Footprint (none) -> 0805; Part-DB ID (none) -> 324; Part-DB URL (none) -> https://inventory.lan/de/part/324/info; Stock (none) -> 0
- MP1101: symbol Mechanical_Kampi:Light_Pipe -> Mechanical:Light_Pipe
- R1101: symbol Device:R -> partdb:CR0805-FX-1002ELF; Category (none) -> Widerstand/Dickfilmwiderstand; MPN (none) -> CR0805-FX-1002ELF; Manufacturer (none) -> Bourns; Manufacturing Status (none) -> Active; Mass (none) -> 0.006 g; Mouser SPN (none) -> 652-CR0805FX-1002ELF; Part-DB Footprint (none) -> 0805; Part-DB ID (none) -> 343; Part-DB URL (none) -> https://inventory.lan/de/part/343/info; Stock (none) -> 0; manf# CR0805-FX-1002GLF -> CR0805-FX-1002ELF; mouser# 652-CR0805-FX-1002GLF -> 652-CR0805FX-1002ELF
- R1103: symbol Device:R -> partdb:CR0805-FX-1002ELF; Category (none) -> Widerstand/Dickfilmwiderstand; MPN (none) -> CR0805-FX-1002ELF; Manufacturer (none) -> Bourns; Manufacturing Status (none) -> Active; Mass (none) -> 0.006 g; Mouser SPN (none) -> 652-CR0805FX-1002ELF; Part-DB Footprint (none) -> 0805; Part-DB ID (none) -> 343; Part-DB URL (none) -> https://inventory.lan/de/part/343/info; Stock (none) -> 0; manf# CR0805-JW-103GLF -> CR0805-FX-1002ELF; mouser# 652-CR0805-JW-103GLF -> 652-CR0805FX-1002ELF
