File: gateway/LoRa.kicad_sch (KiCad schematic)
At the start: 16 parts, among them IC1101 TLV75733PDBV, IC1102 74LVC1G07, X1101 LoRa

Commit message: Prepare Release 1.0.0
Co-Authored-By: Claude Opus 5.5 <noreply@anthropic.com>
Parts:
- IC1001: renamed from IC1101; manf# TLV75733PDBVR -> TLV75733PDBVT; mouser# 595-TLV75733PDBVR -> 595-TLV75733PDBVT
- IC1002: renamed from IC1102; manf Diodes Incorporated -> Nexperia; manf# 74LVC1G07QSE-7 -> 74LVC1G07GW,125; mouser# 621-74LVC1G07QSE-7 -> 771-74LVC1G07GW-G
- R1002: renamed from R1102; mouser# 652-CR0805-JW-680GLF -> 652-CR0805JW-680GLF
- renumbered AE1101 to AE1001, C1101 to C1001, C1102 to C1002, H1101 to H1001, H1102 to H1002, LED1101 to LED1001, MP1101 to MP1001, R1101 to R1001, R1103 to R1003, TP1101 to TP1001, TP1102 to TP1002, TP1103 to TP1003, X1101 to X1001

Commit message: Update schematic and board
- Use Part-DB symbols, BT901 changed to Keystone 3030TR
- Add the revision text to the board
- Include more parts in BOM and position files

Co-Authored-By: Claude Opus 5.5 <noreply@anthropic.com>
Parts:
- R1001: now in the parts list
Changed lines of the file:
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@@
 		(body_style 1)
 		(exclude_from_sim no)
-		(in_bom no)
+		(in_bom yes)
 		(on_board yes)
-		(in_pos_files no)
+		(in_pos_files yes)
 		(dnp yes)
 		(property "Reference" "R1001"
