File: gateway/NVMe.kicad_sch (KiCad schematic)
At the start: 24 parts, among them IC1601 ST1S14PHR, X1601 SSD

Commit message: Working on revision 1.0.0
Parts:
- C1601, C1602, C1611: symbol Device:C -> partdb:0805X7R106KT1AT; Category (none) -> Kondensator/MLCC; MPN (none) -> 0805X7R106KT1AT; Manufacturer (none) -> KYOCERA AVX; Manufacturing Status (none) -> Active; Mouser SPN (none) -> 581-0805X7R106KT1AT; Part-DB Footprint (none) -> 0805; Part-DB ID (none) -> 331; Part-DB URL (none) -> https://inventory.lan/de/part/331/info; Stock (none) -> 0
- C1603, C1605, C1608, C1609: symbol Device:C -> partdb:08055C104K4Z4A; Category (none) -> Kondensator/MLCC; MPN (none) -> 08055C104K4Z4A; Manufacturer (none) -> KYOCERA AVX; Manufacturing Status (none) -> Active; Mass (none) -> 0.006 g; Mouser SPN (none) -> 581-08055C104K4Z4A; Part-DB Footprint (none) -> 0805; Part-DB ID (none) -> 109; Part-DB URL (none) -> https://inventory.lan/de/part/109/info; Stock (none) -> 6; Storage Location (none) -> Sortierregal; manf# 08053C104M4T4A -> 08055C104K4Z4A; mouser# 581-08053C104M4T4A -> 581-08055C104K4Z4A
- H1601: value 2230 -> Spacer; footprint Wuerth:9774015151R -> Wuerth:9774025151R; symbol Mechanical:Spacer -> partdb:9774025151R; Category (none) -> Mechanik/Abstandshalter; MPN (none) -> 9774025151R; Manufacturer (none) -> Wurth Elektronik; Manufacturing Status (none) -> Active; Mass (none) -> 0.371 g; Mouser SPN (none) -> 710-9774025151R; Part-DB Footprint (none) -> WA-SMSI M2.5; Part-DB ID (none) -> 374; Part-DB URL (none) -> https://inventory.lan/de/part/374/info; Stock (none) -> 0; manf# 9774015151R -> 9774025151R; mouser# 710-9774015151R -> 710-9774025151R
- R1601, R1602, R1607: symbol Device:R -> partdb:RT0805FRE13100KL; Category (none) -> Widerstand/Dünnfilmwiderstand; MPN (none) -> RT0805FRE13100KL; Manufacturer (none) -> YAGEO; Manufacturing Status (none) -> Active; Mass (none) -> 0.006 g; Mouser SPN (none) -> 603-RT0805FRE13100KL; Part-DB Footprint (none) -> 0805; Part-DB ID (none) -> 66; Part-DB URL (none) -> https://inventory.lan/de/part/66/info; Stock (none) -> 4; Storage Location (none) -> Sortierregal; manf Bourns -> YAGEO; manf# CR0805-JW-104GLF -> RT0805FRE13100KL; mouser# 652-CR0805-JW-104GLF -> 603-RT0805FRE13100KL
- R1606: symbol Device:R -> partdb:CR0805-JW-472ELF; Category (none) -> Widerstand/Dickfilmwiderstand; MPN (none) -> CR0805-JW-472ELF; Manufacturer (none) -> Bourns; Manufacturing Status (none) -> Active; Mass (none) -> 0.006 g; Mouser SPN (none) -> 652-CR0805JW-472ELF; Part-DB Footprint (none) -> 0805; Part-DB ID (none) -> 78; Part-DB URL (none) -> https://inventory.lan/de/part/78/info; Stock (none) -> 50; Storage Location (none) -> Sortierregal; mouser# 652-CR0805-JW-472ELF -> 652-CR0805JW-472ELF
