File: gateway/NVMe.kicad_sch (KiCad schematic)
At the start: 24 parts, among them IC1601 ST1S14PHR, X1601 SSD

Commit message: Prepare Release 1.0.0
Co-Authored-By: Claude Opus 5.5 <noreply@anthropic.com>
Parts:
- R1505: renamed from R1605; mouser# 652-CR0805-FX-4872ELF -> 652-CR0805FX-4872ELF
- renumbered C1602 to C1501, C1601 to C1502, C1603 to C1503, C1604 to C1504, C1605 to C1505, C1606 to C1506, C1607 to C1507, C1608 to C1508, C1609 to C1509, C1610 to C1510, C1611 to C1511, D1601 to D1501, H1601 to H1501, IC1601 to IC1501, L1601 to L1501, R1602 to R1501, R1607 to R1502, R1601 to R1503, R1604 to R1504, R1606 to R1506, TP1602 to TP1501, TP1603 to TP1502, X1601 to X1501
