File: gateway/Power Input.kicad_sch (KiCad schematic)
At the start: 21 parts, among them IC701 TPS2121RUXT, IC702 INA219AxD, Q701 BSS123, X701 DC In

Commit message: Working on revision 1.0.0
Parts:
- C702: symbol Device:C -> partdb:08055C104K4Z4A; Category (none) -> Kondensator/MLCC; MPN (none) -> 08055C104K4Z4A; Manufacturer (none) -> KYOCERA AVX; Manufacturing Status (none) -> Active; Mass (none) -> 0.006 g; Mouser SPN (none) -> 581-08055C104K4Z4A; Part-DB Footprint (none) -> 0805; Part-DB ID (none) -> 109; Part-DB URL (none) -> https://inventory.lan/de/part/109/info; Stock (none) -> 6; Storage Location (none) -> Sortierregal; manf# 08053C104M4T4A -> 08055C104K4Z4A; mouser# 581-08053C104M4T4A -> 581-08055C104K4Z4A
- Q701: value BSS123 -> BSS138; symbol Transistor_FET:BSS123 -> partdb:BSS138; Category (none) -> Transistor/N-Kanal; MPN (none) -> BSS138; Manufacturer (none) -> onsemi / Fairchild; Manufacturing Status (none) -> Active; Mass (none) -> 0.008 g; Mouser SPN (none) -> 512-BSS138; Part-DB Footprint (none) -> SOT-23-3; Part-DB ID (none) -> 353; Part-DB URL (none) -> https://inventory.lan/de/part/353/info; Stock (none) -> 0; manf onsemi -> onsemi / Fairchild; manf# BSS123 -> BSS138; mouser# 512-BSS123 -> 512-BSS138
- R702, R703: symbol Device:R -> partdb:CR0805-FX-1002ELF; Category (none) -> Widerstand/Dickfilmwiderstand; MPN (none) -> CR0805-FX-1002ELF; Manufacturer (none) -> Bourns; Manufacturing Status (none) -> Active; Mass (none) -> 0.006 g; Mouser SPN (none) -> 652-CR0805FX-1002ELF; Part-DB Footprint (none) -> 0805; Part-DB ID (none) -> 343; Part-DB URL (none) -> https://inventory.lan/de/part/343/info; Stock (none) -> 0; manf# CR0805-JW-103GLF -> CR0805-FX-1002ELF; mouser# 652-CR0805-JW-103GLF -> 652-CR0805FX-1002ELF
- R705, R706, R707, R708: symbol Device:R -> partdb:CR0805-J/-000ELF; Category (none) -> Widerstand/Dickfilmwiderstand; MPN (none) -> CR0805-J/-000ELF; Manufacturer (none) -> Bourns; Manufacturing Status (none) -> Active; Mass (none) -> 0.006 g; Mouser SPN (none) -> 652-CR0805-J/-000ELF; Part-DB Footprint (none) -> 0805; Part-DB ID (none) -> 322; Part-DB URL (none) -> https://inventory.lan/de/part/322/info; Stock (none) -> 0
- R709: symbol Device:R -> partdb:RT0805FRE13100KL; Category (none) -> Widerstand/Dünnfilmwiderstand; MPN (none) -> RT0805FRE13100KL; Manufacturer (none) -> YAGEO; Manufacturing Status (none) -> Active; Mass (none) -> 0.006 g; Mouser SPN (none) -> 603-RT0805FRE13100KL; Part-DB Footprint (none) -> 0805; Part-DB ID (none) -> 66; Part-DB URL (none) -> https://inventory.lan/de/part/66/info; Stock (none) -> 4; Storage Location (none) -> Sortierregal; manf Bourns -> YAGEO; manf# CR0805-JW-104GLF -> RT0805FRE13100KL; mouser# 652-CR0805-JW-104GLF -> 603-RT0805FRE13100KL
