File: gateway/Power Input.kicad_sch (KiCad schematic)
At the start: 21 parts, among them IC701 TPS2121RUXT, IC702 INA219AxD, Q701 BSS138, X701 DC In

Commit message: Prepare Release 1.0.0
Co-Authored-By: Claude Opus 5.5 <noreply@anthropic.com>
Parts:
- R601: renamed from R711; mouser# 652-CR0805-JW-303ELF -> 652-CR0805JW-303ELF
- R602: renamed from R712; mouser# 652-CR0805-FX-2001ELF -> 652-CR0805FX-2001ELF
- R603: renamed from R701; mouser# 652-CR0805-JW-333ELF -> 652-CR0805JW-333ELF
- R612: renamed from R710; mouser# 652-CR0805-FX-1202ELF -> 652-CR0805FX-1202ELF
- renumbered C701 to C601, C702 to C602, IC701 to IC601, IC702 to IC602, Q701 to Q601, R702 to R604, R703 to R605, R704 to R606, R705 to R607, R706 to R608, R707 to R609, R708 to R610, R709 to R611, TP701 to TP601, TP702 to TP602, TP703 to TP603, X701 to X601
