File: gateway/Zigbee.kicad_sch (KiCad schematic)
At the start: 28 parts, among them IC1201 MIC5317-3.3xM5, IC1202 TXB0102DCT, IC1203 74LVC1G07, IC1204 74LVC1G07, M1201 RF-BM-2652

Commit message: Working on PCB
Parts:
- removed IC1201: MIC5317-3.3xM5, Package_TO_SOT_SMD:SOT-23-5, symbol Regulator_Linear:MIC5317-3.3xM5
- removed TP1204, TP1205: (no value), Testpoints_Kampi:TestPoint_Pad_1.0x1.0mm, symbol Connector:TestPoint
- added IC1201: TLV75733PDBV, Package_TO_SOT_SMD:SOT-23-5, symbol Regulator_Linear:TLV75733PDBV
- TP1201, TP1202, TP1203, TP1206: value (none) -> ~
- renumbered C1204 to C1203, C1203 to C1204
Connections:
- net +3V3: now also IC1201.5 (OUT)
- net +5V: now also IC1201.1 (IN)
- net GND: now also IC1201.2 (GND)
- net Zigbee-Power-Enable: now also IC1201.3 (EN)

Commit message: Working on layout
Connections:
- net CC2652-Boot: no longer names the net of IC1204.4, M1201.16 (DIO15), R1208.2
Changed lines of the file:
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@@
-		)
-	)
-	(label "CC2652-Boot"
-		(at 250.19 97.79 0)
-		(effects
-			(font
-				(size 1.27 1.27)
-			)
-			(justify left bottom)
 		)
 	)

Commit message: Working on revision 1.0.0
Parts:
- C1201, C1202: symbol Device:C -> partdb:08053G105MAT2A; Category (none) -> Kondensator/MLCC; MPN (none) -> 08053G105MAT2A; Manufacturer (none) -> KYOCERA AVX; Manufacturing Status (none) -> Active; Mass (none) -> 0.006 g; Mouser SPN (none) -> 581-08053G105MAT2A; Part-DB Footprint (none) -> 0805; Part-DB ID (none) -> 349; Part-DB URL (none) -> https://inventory.lan/de/part/349/info; Stock (none) -> 0; manf# 08056C105MAT2A -> 08053G105MAT2A; mouser# 581-08056C105MAT2A -> 581-08053G105MAT2A
- C1203, C1204, C1205: symbol Device:C -> partdb:08055C104K4Z4A; Category (none) -> Kondensator/MLCC; MPN (none) -> 08055C104K4Z4A; Manufacturer (none) -> KYOCERA AVX; Manufacturing Status (none) -> Active; Mass (none) -> 0.006 g; Mouser SPN (none) -> 581-08055C104K4Z4A; Part-DB Footprint (none) -> 0805; Part-DB ID (none) -> 109; Part-DB URL (none) -> https://inventory.lan/de/part/109/info; Stock (none) -> 6; Storage Location (none) -> Sortierregal; manf# 08053C104M4T4A -> 08055C104K4Z4A; mouser# 581-08053C104M4T4A -> 581-08055C104K4Z4A
- C1206: symbol Device:C -> partdb:0805X7R106KT1AT; Category (none) -> Kondensator/MLCC; MPN (none) -> 0805X7R106KT1AT; Manufacturer (none) -> KYOCERA AVX; Manufacturing Status (none) -> Active; Mouser SPN (none) -> 581-0805X7R106KT1AT; Part-DB Footprint (none) -> 0805; Part-DB ID (none) -> 331; Part-DB URL (none) -> https://inventory.lan/de/part/331/info; Stock (none) -> 0
- IC1202: value TXB0102DCT -> TXB0102DCU; Category (none) -> IC/Pegelwandler; MPN (none) -> TXB0102DCUR; Manufacturer (none) -> Texas Instruments; Mass (none) -> 0.01 g; Mouser SPN (none) -> 595-TXB0102DCUR; Part-DB Footprint (none) -> VSSOP-8_2.3x2mm_P0.5mm; Part-DB ID (none) -> 280; Part-DB URL (none) -> https://inventory.lan/de/part/280/info; Stock (none) -> 0; manf# TXB0102DCT -> TXB0102DCUR; mouser# 595-TXB0102DCT -> 595-TXB0102DCUR
- LED1201: symbol Device:LED -> partdb:SM0805YC; Category (none) -> Diode/LED/Gelb; MPN (none) -> SM0805YC; Manufacturer (none) -> Bivar; Manufacturing Status (none) -> Active; Mass (none) -> 0.004 g; Mouser SPN (none) -> 749-SM0805YC; Part-DB Footprint (none) -> 0805; Part-DB ID (none) -> 324; Part-DB URL (none) -> https://inventory.lan/de/part/324/info; Stock (none) -> 0
- MP1201: symbol Mechanical_Kampi:Light_Pipe -> Mechanical:Light_Pipe
- R1201: symbol Device:R -> partdb:CR0805-FX-1002ELF; Category (none) -> Widerstand/Dickfilmwiderstand; MPN (none) -> CR0805-FX-1002ELF; Manufacturer (none) -> Bourns; Manufacturing Status (none) -> Active; Mass (none) -> 0.006 g; Mouser SPN (none) -> 652-CR0805FX-1002ELF; Part-DB Footprint (none) -> 0805; Part-DB ID (none) -> 343; Part-DB URL (none) -> https://inventory.lan/de/part/343/info; Stock (none) -> 0; manf# CR0805-FX-1002GLF -> CR0805-FX-1002ELF; mouser# 652-CR0805-FX-1002GLF -> 652-CR0805FX-1002ELF
- R1202, R1203, R1205, R1206: symbol Device:R -> partdb:CR0805-J/-000ELF; Category (none) -> Widerstand/Dickfilmwiderstand; MPN (none) -> CR0805-J/-000ELF; Manufacturer (none) -> Bourns; Manufacturing Status (none) -> Active; Mass (none) -> 0.006 g; Mouser SPN (none) -> 652-CR0805-J/-000ELF; Part-DB Footprint (none) -> 0805; Part-DB ID (none) -> 322; Part-DB URL (none) -> https://inventory.lan/de/part/322/info; Stock (none) -> 0
- R1207, R1208: symbol Device:R -> partdb:CR0805-FX-1002ELF; Category (none) -> Widerstand/Dickfilmwiderstand; MPN (none) -> CR0805-FX-1002ELF; Manufacturer (none) -> Bourns; Manufacturing Status (none) -> Active; Mass (none) -> 0.006 g; Mouser SPN (none) -> 652-CR0805FX-1002ELF; Part-DB Footprint (none) -> 0805; Part-DB ID (none) -> 343; Part-DB URL (none) -> https://inventory.lan/de/part/343/info; Stock (none) -> 0; manf# CR0805-JW-103GLF -> CR0805-FX-1002ELF; mouser# 652-CR0805-JW-103GLF -> 652-CR0805FX-1002ELF
