File: gateway/Zigbee.kicad_sch (KiCad schematic)
At the start: 26 parts, among them IC1201 TLV75733PDBV, IC1202 TXB0102DCU, IC1203 74LVC1G07, IC1204 74LVC1G07, M1201 RF-BM-2652

Commit message: Prepare Release 1.0.0
Co-Authored-By: Claude Opus 5.5 <noreply@anthropic.com>
Parts:
- IC1101: renamed from IC1201; manf# TLV75733PDBVR -> TLV75733PDBVT; mouser# 595-TLV75733PDBVR -> 595-TLV75733PDBVT
- IC1103: renamed from IC1203; manf Diodes Incorporated -> Nexperia; manf# 74LVC1G07QSE-7 -> 74LVC1G07GW,125; mouser# 621-74LVC1G07QSE-7 -> 771-74LVC1G07GW-G
- IC1104: renamed from IC1204; manf Diodes Incorporated -> Nexperia; manf# 74LVC1G07QSE-7 -> 74LVC1G07GW,125; mouser# 621-74LVC1G07QSE-7 -> 771-74LVC1G07GW-G
- R1104: renamed from R1204; mouser# 652-CR0805-JW-680GLF -> 652-CR0805JW-680GLF
- renumbered AE1201 to AE1101, C1201 to C1101, C1202 to C1102, C1203 to C1103, C1204 to C1104, C1205 to C1105, C1206 to C1106, IC1202 to IC1102, LED1201 to LED1101, M1201 to M1101, MP1201 to MP1101, R1201 to R1101, R1202 to R1102, R1203 to R1103, R1205 to R1105, R1206 to R1106, R1207 to R1107, R1208 to R1108, TP1201 to TP1101, TP1202 to TP1102, TP1203 to TP1103, TP1206 to TP1104

Commit message: Update schematic and board
- Use Part-DB symbols, BT901 changed to Keystone 3030TR
- Add the revision text to the board
- Include more parts in BOM and position files

Co-Authored-By: Claude Opus 5.5 <noreply@anthropic.com>
Parts:
- R1101: now in the parts list
Changed lines of the file:
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@@
 		(body_style 1)
 		(exclude_from_sim no)
-		(in_bom no)
+		(in_bom yes)
 		(on_board yes)
-		(in_pos_files no)
+		(in_pos_files yes)
 		(dnp yes)
 		(property "Reference" "R1101"
