File: gateway/wMBus.kicad_sch (KiCad schematic)
At the start: 21 parts, among them IC1401 TLV75733PDBV, IC1402 74LVC1G07, IC1403 TXB0102DCT, M1401 iM891A-XL

Commit message: Working on revision 1.0.0
Parts:
- C1401, C1402: symbol Device:C -> partdb:08053G105MAT2A; Category (none) -> Kondensator/MLCC; MPN (none) -> 08053G105MAT2A; Manufacturer (none) -> KYOCERA AVX; Manufacturing Status (none) -> Active; Mass (none) -> 0.006 g; Mouser SPN (none) -> 581-08053G105MAT2A; Part-DB Footprint (none) -> 0805; Part-DB ID (none) -> 349; Part-DB URL (none) -> https://inventory.lan/de/part/349/info; Stock (none) -> 0; manf# 08056C105MAT2A -> 08053G105MAT2A; mouser# 581-08056C105MAT2A -> 581-08053G105MAT2A
- C1403, C1404: symbol Device:C -> partdb:08055C104K4Z4A; Category (none) -> Kondensator/MLCC; MPN (none) -> 08055C104K4Z4A; Manufacturer (none) -> KYOCERA AVX; Manufacturing Status (none) -> Active; Mass (none) -> 0.006 g; Mouser SPN (none) -> 581-08055C104K4Z4A; Part-DB Footprint (none) -> 0805; Part-DB ID (none) -> 109; Part-DB URL (none) -> https://inventory.lan/de/part/109/info; Stock (none) -> 6; Storage Location (none) -> Sortierregal; manf# 08053C104M4T4A -> 08055C104K4Z4A; mouser# 581-08053C104M4T4A -> 581-08055C104K4Z4A
- LED1401: symbol Device:LED -> partdb:SM0805YC; Category (none) -> Diode/LED/Gelb; MPN (none) -> SM0805YC; Manufacturer (none) -> Bivar; Manufacturing Status (none) -> Active; Mass (none) -> 0.004 g; Mouser SPN (none) -> 749-SM0805YC; Part-DB Footprint (none) -> 0805; Part-DB ID (none) -> 324; Part-DB URL (none) -> https://inventory.lan/de/part/324/info; Stock (none) -> 0
- MP1401: symbol Mechanical_Kampi:Light_Pipe -> Mechanical:Light_Pipe
- R1401: symbol Device:R -> partdb:CR0805-FX-1002ELF; Category (none) -> Widerstand/Dickfilmwiderstand; MPN (none) -> CR0805-FX-1002ELF; Manufacturer (none) -> Bourns; Manufacturing Status (none) -> Active; Mass (none) -> 0.006 g; Mouser SPN (none) -> 652-CR0805FX-1002ELF; Part-DB Footprint (none) -> 0805; Part-DB ID (none) -> 343; Part-DB URL (none) -> https://inventory.lan/de/part/343/info; Stock (none) -> 0; manf# CR0805-FX-1002GLF -> CR0805-FX-1002ELF; mouser# 652-CR0805-FX-1002GLF -> 652-CR0805FX-1002ELF
- R1403, R1404, R1405, R1406: symbol Device:R -> partdb:CR0805-J/-000ELF; Category (none) -> Widerstand/Dickfilmwiderstand; MPN (none) -> CR0805-J/-000ELF; Manufacturer (none) -> Bourns; Manufacturing Status (none) -> Active; Mass (none) -> 0.006 g; Mouser SPN (none) -> 652-CR0805-J/-000ELF; Part-DB Footprint (none) -> 0805; Part-DB ID (none) -> 322; Part-DB URL (none) -> https://inventory.lan/de/part/322/info; Stock (none) -> 0
- R1407: symbol Device:R -> partdb:CR0805-FX-1002ELF; Category (none) -> Widerstand/Dickfilmwiderstand; MPN (none) -> CR0805-FX-1002ELF; Manufacturer (none) -> Bourns; Manufacturing Status (none) -> Active; Mass (none) -> 0.006 g; Mouser SPN (none) -> 652-CR0805FX-1002ELF; Part-DB Footprint (none) -> 0805; Part-DB ID (none) -> 343; Part-DB URL (none) -> https://inventory.lan/de/part/343/info; Stock (none) -> 0; manf# CR0805-JW-103GLF -> CR0805-FX-1002ELF; mouser# 652-CR0805-JW-103GLF -> 652-CR0805FX-1002ELF
