File: gateway/wMBus.kicad_sch (KiCad schematic)
At the start: 21 parts, among them IC1401 TLV75733PDBV, IC1402 74LVC1G07, IC1403 TXB0102DCT, M1401 iM891A-XL

Commit message: Prepare release 1.0.0
Parts:
- AE1401, C1401, C1402, C1403, C1404, IC1401, IC1402, IC1403, LED1401, M1401, R1401, R1402, R1403, R1404, R1405, R1406, R1407: Config (none) -> +WMBUS
Changed lines of the file:
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@@
 			)
 		)
+		(property "Config" "+WMBUS"
+			(at 0 0 0)
+			(show_name no)
+			(do_not_autoplace no)
+			(effects
+				(font
+					(size 1.27 1.27)
+				)
+			)
+		)
 		(pin "2"
 		)
@@
 			)
 		)
+		(property "Config" "+WMBUS"
+			(at 0 0 0)
+			(show_name no)
+			(do_not_autoplace no)
+			(effects
+				(font
+					(size 1.27 1.27)
+				)
+			)
+		)
 		(pin "1"
 		)
@@
 			)
 		)
+		(property "Config" "+WMBUS"
+			(at 44.45 251.46 0)
+			(hide yes)
+			(show_name no)
+			(do_not_autoplace no)
+			(effects
+				(font
+					(size 1.27 1.27)
+				)
+			)
+		)
 		(pin "2"
 		)
@@
 			)
 		)
+		(property "Config" "+WMBUS"
+			(at 0 502.92 0)
+			(hide yes)
+			(show_name no)
+			(do_not_autoplace no)
+			(effects
+				(font
+					(size 1.27 1.27)
+				)
+			)
+		)
 		(pin "2"
 		)
@@
 			)
 		)
+		(property "Config" "+WMBUS"
+			(at 383.54 0 0)
+			(show_name no)
+			(do_not_autoplace no)
+			(effects
+				(font
+					(size 1.27 1.27)
+				)
+			)
+		)
 		(pin "1"
 		)
@@
 			)
 		)
+		(property "Config" "+WMBUS"
+			(at 0 0 0)
+			(show_name no)
+			(do_not_autoplace no)
+			(effects
+				(font
+					(size 1.27 1.27)
+				)
+			)
+		)
 		(pin "1"
 		)
@@
 			)
 		)
+		(property "Config" "+WMBUS"
+			(at 27.94 375.92 0)
+			(hide yes)
+			(show_name no)
+			(do_not_autoplace no)
+			(effects
+				(font
+					(size 1.27 1.27)
+				)
+			)
+		)
 		(pin "1"
 		)
@@
 			)
 		)
+		(property "Config" "+WMBUS"
+			(at 0 0 0)
+			(hide yes)
+			(show_name no)
+			(do_not_autoplace no)
+			(effects
+				(font
+					(size 1.27 1.27)
+				)
+			)
+		)
 		(pin "2"
 		)
@@
 			)
 		)
+		(property "Config" "+WMBUS"
+			(at 0 0 0)
+			(show_name no)
+			(do_not_autoplace no)
+			(effects
+				(font
+					(size 1.27 1.27)
+				)
+			)
+		)
 		(pin "5"
 		)
@@
 			)
 		)
+		(property "Config" "+WMBUS"
+			(at 0 0 0)
+			(show_name no)
+			(do_not_autoplace no)
+			(effects
+				(font
+					(size 1.27 1.27)
+				)
+			)
+		)
 		(pin "2"
 		)
@@
 			)
 		)
+		(property "Config" "+WMBUS"
+			(at 33.02 370.84 0)
+			(hide yes)
+			(show_name no)
+			(do_not_autoplace no)
+			(effects
+				(font
+					(size 1.27 1.27)
+				)
+			)
+		)
 		(pin "1"
 		)
@@
 			)
 		)
+		(property "Config" "+WMBUS"
+			(at -12.7 335.28 0)
+			(hide yes)
+			(show_name no)
+			(do_not_autoplace no)
+			(effects
+				(font
+					(size 1.27 1.27)
+				)
+			)
+		)
 		(pin "1"
 		)
@@
 			)
 		)
+		(property "Config" "+WMBUS"
+			(at -7.62 330.2 0)
+			(hide yes)
+			(show_name no)
+			(do_not_autoplace no)
+			(effects
+				(font
+					(size 1.27 1.27)
+				)
+			)
+		)
 		(pin "1"
 		)
@@
 			)
 		)
+		(property "Config" "+WMBUS"
+			(at 358.14 358.14 0)
+			(hide yes)
+			(show_name no)
+			(do_not_autoplace no)
+			(effects
+				(font
+					(size 1.27 1.27)
+				)
+			)
+		)
 		(pin "1"
 		)
@@
 			)
 		)
+		(property "Config" "+WMBUS"
+			(at 199.39 274.32 0)
+			(hide yes)
+			(show_name no)
+			(do_not_autoplace no)
+			(effects
+				(font
+					(size 1.27 1.27)
+				)
+			)
+		)
 		(pin "1"
 		)
@@
 			)
 		)
+		(property "Config" ""
+			(at 187.96 276.86 0)
+			(hide yes)
+			(show_name no)
+			(do_not_autoplace no)
+			(effects
+				(font
+					(size 1.27 1.27)
+				)
+			)
+		)
 		(instances
 			(project "Gateway"
@@
 			)
 		)
+		(property "Config" "+WMBUS"
+			(at 218.44 0 0)
+			(show_name no)
+			(do_not_autoplace no)
+			(effects
+				(font
+					(size 1.27 1.27)
+				)
+			)
+		)
 		(pin "1"
 		)
@@
 			(hide yes)
 			(show_name no)
+			(do_not_autoplace no)
+			(effects
+				(font
+					(size 1.27 1.27)
+				)
+			)
+		)
+		(property "Config" "+WMBUS"
+			(at 0 0 0)
+			(hide yes)
+			(show_name no)

Commit message: Smaller changes
Changed lines of the file:
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@@
 		(property "Config" "+WMBUS"
 			(at 0 0 0)
+			(hide yes)
 			(show_name no)
 			(do_not_autoplace no)
@@
 		(property "Config" "+WMBUS"
 			(at 0 0 0)
+			(hide yes)
 			(show_name no)
 			(do_not_autoplace no)
@@
 		(property "Config" "+WMBUS"
 			(at 383.54 0 0)
+			(hide yes)
 			(show_name no)
 			(do_not_autoplace no)
@@
 		(property "Config" "+WMBUS"
 			(at 0 0 0)
+			(hide yes)
 			(show_name no)
 			(do_not_autoplace no)
@@
 		(property "Config" "+WMBUS"
 			(at 0 0 0)
+			(hide yes)
 			(show_name no)
 			(do_not_autoplace no)
@@
 		(property "Config" "+WMBUS"
 			(at 0 0 0)
+			(hide yes)
 			(show_name no)
 			(do_not_autoplace no)
@@
 		(property "Config" "+WMBUS"
 			(at 218.44 0 0)
+			(hide yes)
 			(show_name no)
 			(do_not_autoplace no)

Commit message: Working on revision 1.0.0
Parts:
- C1401, C1402: symbol Device:C -> partdb:08053G105MAT2A; Category (none) -> Kondensator/MLCC; MPN (none) -> 08053G105MAT2A; Manufacturer (none) -> KYOCERA AVX; Manufacturing Status (none) -> Active; Mass (none) -> 0.006 g; Mouser SPN (none) -> 581-08053G105MAT2A; Part-DB Footprint (none) -> 0805; Part-DB ID (none) -> 349; Part-DB URL (none) -> https://inventory.lan/de/part/349/info; Stock (none) -> 0; manf# 08056C105MAT2A -> 08053G105MAT2A; mouser# 581-08056C105MAT2A -> 581-08053G105MAT2A
- C1403, C1404: symbol Device:C -> partdb:08055C104K4Z4A; Category (none) -> Kondensator/MLCC; MPN (none) -> 08055C104K4Z4A; Manufacturer (none) -> KYOCERA AVX; Manufacturing Status (none) -> Active; Mass (none) -> 0.006 g; Mouser SPN (none) -> 581-08055C104K4Z4A; Part-DB Footprint (none) -> 0805; Part-DB ID (none) -> 109; Part-DB URL (none) -> https://inventory.lan/de/part/109/info; Stock (none) -> 6; Storage Location (none) -> Sortierregal; manf# 08053C104M4T4A -> 08055C104K4Z4A; mouser# 581-08053C104M4T4A -> 581-08055C104K4Z4A
- IC1403: value TXB0102DCT -> TXB0102DCU; Category (none) -> IC/Pegelwandler; MPN (none) -> TXB0102DCUR; Manufacturer (none) -> Texas Instruments; Mass (none) -> 0.01 g; Mouser SPN (none) -> 595-TXB0102DCUR; Part-DB Footprint (none) -> VSSOP-8_2.3x2mm_P0.5mm; Part-DB ID (none) -> 280; Part-DB URL (none) -> https://inventory.lan/de/part/280/info; Stock (none) -> 0; manf# TXB0102DCT -> TXB0102DCUR; mouser# 595-TXB0102DCT -> 595-TXB0102DCUR
- LED1401: symbol Device:LED -> partdb:SM0805YC; Category (none) -> Diode/LED/Gelb; MPN (none) -> SM0805YC; Manufacturer (none) -> Bivar; Manufacturing Status (none) -> Active; Mass (none) -> 0.004 g; Mouser SPN (none) -> 749-SM0805YC; Part-DB Footprint (none) -> 0805; Part-DB ID (none) -> 324; Part-DB URL (none) -> https://inventory.lan/de/part/324/info; Stock (none) -> 0
- MP1401: symbol Mechanical_Kampi:Light_Pipe -> Mechanical:Light_Pipe
- R1401: symbol Device:R -> partdb:CR0805-FX-1002ELF; Category (none) -> Widerstand/Dickfilmwiderstand; MPN (none) -> CR0805-FX-1002ELF; Manufacturer (none) -> Bourns; Manufacturing Status (none) -> Active; Mass (none) -> 0.006 g; Mouser SPN (none) -> 652-CR0805FX-1002ELF; Part-DB Footprint (none) -> 0805; Part-DB ID (none) -> 343; Part-DB URL (none) -> https://inventory.lan/de/part/343/info; Stock (none) -> 0; manf# CR0805-FX-1002GLF -> CR0805-FX-1002ELF; mouser# 652-CR0805-FX-1002GLF -> 652-CR0805FX-1002ELF
- R1403, R1404, R1405, R1406: symbol Device:R -> partdb:CR0805-J/-000ELF; Category (none) -> Widerstand/Dickfilmwiderstand; MPN (none) -> CR0805-J/-000ELF; Manufacturer (none) -> Bourns; Manufacturing Status (none) -> Active; Mass (none) -> 0.006 g; Mouser SPN (none) -> 652-CR0805-J/-000ELF; Part-DB Footprint (none) -> 0805; Part-DB ID (none) -> 322; Part-DB URL (none) -> https://inventory.lan/de/part/322/info; Stock (none) -> 0
- R1407: symbol Device:R -> partdb:CR0805-FX-1002ELF; Category (none) -> Widerstand/Dickfilmwiderstand; MPN (none) -> CR0805-FX-1002ELF; Manufacturer (none) -> Bourns; Manufacturing Status (none) -> Active; Mass (none) -> 0.006 g; Mouser SPN (none) -> 652-CR0805FX-1002ELF; Part-DB Footprint (none) -> 0805; Part-DB ID (none) -> 343; Part-DB URL (none) -> https://inventory.lan/de/part/343/info; Stock (none) -> 0; manf# CR0805-JW-103GLF -> CR0805-FX-1002ELF; mouser# 652-CR0805-JW-103GLF -> 652-CR0805FX-1002ELF
