File: gateway/wMBus.kicad_sch (KiCad schematic)
At the start: 21 parts, among them IC1401 TLV75733PDBV, IC1402 74LVC1G07, IC1403 TXB0102DCU, M1401 iM891A-XL

Commit message: Prepare Release 1.0.0
Co-Authored-By: Claude Opus 5.5 <noreply@anthropic.com>
Parts:
- R1302: renamed from R1402; mouser# 652-CR0805-JW-680GLF -> 652-CR0805JW-680GLF
- renumbered AE1401 to AE1301, C1401 to C1301, C1402 to C1302, C1403 to C1303, C1404 to C1304, IC1401 to IC1301, IC1402 to IC1302, IC1403 to IC1303, LED1401 to LED1301, M1401 to M1301, MP1401 to MP1301, R1401 to R1301, R1403 to R1303, R1404 to R1304, R1405 to R1305, R1406 to R1306, R1407 to R1307, TP1401 to TP1301, TP1402 to TP1302, TP1403 to TP1303
