File: gateway/wMBus.kicad_sch (KiCad schematic)
At the start: 21 parts, among them IC1401 TLV75733PDBV, IC1402 74LVC1G07, IC1403 TXB0102DCU, M1401 iM891A-XL

Commit message: Prepare Release 1.0.0
Co-Authored-By: Claude Opus 5.5 <noreply@anthropic.com>
Parts:
- IC1301: renamed from IC1401; manf# TLV75733PDBVR -> TLV75733PDBVT; mouser# 595-TLV75733PDBVR -> 595-TLV75733PDBVT
- IC1302: renamed from IC1402; manf Diodes Incorporated -> Nexperia; manf# 74LVC1G07QSE-7 -> 74LVC1G07GW,125; mouser# 621-74LVC1G07QSE-7 -> 771-74LVC1G07GW-G
- R1302: renamed from R1402; mouser# 652-CR0805-JW-680GLF -> 652-CR0805JW-680GLF
- renumbered AE1401 to AE1301, C1401 to C1301, C1402 to C1302, C1403 to C1303, C1404 to C1304, IC1403 to IC1303, LED1401 to LED1301, M1401 to M1301, MP1401 to MP1301, R1401 to R1301, R1403 to R1303, R1404 to R1304, R1405 to R1305, R1406 to R1306, R1407 to R1307, TP1401 to TP1301, TP1402 to TP1302, TP1403 to TP1303

Commit message: Update schematic and board
- Use Part-DB symbols, BT901 changed to Keystone 3030TR
- Add the revision text to the board
- Include more parts in BOM and position files

Co-Authored-By: Claude Opus 5.5 <noreply@anthropic.com>
Parts:
- R1301: now in the parts list
Changed lines of the file:
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@@
 		(body_style 1)
 		(exclude_from_sim no)
-		(in_bom no)
+		(in_bom yes)
 		(on_board yes)
-		(in_pos_files no)
+		(in_pos_files yes)
 		(dnp yes)
 		(property "Reference" "R1301"
