File: gateway/Gateway.kicad_sch (KiCad schematic)
At the start: 0 parts

Commit message: Prepare Release 1.0.0
Co-Authored-By: Claude Opus 5.5 <noreply@anthropic.com>
Other:
- removed sheet Power - Sequencing
Changed lines of the file:
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@@
-			(project "Gateway"
-				(path "/d5742f03-3b1a-42e5-a384-018bd4b919aa"
-					(page "5")
-				)
-			)
-		)
-	)
-	(sheet
-		(at 346.71 314.96)
-		(size 35.56 5.08)
-		(exclude_from_sim no)
-		(in_bom yes)
-		(on_board yes)
-		(dnp no)
-		(stroke
-			(width 0.1524)
-			(type solid)
-		)
-		(fill
-			(color 0 0 0 0)
-		)
-		(property "Sheetname" "Power - Sequencing"
-			(at 346.71 313.9309 0)
-			(show_name no)
-			(do_not_autoplace no)
-			(effects
-				(font
-					(face "Times New Roman")
-					(size 1.905 1.905)
-					(bold yes)
-					(color 0 0 0 1)
-				)
-				(justify left bottom)
-			)
-		)
-		(property "Sheetfile" "Power - Sequencing.kicad_sch"
-			(at 347.98 316.23 0)
-			(show_name no)
-			(do_not_autoplace no)
-			(effects
-				(font
-					(face "Arial")
-					(size 1.27 1.27)
-				)
-				(justify left top)
-			)
-		)
-		(instances
-			(project "KDT_Hierarchical_KiBot"
-				(path "/f9e05184-c88b-4a88-ae9c-ab2bdb32be7c"
-					(page "6")
-				)
-			)
 			(project "Gateway"
 				(path "/d5742f03-3b1a-42e5-a384-018bd4b919aa"
@@
 			(project "Gateway"
 				(path "/d5742f03-3b1a-42e5-a384-018bd4b919aa"
-					(page "18")
+					(page "17")
 				)
 			)
@@
 			(project "Gateway"
 				(path "/d5742f03-3b1a-42e5-a384-018bd4b919aa"
-					(page "6")
+					(page "5")
 				)
 			)
