File: gateway/Thread.kicad_sch (KiCad schematic)
At the start: 33 parts, among them IC1301 TLV75733PDBV, IC1302 74LVC1G07, IC1303 74LVC1G07, IC1304 TXB0104PWR, M1301 BT40, X1301 DEBUG, X1302 UART

Commit message: Prepare Release 1.0.0
Co-Authored-By: Claude Opus 5.5 <noreply@anthropic.com>
Parts:
- R1202: renamed from R1302; mouser# 652-CR0805-JW-680GLF -> 652-CR0805JW-680GLF
- R1203: renamed from R1303; mouser# 652-CR0805-JW-680GLF -> 652-CR0805JW-680GLF
- renumbered AE1301 to AE1201, C1301 to C1201, C1302 to C1202, C1303 to C1203, C1304 to C1204, IC1301 to IC1201, IC1302 to IC1202, IC1303 to IC1203, IC1304 to IC1204, LED1301 to LED1201, LED1302 to LED1202, M1301 to M1201, MP1301 to MP1201, R1301 to R1201, R1304 to R1204, R1305 to R1205, R1306 to R1206, R1307 to R1207, R1308 to R1208, R1309 to R1209, R1310 to R1210, R1311 to R1211, R1312 to R1212, R1313 to R1213, TP1301 to TP1201, TP1302 to TP1202, TP1303 to TP1203, TP1304 to TP1204, TP1309 to TP1205, X1301 to X1201, X1302 to X1202
