File: gateway/Thread.kicad_sch (KiCad schematic)
At the start: 33 parts, among them IC1301 TLV75733PDBV, IC1302 74LVC1G07, IC1303 74LVC1G07, IC1304 TXB0104PWR, M1301 BT40, X1301 DEBUG, X1302 UART

Commit message: Prepare Release 1.0.0
Co-Authored-By: Claude Opus 5.5 <noreply@anthropic.com>
Parts:
- IC1201: renamed from IC1301; manf# TLV75733PDBVR -> TLV75733PDBVT; mouser# 595-TLV75733PDBVR -> 595-TLV75733PDBVT
- IC1202: renamed from IC1302; manf Diodes Incorporated -> Nexperia; manf# 74LVC1G07QSE-7 -> 74LVC1G07GW,125; mouser# 621-74LVC1G07QSE-7 -> 771-74LVC1G07GW-G
- IC1203: renamed from IC1303; manf Diodes Incorporated -> Nexperia; manf# 74LVC1G07QSE-7 -> 74LVC1G07GW,125; mouser# 621-74LVC1G07QSE-7 -> 771-74LVC1G07GW-G
- IC1204: renamed from IC1304; value TXB0104PWR -> NXB0104PW; manf Texas Instruments -> Nexperia; manf# TXB0104PWR -> NXB0104PWJ; mouser# 595-TXB0104PWR -> 771-NXB0104PWJ
- R1202: renamed from R1302; mouser# 652-CR0805-JW-680GLF -> 652-CR0805JW-680GLF
- R1203: renamed from R1303; mouser# 652-CR0805-JW-680GLF -> 652-CR0805JW-680GLF
- renumbered AE1301 to AE1201, C1301 to C1201, C1302 to C1202, C1303 to C1203, C1304 to C1204, LED1301 to LED1201, LED1302 to LED1202, M1301 to M1201, MP1301 to MP1201, R1301 to R1201, R1304 to R1204, R1305 to R1205, R1306 to R1206, R1307 to R1207, R1308 to R1208, R1309 to R1209, R1310 to R1210, R1311 to R1211, R1312 to R1212, R1313 to R1213, TP1301 to TP1201, TP1302 to TP1202, TP1303 to TP1203, TP1304 to TP1204, TP1309 to TP1205, X1301 to X1201, X1302 to X1202

Commit message: Update schematic and board
- Use Part-DB symbols, BT901 changed to Keystone 3030TR
- Add the revision text to the board
- Include more parts in BOM and position files

Co-Authored-By: Claude Opus 5.5 <noreply@anthropic.com>
Parts:
- R1201: now in the parts list
Changed lines of the file:
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@@
 		(body_style 1)
 		(exclude_from_sim no)
-		(in_bom no)
+		(in_bom yes)
 		(on_board yes)
-		(in_pos_files no)
+		(in_pos_files yes)
 		(dnp yes)
 		(property "Reference" "R1201"
