File: gateway/SoM.kicad_sch (KiCad schematic)
At the start: 25 parts, among them Q1001 BSS138, SW1001 Reset, SW1002 On / Off, X1001 UART, X1002 SoM

Commit message: Prepare Release 1.0.0
Co-Authored-By: Claude Opus 5.5 <noreply@anthropic.com>
Parts:
- R902: renamed from R1005; mouser# 652-CR0805-JW-152GLF -> 652-CR0805JW-152GLF
- renumbered BT1001 to BT901, C1001 to C901, H1001 to H901, H1003 to H902, H1002 to H903, JP1001 to JP901, LED1001 to LED901, MP1001 to MP901, Q1001 to Q901, R1004 to R901, R1001 to R903, R1002 to R904, R1006 to R905, R1007 to R906, R1008 to R907, R1009 to R908, R1010 to R909, R1011 to R910, R1012 to R911, R1013 to R912, SW1001 to SW901, SW1002 to SW902, X1001 to X901, X1002 to X902

Commit message: Update schematic and board
- Use Part-DB symbols, BT901 changed to Keystone 3030TR
- Add the revision text to the board
- Include more parts in BOM and position files

Co-Authored-By: Claude Opus 5.5 <noreply@anthropic.com>
Parts:
- BT901: symbol Device:Battery_Cell -> partdb:3030TR; Category (none) -> Batterie/Batteriehalter; MPN (none) -> 3030TR; Manufacturer (none) -> Keystone Electronics; Manufacturing Status (none) -> Active; Mass (none) -> 1 g; Mouser SPN (none) -> 534-3030TR; Part-DB Footprint (none) -> 3030TR; Part-DB ID (none) -> 391; Part-DB URL (none) -> https://inventory.lan/de/part/391/info; Stock (none) -> 0; manf# 3030KTR -> 3030TR; mouser# 534-3030KTR -> 534-3030TR
Changed lines of the file:
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@@
 		(in_bom yes)
 		(on_board yes)
-		(in_pos_files no)
+		(in_pos_files yes)
 		(dnp yes)
 		(property "Reference" "R906"
@@
 			)
 		)
+		(property "Config" ""
+			(at 318.77 107.95 0)
+			(hide yes)
+			(show_name no)
+			(do_not_autoplace no)
+			(effects
+				(font
+					(size 1.27 1.27)
+				)
+			)
+		)
 		(pin "1"
 		)
@@
 		(in_bom yes)
 		(on_board yes)
-		(in_pos_files no)
+		(in_pos_files yes)
 		(dnp yes)
 		(property "Reference" "R905"
@@
 		(in_bom yes)
 		(on_board yes)
-		(in_pos_files no)
+		(in_pos_files yes)
 		(dnp yes)
 		(property "Reference" "R910"
@@
 			)
 		)
+		(property "Config" ""
+			(at 303.53 190.5 0)
+			(hide yes)
+			(show_name no)
+			(do_not_autoplace no)
+			(effects
+				(font
+					(size 1.27 1.27)
+				)
+			)
+		)
 		(pin "1"
 		)
@@
 	)
 	(symbol
-		(lib_id "Device:Battery_Cell")
+		(lib_id "partdb:3030TR")
 		(at 215.9 168.91 0)
 		(mirror y)
@@
 			)
 		)
-		(property "Datasheet" "https://www.keyelco.com/product-pdf.cfm?p=14595"
+		(property "Datasheet" "https://www.mouser.com/datasheet/3/201/1/3030TR.pdf"
 			(at 215.9 167.386 90)
 			(hide yes)
@@
 			)
 		)
-		(property "Description" "Single-cell battery"
+		(property "Description" "Knopfzellen-Batteriehalter SM RETAINER TAPE/REEL 1500PC 10mm"
 			(at 215.9 168.91 0)
 			(hide yes)
@@
 			)
 		)
-		(property "manf#" "3030KTR"
+		(property "manf#" "3030TR"
+			(at 215.9 168.91 0)
+			(hide yes)
+			(show_name no)
+			(do_not_autoplace no)
+			(effects
+				(font
+					(size 1.27 1.27)
+				)
+			)
+		)
+		(property "mouser#" "534-3030TR"
+			(at 215.9 168.91 0)
+			(hide yes)
+			(show_name no)
+			(do_not_autoplace no)
+			(effects
+				(font
+					(size 1.27 1.27)
+				)
+			)
+		)
+		(property "Config" ""
+			(at 215.9 168.91 0)
+			(hide yes)
+			(show_name no)
+			(do_not_autoplace no)
+			(effects
+				(font
+					(size 1.27 1.27)
+				)
+			)
+		)
+		(property "Sim.Device" "V"
 			(at 215.9 168.91 0)
 			(hide yes)
@@
 			)
 		)
-		(property "mouser#" "534-3030KTR"
+		(property "Sim.Type" "DC"
+			(at 215.9 168.91 0)
+			(hide yes)
+			(show_name no)
+			(do_not_autoplace no)
+			(effects
+				(font
+					(size 1.27 1.27)
+				)
+			)
+		)
+		(property "Sim.Pins" "1=+ 2=-"
+			(at 215.9 168.91 0)
+			(hide yes)
+			(show_name no)
+			(do_not_autoplace no)
+			(effects
+				(font
+					(size 1.27 1.27)
+				)
+			)
+		)
+		(property "Part-DB URL" "https://inventory.lan/de/part/391/info"
+			(at 215.9 168.91 0)
+			(hide yes)
+			(show_name no)
+			(do_not_autoplace no)
+			(effects
+				(font
+					(size 1.27 1.27)
+				)
+			)
+		)
+		(property "Category" "Batterie/Batteriehalter"
+			(at 215.9 168.91 0)
+			(hide yes)
+			(show_name no)
+			(do_not_autoplace no)
+			(effects
+				(font
+					(size 1.27 1.27)
+				)
+			)
+		)
+		(property "Manufacturer" "Keystone Electronics"
+			(at 215.9 168.91 0)
+			(hide yes)
+			(show_name no)
+			(do_not_autoplace no)
+			(effects
+				(font
+					(size 1.27 1.27)
+				)
+			)
+		)
+		(property "MPN" "3030TR"
+			(at 215.9 168.91 0)
+			(hide yes)
+			(show_name no)
+			(do_not_autoplace no)
+			(effects
+				(font
+					(size 1.27 1.27)
+				)
+			)
+		)
+		(property "Manufacturing Status" "Active"
+			(at 215.9 168.91 0)
+			(hide yes)
+			(show_name no)
+			(do_not_autoplace no)
+			(effects
+				(font
+					(size 1.27 1.27)
+				)
+			)
+		)
+		(property "Part-DB Footprint" "3030TR"
+			(at 215.9 168.91 0)
+			(hide yes)
+			(show_name no)
+			(do_not_autoplace no)
+			(effects
+				(font
+					(size 1.27 1.27)
+				)
+			)
+		)
+		(property "Mass" "1 g"
+			(at 215.9 168.91 0)
+			(hide yes)
+			(show_name no)
+			(do_not_autoplace no)
+			(effects
+				(font
+					(size 1.27 1.27)
+				)
+			)
+		)
+		(property "Part-DB ID" "391"
+			(at 215.9 168.91 0)
+			(hide yes)
+			(show_name no)
+			(do_not_autoplace no)
+			(effects
+				(font
+					(size 1.27 1.27)
+				)
+			)
+		)
+		(property "Mouser SPN" "534-3030TR"
+			(at 215.9 168.91 0)
+			(hide yes)
+			(show_name no)
+			(do_not_autoplace no)
+			(effects
+				(font
+					(size 1.27 1.27)
+				)
+			)
+		)
+		(property "Stock" "0"
 			(at 215.9 168.91 0)
 			(hide yes)
